File: hardware/PV-PWR-4/sheets/01_pc.kicad_sch (KiCad schematic)
At the start: 84 parts, among them J101 X9555WV-2x32-6TV01, Q101 BSS138BK, Q102 BSS138BK, Q103 BSS138BK, Q104 BSS138BK, U101 SN74AHCT1G08DBVR, U102 SN74AHCT1G08DBVR, U103 SN74AHCT1G08DBVR, U104 SN74AHCT1G08DBVR, U105 SN74AHCT1G08DBVR, U106 SN74AHCT1G08DBVR, U107 SN74AHCT1G08DBVR, U108 SN74AHCT1G08DBVR, U109 SN74AHCT1G08DBVR, U110 SN74AHCT1G08DBVR, U111 SN74AHCT1G08DBVR, U112 SN74AHCT1G08DBVR, U113 SN74AHCT1G08DBVR, U114 SN74AHCT1G08DBVR, U115 SN74AHCT1G08DBVR, U116 SN74AHCT1G08DBVR, U117 SN74AHCT1G08DBVR, U118 SN74AHCT1G08DBVR, U119 SN74AHCT1G08DBVR, U120 TPS3710DDCR, U121 SN74LVC1G32DBVR

Commit message: Board revisions PV-PWR A2 / PV-CTL A1, inverter filter magnetics, documentation refresh (D-056..D-058)
Boards (every build check passes)
- PV-PWR / PV-PWR-4 rev A2: seventh battery-side film capacitor on the three-phase board (closes the
  load-rejection overshoot), bleeder 8 x 73.2 k so the bank still discharges within its 10-minute label.
- PV-CTL rev A1: hardware over-current window 68.9-79.9 A, thresholds derived from each sensor's own
  reference; the board-to-board contract carries the four references on the former 24 V / 5 V pins.
- Records aligned (contract comments, architecture corrections, port-current bandwidth); the frozen
  platform's module BOMs are kept instead of being re-rolled from the cost-first thermal data.

Magnetics
- Inverter filter designed and verified: L1, L2 and the AC common-mode choke (design_pcs_*.json). The filter
  comes to 745 USD at catalogue prices and 611 USD at 5,000 units, against 207 / 167 in the study: the
  inverter's cost is provisional and its stage and filter are being re-optimised.
- PV inductor loss check made non-circular; hot-spot margin reported per build (PV-P100/110: -5.3 K, MG-17).

Results: PV-P75 952 USD at catalogue prices / 796 USD at 5,000 units; Megarevo comparison 2 better,
24 meet, 3 below, 5 not assessed. Documentation corrected for the revised boards (51 statements).
Everything is calculated or estimated; nothing is bench-validated.

Co-Authored-By: Claude Fable 5.1 <noreply@anthropic.com>
Parts:
- removed C127: 100p 50V, symbol dcdc:C
- removed C128, C130: 100n 50V, symbol dcdc:C
- removed C129: 1n 50V, symbol dcdc:C
- C101: value 10u 50V -> 10u 16V
- C103, C105: value 10u 16V -> 100n 50V; Package 1210 -> 0603
- C122, C123: value 100n 50V -> 100p 50V
- C125: value 100n 50V -> 1n 50V
- C126: value 100p 50V -> 100n 50V
Connections:
- net +3V3: now also C101.1, C102.1, C126.1; no longer C105.1, C106.1
- net +5V: now also C105.1, C106.1; no longer C121.1, C122.1, C123.1, J101.5 (Pin_5), J101.6 (Pin_6)
- net +5V_GD: now also C121.1; no longer C125.1
- net FLT_N: now also C123.1
- net RDY: now also C122.1; no longer C126.1
- net SUP5_SNS: now also C125.1
- removed net +24V: C101.1, C102.1, J101.1 (Pin_1), J101.2 (Pin_2)
- new net IL1R: J101.1 (Pin_1)
- new net IL2R: J101.2 (Pin_2)
- new net IL3R: J101.5 (Pin_5)
- new net IL4R: J101.6 (Pin_6)
Other:
- note added: "Both boards live: GND = AGND = BUS-. +3V3 goes TO the control board (rev A2: the former +24V / +5V pins carry the sensor references IL1R-IL4R). Commands are 3.3 V logic after the control board's trip latch; every command input is pulled low here (open = off)."
- note removed: "Both boards live: GND = AGND = BUS-. Supplies +24V / +5V / +3V3 go TO the control board. Commands are 3.3 V logic after the control board's trip latch; every command input is pulled low here (open = off)."
- moved on the sheet: C103, C104, C105, C106, C107, C108, C109, C110, C111, C112, C113, C114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
