File: hardware/PV-PWR-4/sheets/02_ph1_power.kicad_sch (KiCad schematic)
At the start: 127 parts, among them J201 7461057, J202 7461057, J203 KF2EDGR-3.5-2P, J204 KF2EDGR-3.5-2P, P201 PAD AlN 1 mm (CUSTOM), P202 PAD AlN 1 mm (CUSTOM), P203 PAD AlN 1 mm (CUSTOM), P204 PAD AlN 1 mm (CUSTOM), P205 PAD AlN 1 mm (CUSTOM), P206 PAD AlN 1 mm (CUSTOM), P207 PAD AlN 1 mm (CUSTOM), P208 PAD AlN 1 mm (CUSTOM), Q201 SG2M040170HJ, Q202 SG2M040170HJ, Q203 SG2M040170HJ, Q204 SG2M040170HJ, Q205 SG2M040170HJ, Q206 SG2M040170HJ, Q207 SG2M040170HJ, Q208 SG2M040170HJ, Q209 PBSS5540X,135, Q210 PBSS5540X,135, Q211 PBSS5540X,135, Q212 PBSS5540X,135, T201 Gate-bias transformer per pha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, U201 SN6505BDBVR, U202 ATL431BIDBZR, U203 ATL431BIDBZR, U204 ATL431BIDBZR, U205 ATL431BIDBZR, U206 ATL431BIDBZR, U207 ATL431BIDBZR, U208 ATL431BIDBZR, U209 ATL431BIDBZR

Commit message: Board revisions PV-PWR A2 / PV-CTL A1, inverter filter magnetics, documentation refresh (D-056..D-058)
Boards (every build check passes)
- PV-PWR / PV-PWR-4 rev A2: seventh battery-side film capacitor on the three-phase board (closes the
  load-rejection overshoot), bleeder 8 x 73.2 k so the bank still discharges within its 10-minute label.
- PV-CTL rev A1: hardware over-current window 68.9-79.9 A, thresholds derived from each sensor's own
  reference; the board-to-board contract carries the four references on the former 24 V / 5 V pins.
- Records aligned (contract comments, architecture corrections, port-current bandwidth); the frozen
  platform's module BOMs are kept instead of being re-rolled from the cost-first thermal data.

Magnetics
- Inverter filter designed and verified: L1, L2 and the AC common-mode choke (design_pcs_*.json). The filter
  comes to 745 USD at catalogue prices and 611 USD at 5,000 units, against 207 / 167 in the study: the
  inverter's cost is provisional and its stage and filter are being re-optimised.
- PV inductor loss check made non-circular; hot-spot margin reported per build (PV-P100/110: -5.3 K, MG-17).

Results: PV-P75 952 USD at catalogue prices / 796 USD at 5,000 units; Megarevo comparison 2 better,
24 meet, 3 below, 5 not assessed. Documentation corrected for the revised boards (51 statements).
Everything is calculated or estimated; nothing is bench-validated.

Co-Authored-By: Claude Fable 5.1 <noreply@anthropic.com>
Parts:
- added C233: 2.2u 50V, symbol dcdc:C
- added R243: 10k, symbol dcdc:R
- C217: value 100n 50V -> 1n 50V
- C219: value 10u 16V -> 100n 50V; Package 1206 -> 0603
- C220: value 100n 50V -> 10u 16V; Package 0603 -> 1206
- C221: value 4.7u 50V -> 100n 50V; Domain GD_P1S1 -> LIVE; Package 1206 -> 0603
- C222, C225, C228, C231: value 10n 50V -> 4.7u 50V; Package 0603 -> 1206
- C223, C226, C229, C232: value 2.2u 50V -> 10n 50V; Package 0805 -> 0603
- C224: value 4.7u 50V -> 2.2u 50V; Domain GD_P1S2 -> GD_P1S1; Package 1206 -> 0805
- C227: value 4.7u 50V -> 2.2u 50V; Domain GD_P1S3 -> GD_P1S2; Package 1206 -> 0805
- C230: value 4.7u 50V -> 2.2u 50V; Domain GD_P1S4 -> GD_P1S3; Package 1206 -> 0805
- R214: value 10k -> 100R
- R215: Domain GD_P1S1 -> LIVE
- R216, R223, R230, R237: value 1k -> 10k
- R217, R224, R231, R238: value 77.7k -> 1k
- R218, R225, R232, R239: value 10.2k -> 77.7k
- R219, R226, R233, R240: value 4.7k -> 10.2k; Package 0805 -> 0603
- R220, R227, R234, R241: value 4.02k -> 4.7k; Package 0603 -> 0805
- R221, R228, R235, R242: value 10k -> 4.02k
- R222: Domain GD_P1S2 -> GD_P1S1
- R229: Domain GD_P1S3 -> GD_P1S2
- R236: Domain GD_P1S4 -> GD_P1S3
Connections:
- net +5V: now also C221.1; no longer C219.1
- net AGND: now also C219.2
- net BIAS_EN5: now also R215.1; no longer R214.1
- net COM_P1S1: now also R220.2, R221.1; no longer R219.2, R220.1
- net COM_P1S2: now also R227.2, R228.1; no longer R226.2, R227.1
- net COM_P1S3: now also R234.2, R235.1; no longer R233.2, R234.1
- net COM_P1S4: now also R241.2, R242.1; no longer R240.2, R241.1
- net CREF_PH1P1S1: now also R221.2, R222.1; no longer R220.2, R221.1
- net CREF_PH1P1S2: now also R228.2, R229.1; no longer R227.2, R228.1
- net CREF_PH1P1S3: now also R235.2, R236.1; no longer R234.2, R235.1
- net CREF_PH1P1S4: now also R242.2, R243.1; no longer R241.2, R242.1
- net GND: now also C221.2, R215.2; no longer C219.2, R214.2
- net NTC1: now also C218.1; no longer C217.1
- net NTC5: now also C219.1; no longer C218.1
- net RAW_PH1P1S1: now also C222.1, R216.1; no longer C221.1, R215.1
- net RAW_PH1P1S2: now also C225.1, R223.1; no longer C224.1, R222.1
- net RAW_PH1P1S3: now also C228.1, R230.1; no longer C227.1, R229.1
- net RAW_PH1P1S4: now also C231.1, R237.1; no longer C230.1, R236.1
- net RB_PH1P1S1: now also R216.2, R217.1; no longer R215.2, R216.1
- net RB_PH1P1S2: now also R223.2, R224.1; no longer R222.2, R223.1
- net RB_PH1P1S3: now also R230.2, R231.1; no longer R229.2, R230.1
- net RB_PH1P1S4: now also R237.2, R238.1; no longer R236.2, R237.1
- net RK_PH1P1S1: now also C223.1, R217.2; no longer C222.1, R216.2
- net RK_PH1P1S2: now also C226.1, R224.2; no longer C225.1, R223.2
- net RK_PH1P1S3: now also C229.1, R231.2; no longer C228.1, R230.2
- net RK_PH1P1S4: now also C232.1, R238.2; no longer C231.1, R237.2
- net RREF_PH1P1S1: now also C223.2, R218.2, R219.1; no longer C222.2, R217.2, R218.1
- net RREF_PH1P1S2: now also C226.2, R225.2, R226.1; no longer C225.2, R224.2, R225.1
- net RREF_PH1P1S3: now also C229.2, R232.2, R233.1; no longer C228.2, R231.2, R232.1
- net RREF_PH1P1S4: now also C232.2, R239.2, R240.1; no longer C231.2, R238.2, R239.1
- net VDD_P1S1: now also C224.1, R218.1, R220.1; no longer C223.1, R217.1, R219.1
- net VDD_P1S2: now also C227.1, R225.1, R227.1; no longer C226.1, R224.1, R226.1
- net VDD_P1S3: now also C230.1, R232.1, R234.1; no longer C229.1, R231.1, R233.1
- net VDD_P1S4: now also R239.1, R241.1, C233.1; no longer C232.1, R238.1, R240.1
- net VEE_P1S1: now also C222.2, C224.2, R219.2, R222.2; no longer C221.2, C223.2, R218.2, R221.2
- net VEE_P1S2: now also C225.2, C227.2, R226.2, R229.2; no longer C224.2, C226.2, R225.2, R228.2
- net VEE_P1S3: now also C228.2, C230.2, R233.2, R236.2; no longer C227.2, C229.2, R232.2, R235.2
- net VEE_P1S4: now also C231.2, R240.2, C233.2, R243.2; no longer C230.2, C232.2, R239.2, R242.2
- net IL1R_S: now reaches CS201.4 (UREF)
- net IL1R_S: now also R214.1
- new net IL1R: C217.1, R214.2
- no-connect marks 2 -> 1
Other:
- note added: "2 x FCSA3DS456 (45 uF) on A_BUS+ and 2 on B_BUS+, at this phase's legs: the banks of all phases form the port A / port B DC links (8 / 8 x 45 uF). Bleeders: one string per port on the port sheets."
- note added: "Lead A from SW_A1 passes the STK-HO/A 75 U-primary (pins 6-9 in, 10-13 out: + = SW_A -> SW_B) to stud L_A1; lead B on stud SW_B1. IL1 = 2.5 V + 10.667 mV/A (Vref 2.48-2.52 V), 0.5-4.5 V over +/-187.5 A; 100R + 1 nF at the source. IL1R = the sensor's own Uref (pin 4), 100R + 1 nF: PV-CTL references its trip window to it. Primary at the switch node: functional barrier (4 kV rms, 8 kV impulse)."
- note removed: "2 x FCSA3DS456 (45 uF) on A_BUS+ and 2 on B_BUS+, at this phase's legs: the banks of all phases form the port A / port B DC links. Bleeders: one string per port on the port sheets."
- note removed: "Lead A from SW_A1 passes the STK-HO/A 75 U-primary (pins 6-9 in, 10-13 out: + = SW_A -> SW_B) to stud L_A1; lead B on stud SW_B1. IL1 = 2.5 V + 10.667 mV/A (Vref 2.48-2.52 V), 0.5-4.5 V over +/-187.5 A; 100R + 1 nF at the source. Primary at the switch node: functional barrier (4 kV rms, 8 kV impulse)."
- moved on the sheet: C217, C218, C219, C220, C221, C222, C223, C224, C225, C226, C227, C228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

Commit message: Resolve the independent PCM review of 033d8d8 (PCM-01..27): verify, classify, fix at the root (D-065..D-072)
Register gen/data/review_pcm.csv: 27 findings, each verified before a change - 21 Confirmed, 2 Firmware
Handled, 3 Improvement Recommended, 1 Not Applicable; 20 closed, 7 open with their closing path.

PV family (D-065, D-072): the 45 A port rating no longer clamps the inductor current in the near-unity
band (inductor rating 47.7 A there; 550/550 V 73.3 kW; rated power from 562 V); control model re-based on
the drawn boards with a published delivered-power envelope per product and direction; leg commutation
re-run on the drawn Jianghai capacitors (1374 V worst vs 1445 V); comparator common-mode term in every
trip band (window 67.9-80.5 A, the 1.10 margin rule missed by 0.58 A and left open; firmware OV derived
from the drawn band, 1034 V); one fan-supply contract; cold-start passive-power restriction modelled;
port A interface declared; aux pull-in and retry rules.

PCS-P125 (D-066, D-067): control study sim/pcs_control.py (PR current loop 1750 Hz, PM >= 48.7 deg to
SCR 5 with the passive damping branch, PLL, DC-link loop, grid forming, state machine); DC-link inventory
409.4 uF with bleeders, precharge rating and the 15 min label re-derived; upper-half limit in firmware;
P-Q-Vdc-Vac envelope (AC-02's 600 V full-load figure not reachable at a +15 % grid: owner's decision);
R_DS(on) acceptance rule for the six paralleled devices; DESAT string 3 -> 2 diodes (band 6.41-9.37 V);
fuse-contactor coordination bands and installation requirements; phase-current sensor frozen to Sinomags
STK-250HO/4 and the control-board ladders re-valued; Al2O3 pad text.

DAB-D60 (D-068): study vs drawn-board identity made explicit; short-circuit chain corrected (energy-
equivalent 0.99 x the assumed withstand; release block t_SC >= 2.22 us / E_SC >= 2.18 J); admitted map
follows the 1200 V deck envelope (900-950 V rows derated until a double-pulse test); zero/light-load policy;
0.41 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
Other:
- moved on the sheet: C201, C202, C203, C204, C205, C206, C207, C208, C209, C210, C211, C212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
