File: hardware/PV-PWR-4/sheets/05_ph2_power.kicad_sch (KiCad schematic)
At the start: 127 parts, among them J501 7461057, J502 7461057, J503 KF2EDGR-3.5-2P, J504 KF2EDGR-3.5-2P, P501 PAD AlN 1 mm (CUSTOM), P502 PAD AlN 1 mm (CUSTOM), P503 PAD AlN 1 mm (CUSTOM), P504 PAD AlN 1 mm (CUSTOM), P505 PAD AlN 1 mm (CUSTOM), P506 PAD AlN 1 mm (CUSTOM), P507 PAD AlN 1 mm (CUSTOM), P508 PAD AlN 1 mm (CUSTOM), Q501 SG2M040170HJ, Q502 SG2M040170HJ, Q503 SG2M040170HJ, Q504 SG2M040170HJ, Q505 SG2M040170HJ, Q506 SG2M040170HJ, Q507 SG2M040170HJ, Q508 SG2M040170HJ, Q509 PBSS5540X,135, Q510 PBSS5540X,135, Q511 PBSS5540X,135, Q512 PBSS5540X,135, T501 Gate-bias transformer per pha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, U501 SN6505BDBVR, U502 ATL431BIDBZR, U503 ATL431BIDBZR, U504 ATL431BIDBZR, U505 ATL431BIDBZR, U506 ATL431BIDBZR, U507 ATL431BIDBZR, U508 ATL431BIDBZR, U509 ATL431BIDBZR

Commit message: Board revisions PV-PWR A2 / PV-CTL A1, inverter filter magnetics, documentation refresh (D-056..D-058)
Boards (every build check passes)
- PV-PWR / PV-PWR-4 rev A2: seventh battery-side film capacitor on the three-phase board (closes the
  load-rejection overshoot), bleeder 8 x 73.2 k so the bank still discharges within its 10-minute label.
- PV-CTL rev A1: hardware over-current window 68.9-79.9 A, thresholds derived from each sensor's own
  reference; the board-to-board contract carries the four references on the former 24 V / 5 V pins.
- Records aligned (contract comments, architecture corrections, port-current bandwidth); the frozen
  platform's module BOMs are kept instead of being re-rolled from the cost-first thermal data.

Magnetics
- Inverter filter designed and verified: L1, L2 and the AC common-mode choke (design_pcs_*.json). The filter
  comes to 745 USD at catalogue prices and 611 USD at 5,000 units, against 207 / 167 in the study: the
  inverter's cost is provisional and its stage and filter are being re-optimised.
- PV inductor loss check made non-circular; hot-spot margin reported per build (PV-P100/110: -5.3 K, MG-17).

Results: PV-P75 952 USD at catalogue prices / 796 USD at 5,000 units; Megarevo comparison 2 better,
24 meet, 3 below, 5 not assessed. Documentation corrected for the revised boards (51 statements).
Everything is calculated or estimated; nothing is bench-validated.

Co-Authored-By: Claude Fable 5.1 <noreply@anthropic.com>
Parts:
- added C533: 2.2u 50V, symbol dcdc:C
- added R543: 10k, symbol dcdc:R
- C517: value 100n 50V -> 1n 50V
- C519: value 10u 16V -> 100n 50V; Package 1206 -> 0603
- C520: value 100n 50V -> 10u 16V; Package 0603 -> 1206
- C521: value 4.7u 50V -> 100n 50V; Domain GD_P2S1 -> LIVE; Package 1206 -> 0603
- C522, C525, C528, C531: value 10n 50V -> 4.7u 50V; Package 0603 -> 1206
- C523, C526, C529, C532: value 2.2u 50V -> 10n 50V; Package 0805 -> 0603
- C524: value 4.7u 50V -> 2.2u 50V; Domain GD_P2S2 -> GD_P2S1; Package 1206 -> 0805
- C527: value 4.7u 50V -> 2.2u 50V; Domain GD_P2S3 -> GD_P2S2; Package 1206 -> 0805
- C530: value 4.7u 50V -> 2.2u 50V; Domain GD_P2S4 -> GD_P2S3; Package 1206 -> 0805
- R514: value 10k -> 100R
- R515: Domain GD_P2S1 -> LIVE
- R516, R523, R530, R537: value 1k -> 10k
- R517, R524, R531, R538: value 77.7k -> 1k
- R518, R525, R532, R539: value 10.2k -> 77.7k
- R519, R526, R533, R540: value 4.7k -> 10.2k; Package 0805 -> 0603
- R520, R527, R534, R541: value 4.02k -> 4.7k; Package 0603 -> 0805
- R521, R528, R535, R542: value 10k -> 4.02k
- R522: Domain GD_P2S2 -> GD_P2S1
- R529: Domain GD_P2S3 -> GD_P2S2
- R536: Domain GD_P2S4 -> GD_P2S3
Connections:
- net +5V: now also C521.1; no longer C519.1
- net AGND: now also C519.2
- net BIAS_EN5: now also R515.1; no longer R514.1
- net COM_P2S1: now also R520.2, R521.1; no longer R519.2, R520.1
- net COM_P2S2: now also R527.2, R528.1; no longer R526.2, R527.1
- net COM_P2S3: now also R534.2, R535.1; no longer R533.2, R534.1
- net COM_P2S4: now also R541.2, R542.1; no longer R540.2, R541.1
- net CREF_PH2P2S1: now also R521.2, R522.1; no longer R520.2, R521.1
- net CREF_PH2P2S2: now also R528.2, R529.1; no longer R527.2, R528.1
- net CREF_PH2P2S3: now also R535.2, R536.1; no longer R534.2, R535.1
- net CREF_PH2P2S4: now also R542.2, R543.1; no longer R541.2, R542.1
- net GND: now also C521.2, R515.2; no longer C519.2, R514.2
- net NTC2: now also C518.1; no longer C517.1
- net NTC6: now also C519.1; no longer C518.1
- net RAW_PH2P2S1: now also C522.1, R516.1; no longer C521.1, R515.1
- net RAW_PH2P2S2: now also C525.1, R523.1; no longer C524.1, R522.1
- net RAW_PH2P2S3: now also C528.1, R530.1; no longer C527.1, R529.1
- net RAW_PH2P2S4: now also C531.1, R537.1; no longer C530.1, R536.1
- net RB_PH2P2S1: now also R516.2, R517.1; no longer R515.2, R516.1
- net RB_PH2P2S2: now also R523.2, R524.1; no longer R522.2, R523.1
- net RB_PH2P2S3: now also R530.2, R531.1; no longer R529.2, R530.1
- net RB_PH2P2S4: now also R537.2, R538.1; no longer R536.2, R537.1
- net RK_PH2P2S1: now also C523.1, R517.2; no longer C522.1, R516.2
- net RK_PH2P2S2: now also C526.1, R524.2; no longer C525.1, R523.2
- net RK_PH2P2S3: now also C529.1, R531.2; no longer C528.1, R530.2
- net RK_PH2P2S4: now also C532.1, R538.2; no longer C531.1, R537.2
- net RREF_PH2P2S1: now also C523.2, R518.2, R519.1; no longer C522.2, R517.2, R518.1
- net RREF_PH2P2S2: now also C526.2, R525.2, R526.1; no longer C525.2, R524.2, R525.1
- net RREF_PH2P2S3: now also C529.2, R532.2, R533.1; no longer C528.2, R531.2, R532.1
- net RREF_PH2P2S4: now also C532.2, R539.2, R540.1; no longer C531.2, R538.2, R539.1
- net VDD_P2S1: now also C524.1, R518.1, R520.1; no longer C523.1, R517.1, R519.1
- net VDD_P2S2: now also C527.1, R525.1, R527.1; no longer C526.1, R524.1, R526.1
- net VDD_P2S3: now also C530.1, R532.1, R534.1; no longer C529.1, R531.1, R533.1
- net VDD_P2S4: now also R539.1, R541.1, C533.1; no longer C532.1, R538.1, R540.1
- net VEE_P2S1: now also C522.2, C524.2, R519.2, R522.2; no longer C521.2, C523.2, R518.2, R521.2
- net VEE_P2S2: now also C525.2, C527.2, R526.2, R529.2; no longer C524.2, C526.2, R525.2, R528.2
- net VEE_P2S3: now also C528.2, C530.2, R533.2, R536.2; no longer C527.2, C529.2, R532.2, R535.2
- net VEE_P2S4: now also C531.2, R540.2, C533.2, R543.2; no longer C530.2, C532.2, R539.2, R542.2
- net IL2R_S: now reaches CS501.4 (UREF)
- net IL2R_S: now also R514.1
- new net IL2R: C517.1, R514.2
- no-connect marks 2 -> 1
Other:
- note added: "2 x FCSA3DS456 (45 uF) on A_BUS+ and 2 on B_BUS+, at this phase's legs: the banks of all phases form the port A / port B DC links (8 / 8 x 45 uF). Bleeders: one string per port on the port sheets."
- note added: "Lead A from SW_A2 passes the STK-HO/A 75 U-primary (pins 6-9 in, 10-13 out: + = SW_A -> SW_B) to stud L_A2; lead B on stud SW_B2. IL2 = 2.5 V + 10.667 mV/A (Vref 2.48-2.52 V), 0.5-4.5 V over +/-187.5 A; 100R + 1 nF at the source. IL2R = the sensor's own Uref (pin 4), 100R + 1 nF: PV-CTL references its trip window to it. Primary at the switch node: functional barrier (4 kV rms, 8 kV impulse)."
- note removed: "2 x FCSA3DS456 (45 uF) on A_BUS+ and 2 on B_BUS+, at this phase's legs: the banks of all phases form the port A / port B DC links. Bleeders: one string per port on the port sheets."
- note removed: "Lead A from SW_A2 passes the STK-HO/A 75 U-primary (pins 6-9 in, 10-13 out: + = SW_A -> SW_B) to stud L_A2; lead B on stud SW_B2. IL2 = 2.5 V + 10.667 mV/A (Vref 2.48-2.52 V), 0.5-4.5 V over +/-187.5 A; 100R + 1 nF at the source. Primary at the switch node: functional barrier (4 kV rms, 8 kV impulse)."
- moved on the sheet: C517, C518, C519, C520, C521, C522, C523, C524, C525, C526, C527, C528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

Commit message: Resolve the independent PCM review of 033d8d8 (PCM-01..27): verify, classify, fix at the root (D-065..D-072)
Register gen/data/review_pcm.csv: 27 findings, each verified before a change - 21 Confirmed, 2 Firmware
Handled, 3 Improvement Recommended, 1 Not Applicable; 20 closed, 7 open with their closing path.

PV family (D-065, D-072): the 45 A port rating no longer clamps the inductor current in the near-unity
band (inductor rating 47.7 A there; 550/550 V 73.3 kW; rated power from 562 V); control model re-based on
the drawn boards with a published delivered-power envelope per product and direction; leg commutation
re-run on the drawn Jianghai capacitors (1374 V worst vs 1445 V); comparator common-mode term in every
trip band (window 67.9-80.5 A, the 1.10 margin rule missed by 0.58 A and left open; firmware OV derived
from the drawn band, 1034 V); one fan-supply contract; cold-start passive-power restriction modelled;
port A interface declared; aux pull-in and retry rules.

PCS-P125 (D-066, D-067): control study sim/pcs_control.py (PR current loop 1750 Hz, PM >= 48.7 deg to
SCR 5 with the passive damping branch, PLL, DC-link loop, grid forming, state machine); DC-link inventory
409.4 uF with bleeders, precharge rating and the 15 min label re-derived; upper-half limit in firmware;
P-Q-Vdc-Vac envelope (AC-02's 600 V full-load figure not reachable at a +15 % grid: owner's decision);
R_DS(on) acceptance rule for the six paralleled devices; DESAT string 3 -> 2 diodes (band 6.41-9.37 V);
fuse-contactor coordination bands and installation requirements; phase-current sensor frozen to Sinomags
STK-250HO/4 and the control-board ladders re-valued; Al2O3 pad text.

DAB-D60 (D-068): study vs drawn-board identity made explicit; short-circuit chain corrected (energy-
equivalent 0.99 x the assumed withstand; release block t_SC >= 2.22 us / E_SC >= 2.18 J); admitted map
follows the 1200 V deck envelope (900-950 V rows derated until a double-pulse test); zero/light-load policy;
0.41 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
Other:
- moved on the sheet: C501, C502, C503, C504, C505, C506, C507, C508, C509, C510, C511, C512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
