File: hardware/PV-PWR-4/sheets/08_ph3_power.kicad_sch (KiCad schematic)
At the start: 127 parts, among them J801 7461057, J802 7461057, J803 KF2EDGR-3.5-2P, J804 KF2EDGR-3.5-2P, P801 PAD AlN 1 mm (CUSTOM), P802 PAD AlN 1 mm (CUSTOM), P803 PAD AlN 1 mm (CUSTOM), P804 PAD AlN 1 mm (CUSTOM), P805 PAD AlN 1 mm (CUSTOM), P806 PAD AlN 1 mm (CUSTOM), P807 PAD AlN 1 mm (CUSTOM), P808 PAD AlN 1 mm (CUSTOM), Q801 SG2M040170HJ, Q802 SG2M040170HJ, Q803 SG2M040170HJ, Q804 SG2M040170HJ, Q805 SG2M040170HJ, Q806 SG2M040170HJ, Q807 SG2M040170HJ, Q808 SG2M040170HJ, Q809 PBSS5540X,135, Q810 PBSS5540X,135, Q811 PBSS5540X,135, Q812 PBSS5540X,135, T801 Gate-bias transformer per pha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, U801 SN6505BDBVR, U802 ATL431BIDBZR, U803 ATL431BIDBZR, U804 ATL431BIDBZR, U805 ATL431BIDBZR, U806 ATL431BIDBZR, U807 ATL431BIDBZR, U808 ATL431BIDBZR, U809 ATL431BIDBZR

Commit message: Board revisions PV-PWR A2 / PV-CTL A1, inverter filter magnetics, documentation refresh (D-056..D-058)
Boards (every build check passes)
- PV-PWR / PV-PWR-4 rev A2: seventh battery-side film capacitor on the three-phase board (closes the
  load-rejection overshoot), bleeder 8 x 73.2 k so the bank still discharges within its 10-minute label.
- PV-CTL rev A1: hardware over-current window 68.9-79.9 A, thresholds derived from each sensor's own
  reference; the board-to-board contract carries the four references on the former 24 V / 5 V pins.
- Records aligned (contract comments, architecture corrections, port-current bandwidth); the frozen
  platform's module BOMs are kept instead of being re-rolled from the cost-first thermal data.

Magnetics
- Inverter filter designed and verified: L1, L2 and the AC common-mode choke (design_pcs_*.json). The filter
  comes to 745 USD at catalogue prices and 611 USD at 5,000 units, against 207 / 167 in the study: the
  inverter's cost is provisional and its stage and filter are being re-optimised.
- PV inductor loss check made non-circular; hot-spot margin reported per build (PV-P100/110: -5.3 K, MG-17).

Results: PV-P75 952 USD at catalogue prices / 796 USD at 5,000 units; Megarevo comparison 2 better,
24 meet, 3 below, 5 not assessed. Documentation corrected for the revised boards (51 statements).
Everything is calculated or estimated; nothing is bench-validated.

Co-Authored-By: Claude Fable 5.1 <noreply@anthropic.com>
Parts:
- added C833: 2.2u 50V, symbol dcdc:C
- added R843: 10k, symbol dcdc:R
- C817: value 100n 50V -> 1n 50V
- C819: value 10u 16V -> 100n 50V; Package 1206 -> 0603
- C820: value 100n 50V -> 10u 16V; Package 0603 -> 1206
- C821: value 4.7u 50V -> 100n 50V; Domain GD_P3S1 -> LIVE; Package 1206 -> 0603
- C822, C825, C828, C831: value 10n 50V -> 4.7u 50V; Package 0603 -> 1206
- C823, C826, C829, C832: value 2.2u 50V -> 10n 50V; Package 0805 -> 0603
- C824: value 4.7u 50V -> 2.2u 50V; Domain GD_P3S2 -> GD_P3S1; Package 1206 -> 0805
- C827: value 4.7u 50V -> 2.2u 50V; Domain GD_P3S3 -> GD_P3S2; Package 1206 -> 0805
- C830: value 4.7u 50V -> 2.2u 50V; Domain GD_P3S4 -> GD_P3S3; Package 1206 -> 0805
- R814: value 10k -> 100R
- R815: Domain GD_P3S1 -> LIVE
- R816, R823, R830, R837: value 1k -> 10k
- R817, R824, R831, R838: value 77.7k -> 1k
- R818, R825, R832, R839: value 10.2k -> 77.7k
- R819, R826, R833, R840: value 4.7k -> 10.2k; Package 0805 -> 0603
- R820, R827, R834, R841: value 4.02k -> 4.7k; Package 0603 -> 0805
- R821, R828, R835, R842: value 10k -> 4.02k
- R822: Domain GD_P3S2 -> GD_P3S1
- R829: Domain GD_P3S3 -> GD_P3S2
- R836: Domain GD_P3S4 -> GD_P3S3
Connections:
- net +5V_GD: now also C821.1; no longer C819.1
- net AGND: now also C819.2
- net BIAS_EN5G: now also R815.1; no longer R814.1
- net COM_P3S1: now also R820.2, R821.1; no longer R819.2, R820.1
- net COM_P3S2: now also R827.2, R828.1; no longer R826.2, R827.1
- net COM_P3S3: now also R834.2, R835.1; no longer R833.2, R834.1
- net COM_P3S4: now also R841.2, R842.1; no longer R840.2, R841.1
- net CREF_PH3P3S1: now also R821.2, R822.1; no longer R820.2, R821.1
- net CREF_PH3P3S2: now also R828.2, R829.1; no longer R827.2, R828.1
- net CREF_PH3P3S3: now also R835.2, R836.1; no longer R834.2, R835.1
- net CREF_PH3P3S4: now also R842.2, R843.1; no longer R841.2, R842.1
- net GND: now also C821.2, R815.2; no longer C819.2, R814.2
- net NTC3: now also C818.1; no longer C817.1
- net NTC7: now also C819.1; no longer C818.1
- net RAW_PH3P3S1: now also C822.1, R816.1; no longer C821.1, R815.1
- net RAW_PH3P3S2: now also C825.1, R823.1; no longer C824.1, R822.1
- net RAW_PH3P3S3: now also C828.1, R830.1; no longer C827.1, R829.1
- net RAW_PH3P3S4: now also C831.1, R837.1; no longer C830.1, R836.1
- net RB_PH3P3S1: now also R816.2, R817.1; no longer R815.2, R816.1
- net RB_PH3P3S2: now also R823.2, R824.1; no longer R822.2, R823.1
- net RB_PH3P3S3: now also R830.2, R831.1; no longer R829.2, R830.1
- net RB_PH3P3S4: now also R837.2, R838.1; no longer R836.2, R837.1
- net RK_PH3P3S1: now also C823.1, R817.2; no longer C822.1, R816.2
- net RK_PH3P3S2: now also C826.1, R824.2; no longer C825.1, R823.2
- net RK_PH3P3S3: now also C829.1, R831.2; no longer C828.1, R830.2
- net RK_PH3P3S4: now also C832.1, R838.2; no longer C831.1, R837.2
- net RREF_PH3P3S1: now also C823.2, R818.2, R819.1; no longer C822.2, R817.2, R818.1
- net RREF_PH3P3S2: now also C826.2, R825.2, R826.1; no longer C825.2, R824.2, R825.1
- net RREF_PH3P3S3: now also C829.2, R832.2, R833.1; no longer C828.2, R831.2, R832.1
- net RREF_PH3P3S4: now also C832.2, R839.2, R840.1; no longer C831.2, R838.2, R839.1
- net VDD_P3S1: now also C824.1, R818.1, R820.1; no longer C823.1, R817.1, R819.1
- net VDD_P3S2: now also C827.1, R825.1, R827.1; no longer C826.1, R824.1, R826.1
- net VDD_P3S3: now also C830.1, R832.1, R834.1; no longer C829.1, R831.1, R833.1
- net VDD_P3S4: now also R839.1, R841.1, C833.1; no longer C832.1, R838.1, R840.1
- net VEE_P3S1: now also C822.2, C824.2, R819.2, R822.2; no longer C821.2, C823.2, R818.2, R821.2
- net VEE_P3S2: now also C825.2, C827.2, R826.2, R829.2; no longer C824.2, C826.2, R825.2, R828.2
- net VEE_P3S3: now also C828.2, C830.2, R833.2, R836.2; no longer C827.2, C829.2, R832.2, R835.2
- net VEE_P3S4: now also C831.2, R840.2, C833.2, R843.2; no longer C830.2, C832.2, R839.2, R842.2
- net IL3R_S: now reaches CS801.4 (UREF)
- net IL3R_S: now also R814.1
- new net IL3R: C817.1, R814.2
- no-connect marks 2 -> 1
Other:
- note added: "2 x FCSA3DS456 (45 uF) on A_BUS+ and 2 on B_BUS+, at this phase's legs: the banks of all phases form the port A / port B DC links (8 / 8 x 45 uF). Bleeders: one string per port on the port sheets."
- note added: "Lead A from SW_A3 passes the STK-HO/A 75 U-primary (pins 6-9 in, 10-13 out: + = SW_A -> SW_B) to stud L_A3; lead B on stud SW_B3. IL3 = 2.5 V + 10.667 mV/A (Vref 2.48-2.52 V), 0.5-4.5 V over +/-187.5 A; 100R + 1 nF at the source. IL3R = the sensor's own Uref (pin 4), 100R + 1 nF: PV-CTL references its trip window to it. Primary at the switch node: functional barrier (4 kV rms, 8 kV impulse)."
- note removed: "2 x FCSA3DS456 (45 uF) on A_BUS+ and 2 on B_BUS+, at this phase's legs: the banks of all phases form the port A / port B DC links. Bleeders: one string per port on the port sheets."
- note removed: "Lead A from SW_A3 passes the STK-HO/A 75 U-primary (pins 6-9 in, 10-13 out: + = SW_A -> SW_B) to stud L_A3; lead B on stud SW_B3. IL3 = 2.5 V + 10.667 mV/A (Vref 2.48-2.52 V), 0.5-4.5 V over +/-187.5 A; 100R + 1 nF at the source. Primary at the switch node: functional barrier (4 kV rms, 8 kV impulse)."
- moved on the sheet: C817, C818, C819, C820, C821, C822, C823, C824, C825, C826, C827, C828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

Commit message: Resolve the independent PCM review of 033d8d8 (PCM-01..27): verify, classify, fix at the root (D-065..D-072)
Register gen/data/review_pcm.csv: 27 findings, each verified before a change - 21 Confirmed, 2 Firmware
Handled, 3 Improvement Recommended, 1 Not Applicable; 20 closed, 7 open with their closing path.

PV family (D-065, D-072): the 45 A port rating no longer clamps the inductor current in the near-unity
band (inductor rating 47.7 A there; 550/550 V 73.3 kW; rated power from 562 V); control model re-based on
the drawn boards with a published delivered-power envelope per product and direction; leg commutation
re-run on the drawn Jianghai capacitors (1374 V worst vs 1445 V); comparator common-mode term in every
trip band (window 67.9-80.5 A, the 1.10 margin rule missed by 0.58 A and left open; firmware OV derived
from the drawn band, 1034 V); one fan-supply contract; cold-start passive-power restriction modelled;
port A interface declared; aux pull-in and retry rules.

PCS-P125 (D-066, D-067): control study sim/pcs_control.py (PR current loop 1750 Hz, PM >= 48.7 deg to
SCR 5 with the passive damping branch, PLL, DC-link loop, grid forming, state machine); DC-link inventory
409.4 uF with bleeders, precharge rating and the 15 min label re-derived; upper-half limit in firmware;
P-Q-Vdc-Vac envelope (AC-02's 600 V full-load figure not reachable at a +15 % grid: owner's decision);
R_DS(on) acceptance rule for the six paralleled devices; DESAT string 3 -> 2 diodes (band 6.41-9.37 V);
fuse-contactor coordination bands and installation requirements; phase-current sensor frozen to Sinomags
STK-250HO/4 and the control-board ladders re-valued; Al2O3 pad text.

DAB-D60 (D-068): study vs drawn-board identity made explicit; short-circuit chain corrected (energy-
equivalent 0.99 x the assumed withstand; release block t_SC >= 2.22 us / E_SC >= 2.18 J); admitted map
follows the 1200 V deck envelope (900-950 V rows derated until a double-pulse test); zero/light-load policy;
0.41 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
Other:
- moved on the sheet: C801, C802, C803, C804, C805, C806, C807, C808, C809, C810, C811, C812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
