File: hardware/PV-PWR-4/sheets/11_ph4_power.kicad_sch (KiCad schematic)
At the start: 127 parts, among them J1101 7461057, J1102 7461057, J1103 KF2EDGR-3.5-2P, J1104 KF2EDGR-3.5-2P, P1101 PAD AlN 1 mm (CUSTOM), P1102 PAD AlN 1 mm (CUSTOM), P1103 PAD AlN 1 mm (CUSTOM), P1104 PAD AlN 1 mm (CUSTOM), P1105 PAD AlN 1 mm (CUSTOM), P1106 PAD AlN 1 mm (CUSTOM), P1107 PAD AlN 1 mm (CUSTOM), P1108 PAD AlN 1 mm (CUSTOM), Q1101 SG2M040170HJ, Q1102 SG2M040170HJ, Q1103 SG2M040170HJ, Q1104 SG2M040170HJ, Q1105 SG2M040170HJ, Q1106 SG2M040170HJ, Q1107 SG2M040170HJ, Q1108 SG2M040170HJ, Q1109 PBSS5540X,135, Q1110 PBSS5540X,135, Q1111 PBSS5540X,135, Q1112 PBSS5540X,135, T1101 Gate-bias transformer per pha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, U1101 SN6505BDBVR, U1102 ATL431BIDBZR, U1103 ATL431BIDBZR, U1104 ATL431BIDBZR, U1105 ATL431BIDBZR, U1106 ATL431BIDBZR, U1107 ATL431BIDBZR, U1108 ATL431BIDBZR, U1109 ATL431BIDBZR

Commit message: Board revisions PV-PWR A2 / PV-CTL A1, inverter filter magnetics, documentation refresh (D-056..D-058)
Boards (every build check passes)
- PV-PWR / PV-PWR-4 rev A2: seventh battery-side film capacitor on the three-phase board (closes the
  load-rejection overshoot), bleeder 8 x 73.2 k so the bank still discharges within its 10-minute label.
- PV-CTL rev A1: hardware over-current window 68.9-79.9 A, thresholds derived from each sensor's own
  reference; the board-to-board contract carries the four references on the former 24 V / 5 V pins.
- Records aligned (contract comments, architecture corrections, port-current bandwidth); the frozen
  platform's module BOMs are kept instead of being re-rolled from the cost-first thermal data.

Magnetics
- Inverter filter designed and verified: L1, L2 and the AC common-mode choke (design_pcs_*.json). The filter
  comes to 745 USD at catalogue prices and 611 USD at 5,000 units, against 207 / 167 in the study: the
  inverter's cost is provisional and its stage and filter are being re-optimised.
- PV inductor loss check made non-circular; hot-spot margin reported per build (PV-P100/110: -5.3 K, MG-17).

Results: PV-P75 952 USD at catalogue prices / 796 USD at 5,000 units; Megarevo comparison 2 better,
24 meet, 3 below, 5 not assessed. Documentation corrected for the revised boards (51 statements).
Everything is calculated or estimated; nothing is bench-validated.

Co-Authored-By: Claude Fable 5.1 <noreply@anthropic.com>
Parts:
- added C1133: 2.2u 50V, symbol dcdc:C
- added R1143: 10k, symbol dcdc:R
- C1117: value 100n 50V -> 1n 50V
- C1119: value 10u 16V -> 100n 50V; Package 1206 -> 0603
- C1120: value 100n 50V -> 10u 16V; Package 0603 -> 1206
- C1121: value 4.7u 50V -> 100n 50V; Domain GD_P4S1 -> LIVE; Package 1206 -> 0603
- C1122, C1125, C1128, C1131: value 10n 50V -> 4.7u 50V; Package 0603 -> 1206
- C1123, C1126, C1129, C1132: value 2.2u 50V -> 10n 50V; Package 0805 -> 0603
- C1124: value 4.7u 50V -> 2.2u 50V; Domain GD_P4S2 -> GD_P4S1; Package 1206 -> 0805
- C1127: value 4.7u 50V -> 2.2u 50V; Domain GD_P4S3 -> GD_P4S2; Package 1206 -> 0805
- C1130: value 4.7u 50V -> 2.2u 50V; Domain GD_P4S4 -> GD_P4S3; Package 1206 -> 0805
- R1114: value 10k -> 100R
- R1115: Domain GD_P4S1 -> LIVE
- R1116, R1123, R1130, R1137: value 1k -> 10k
- R1117, R1124, R1131, R1138: value 77.7k -> 1k
- R1118, R1125, R1132, R1139: value 10.2k -> 77.7k
- R1119, R1126, R1133, R1140: value 4.7k -> 10.2k; Package 0805 -> 0603
- R1120, R1127, R1134, R1141: value 4.02k -> 4.7k; Package 0603 -> 0805
- R1121, R1128, R1135, R1142: value 10k -> 4.02k
- R1122: Domain GD_P4S2 -> GD_P4S1
- R1129: Domain GD_P4S3 -> GD_P4S2
- R1136: Domain GD_P4S4 -> GD_P4S3
Connections:
- net +5V_GD: now also C1121.1; no longer C1119.1
- net AGND: now also C1119.2
- net BIAS_EN5G: now also R1115.1; no longer R1114.1
- net COM_P4S1: now also R1120.2, R1121.1; no longer R1119.2, R1120.1
- net COM_P4S2: now also R1127.2, R1128.1; no longer R1126.2, R1127.1
- net COM_P4S3: now also R1134.2, R1135.1; no longer R1133.2, R1134.1
- net COM_P4S4: now also R1141.2, R1142.1; no longer R1140.2, R1141.1
- net CREF_PH4P4S1: now also R1121.2, R1122.1; no longer R1120.2, R1121.1
- net CREF_PH4P4S2: now also R1128.2, R1129.1; no longer R1127.2, R1128.1
- net CREF_PH4P4S3: now also R1135.2, R1136.1; no longer R1134.2, R1135.1
- net CREF_PH4P4S4: now also R1142.2, R1143.1; no longer R1141.2, R1142.1
- net GND: now also C1121.2, R1115.2; no longer C1119.2, R1114.2
- net NTC4: now also C1118.1; no longer C1117.1
- net NTC8: now also C1119.1; no longer C1118.1
- net RAW_PH4P4S1: now also C1122.1, R1116.1; no longer C1121.1, R1115.1
- net RAW_PH4P4S2: now also C1125.1, R1123.1; no longer C1124.1, R1122.1
- net RAW_PH4P4S3: now also C1128.1, R1130.1; no longer C1127.1, R1129.1
- net RAW_PH4P4S4: now also C1131.1, R1137.1; no longer C1130.1, R1136.1
- net RB_PH4P4S1: now also R1116.2, R1117.1; no longer R1115.2, R1116.1
- net RB_PH4P4S2: now also R1123.2, R1124.1; no longer R1122.2, R1123.1
- net RB_PH4P4S3: now also R1130.2, R1131.1; no longer R1129.2, R1130.1
- net RB_PH4P4S4: now also R1137.2, R1138.1; no longer R1136.2, R1137.1
- net RK_PH4P4S1: now also C1123.1, R1117.2; no longer C1122.1, R1116.2
- net RK_PH4P4S2: now also C1126.1, R1124.2; no longer C1125.1, R1123.2
- net RK_PH4P4S3: now also C1129.1, R1131.2; no longer C1128.1, R1130.2
- net RK_PH4P4S4: now also C1132.1, R1138.2; no longer C1131.1, R1137.2
- net RREF_PH4P4S1: now also C1123.2, R1118.2, R1119.1; no longer C1122.2, R1117.2, R1118.1
- net RREF_PH4P4S2: now also C1126.2, R1125.2, R1126.1; no longer C1125.2, R1124.2, R1125.1
- net RREF_PH4P4S3: now also C1129.2, R1132.2, R1133.1; no longer C1128.2, R1131.2, R1132.1
- net RREF_PH4P4S4: now also C1132.2, R1139.2, R1140.1; no longer C1131.2, R1138.2, R1139.1
- net VDD_P4S1: now also C1124.1, R1118.1, R1120.1; no longer C1123.1, R1117.1, R1119.1
- net VDD_P4S2: now also C1127.1, R1125.1, R1127.1; no longer C1126.1, R1124.1, R1126.1
- net VDD_P4S3: now also C1130.1, R1132.1, R1134.1; no longer C1129.1, R1131.1, R1133.1
- net VDD_P4S4: now also R1139.1, R1141.1, C1133.1; no longer C1132.1, R1138.1, R1140.1
- net VEE_P4S1: now also C1122.2, C1124.2, R1119.2, R1122.2; no longer C1121.2, C1123.2, R1118.2, R1121.2
- net VEE_P4S2: now also C1125.2, C1127.2, R1126.2, R1129.2; no longer C1124.2, C1126.2, R1125.2, R1128.2
- net VEE_P4S3: now also C1128.2, C1130.2, R1133.2, R1136.2; no longer C1127.2, C1129.2, R1132.2, R1135.2
- net VEE_P4S4: now also C1131.2, R1140.2, C1133.2, R1143.2; no longer C1130.2, C1132.2, R1139.2, R1142.2
- net IL4R_S: now reaches CS1101.4 (UREF)
- net IL4R_S: now also R1114.1
- new net IL4R: C1117.1, R1114.2
- no-connect marks 2 -> 1
Other:
- note added: "2 x FCSA3DS456 (45 uF) on A_BUS+ and 2 on B_BUS+, at this phase's legs: the banks of all phases form the port A / port B DC links (8 / 8 x 45 uF). Bleeders: one string per port on the port sheets."
- note added: "Lead A from SW_A4 passes the STK-HO/A 75 U-primary (pins 6-9 in, 10-13 out: + = SW_A -> SW_B) to stud L_A4; lead B on stud SW_B4. IL4 = 2.5 V + 10.667 mV/A (Vref 2.48-2.52 V), 0.5-4.5 V over +/-187.5 A; 100R + 1 nF at the source. IL4R = the sensor's own Uref (pin 4), 100R + 1 nF: PV-CTL references its trip window to it. Primary at the switch node: functional barrier (4 kV rms, 8 kV impulse)."
- note removed: "2 x FCSA3DS456 (45 uF) on A_BUS+ and 2 on B_BUS+, at this phase's legs: the banks of all phases form the port A / port B DC links. Bleeders: one string per port on the port sheets."
- note removed: "Lead A from SW_A4 passes the STK-HO/A 75 U-primary (pins 6-9 in, 10-13 out: + = SW_A -> SW_B) to stud L_A4; lead B on stud SW_B4. IL4 = 2.5 V + 10.667 mV/A (Vref 2.48-2.52 V), 0.5-4.5 V over +/-187.5 A; 100R + 1 nF at the source. Primary at the switch node: functional barrier (4 kV rms, 8 kV impulse)."
- moved on the sheet: C1117, C1118, C1119, C1120, C1121, C1122, C1123, C1124, C1125, C1126, C1127, C1128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

Commit message: Resolve the independent PCM review of 033d8d8 (PCM-01..27): verify, classify, fix at the root (D-065..D-072)
Register gen/data/review_pcm.csv: 27 findings, each verified before a change - 21 Confirmed, 2 Firmware
Handled, 3 Improvement Recommended, 1 Not Applicable; 20 closed, 7 open with their closing path.

PV family (D-065, D-072): the 45 A port rating no longer clamps the inductor current in the near-unity
band (inductor rating 47.7 A there; 550/550 V 73.3 kW; rated power from 562 V); control model re-based on
the drawn boards with a published delivered-power envelope per product and direction; leg commutation
re-run on the drawn Jianghai capacitors (1374 V worst vs 1445 V); comparator common-mode term in every
trip band (window 67.9-80.5 A, the 1.10 margin rule missed by 0.58 A and left open; firmware OV derived
from the drawn band, 1034 V); one fan-supply contract; cold-start passive-power restriction modelled;
port A interface declared; aux pull-in and retry rules.

PCS-P125 (D-066, D-067): control study sim/pcs_control.py (PR current loop 1750 Hz, PM >= 48.7 deg to
SCR 5 with the passive damping branch, PLL, DC-link loop, grid forming, state machine); DC-link inventory
409.4 uF with bleeders, precharge rating and the 15 min label re-derived; upper-half limit in firmware;
P-Q-Vdc-Vac envelope (AC-02's 600 V full-load figure not reachable at a +15 % grid: owner's decision);
R_DS(on) acceptance rule for the six paralleled devices; DESAT string 3 -> 2 diodes (band 6.41-9.37 V);
fuse-contactor coordination bands and installation requirements; phase-current sensor frozen to Sinomags
STK-250HO/4 and the control-board ladders re-valued; Al2O3 pad text.

DAB-D60 (D-068): study vs drawn-board identity made explicit; short-circuit chain corrected (energy-
equivalent 0.99 x the assumed withstand; release block t_SC >= 2.22 us / E_SC >= 2.18 J); admitted map
follows the 1200 V deck envelope (900-950 V rows derated until a double-pulse test); zero/light-load policy;
0.41 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
Other:
- moved on the sheet: C1101, C1102, C1103, C1104, C1105, C1106, C1107, C1108, C1109, C1110, C1111, C1112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
