File: hardware/PV-PWR-4/sheets/14_leanA_power.kicad_sch (KiCad schematic)
At the start: 111 parts, among them K1601 HFE82V-300C/1000-24-H-C5-1, Q1601 PMV30ENEAR, Q1602 BSS138BK, Q1603 IRFR9214TRPbF, U1401 CNY65B, U1501 REF3030EAIDBZR, U1502 OPA2388IDR, U1503 TLV3502AIDCNR, U1504 SN74LVC1G32DBVR, U1505 TLV3502AIDCNR, U1506 SN74LVC1G32DBVR, U1507 OPA2388IDR, U1508 OPA2388IDR, U1509 TLV3502AIDCNR, U1601 SN74LVC1G11DBVR, U1602 SN74LVC1G11DBVR, U1603 SN74LVC1G32DBVR, X1401 006710340, X1402 006710340, X1403 006710340, X1404 006710340

Commit message: Board revisions PV-PWR A2 / PV-CTL A1, inverter filter magnetics, documentation refresh (D-056..D-058)
Boards (every build check passes)
- PV-PWR / PV-PWR-4 rev A2: seventh battery-side film capacitor on the three-phase board (closes the
  load-rejection overshoot), bleeder 8 x 73.2 k so the bank still discharges within its 10-minute label.
- PV-CTL rev A1: hardware over-current window 68.9-79.9 A, thresholds derived from each sensor's own
  reference; the board-to-board contract carries the four references on the former 24 V / 5 V pins.
- Records aligned (contract comments, architecture corrections, port-current bandwidth); the frozen
  platform's module BOMs are kept instead of being re-rolled from the cost-first thermal data.

Magnetics
- Inverter filter designed and verified: L1, L2 and the AC common-mode choke (design_pcs_*.json). The filter
  comes to 745 USD at catalogue prices and 611 USD at 5,000 units, against 207 / 167 in the study: the
  inverter's cost is provisional and its stage and filter are being re-optimised.
- PV inductor loss check made non-circular; hot-spot margin reported per build (PV-P100/110: -5.3 K, MG-17).

Results: PV-P75 952 USD at catalogue prices / 796 USD at 5,000 units; Megarevo comparison 2 better,
24 meet, 3 below, 5 not assessed. Documentation corrected for the revised boards (51 statements).
Everything is calculated or estimated; nothing is bench-validated.

Co-Authored-By: Claude Fable 5.1 <noreply@anthropic.com>
Parts:
- R1610, R1611, R1612, R1613, R1614, R1615, R1616, R1617: value 82.5k -> 73.2k
Changed lines of the file:
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@@
 	(title_block
 		(title "PV-PWR-4 power board - Port A power path (pv)")
-		(date "2026-10-04")
-		(rev "A1")
+		(date "2026-10-05")
+		(rev "A2")
 		(comment 1 "Live board referenced to BUS-; gate islands functional; SELV winding reinforced; HV-PE basic")
 		(comment 2 "Schematics authored by Chinmoy Bhuyan")
@@
 			)
 		)
-		(property "Value" "82.5k"
+		(property "Value" "73.2k"
 			(at 55.88 192.916 90)
 			(show_name no)
@@
 			)
 		)
-		(property "Description" "Resistor 82.5k 1% 1210 HV thick film, >= 200 V working"
+		(property "Description" "Resistor 73.2k 1% 1210 HV thick film, >= 200 V working"
 			(at 55.88 190.5 0)
 			(hide yes)
@@
 			)
 		)
-		(property "Value" "82.5k"
+		(property "Value" "73.2k"
 			(at 457.2 172.596 90)
 			(show_name no)
@@
 			)
 		)
-		(property "Description" "Resistor 82.5k 1% 1210 HV thick film, >= 200 V working"
+		(property "Description" "Resistor 73.2k 1% 1210 HV thick film, >= 200 V working"
 			(at 457.2 170.18 0)
 			(hide yes)
@@
 			)
 		)
-		(property "Value" "82.5k"
+		(property "Value" "73.2k"
 			(at 566.42 172.596 90)
 			(show_name no)
@@
 			)
 		)
-		(property "Description" "Resistor 82.5k 1% 1210 HV thick film, >= 200 V working"
+		(property "Description" "Resistor 73.2k 1% 1210 HV thick film, >= 200 V working"
 			(at 566.42 170.18 0)
 			(hide yes)
@@
 			)
 		)
-		(property "Value" "82.5k"
+		(property "Value" "73.2k"
 			(at 27.94 192.916 90)
 			(show_name no)
@@
 			)
 		)
-		(property "Description" "Resistor 82.5k 1% 1210 HV thick film, >= 200 V working"
+		(property "Description" "Resistor 73.2k 1% 1210 HV thick film, >= 200 V working"
 			(at 27.94 190.5 0)
 			(hide yes)
@@
 			)
 		)
-		(property "Value" "82.5k"
+		(property "Value" "73.2k"
 			(at 510.54 172.596 90)
 			(show_name no)
@@
 			)
 		)
-		(property "Description" "Resistor 82.5k 1% 1210 HV thick film, >= 200 V working"
+		(property "Description" "Resistor 73.2k 1% 1210 HV thick film, >= 200 V working"
 			(at 510.54 170.18 0)
 			(hide yes)
@@
 			)
 		)
-		(property "Value" "82.5k"
+		(property "Value" "73.2k"
 			(at 482.6 172.596 90)
 			(show_name no)
@@
 			)
 		)
-		(property "Description" "Resistor 82.5k 1% 1210 HV thick film, >= 200 V working"
+		(property "Description" "Resistor 73.2k 1% 1210 HV thick film, >= 200 V working"
 			(at 482.6 170.18 0)
 			(hide yes)
@@
 			)
 		)
-		(property "Value" "82.5k"
+		(property "Value" "73.2k"
 			(at 429.26 172.596 90)
 			(show_name no)
@@
 			)
 		)
-		(property "Description" "Resistor 82.5k 1% 1210 HV thick film, >= 200 V working"
+		(property "Description" "Resistor 73.2k 1% 1210 HV thick film, >= 200 V working"
 			(at 429.26 170.18 0)
 			(hide yes)
@@
 			)
 		)
-		(property "Value" "82.5k"
+		(property "Value" "73.2k"
 			(at 538.48 172.596 90)
 			(show_name no)
@@
 			)
 		)
-		(property "Description" "Resistor 82.5k 1% 1210 HV thick film, >= 200 V working"
+		(property "Description" "Resistor 73.2k 1% 1210 HV thick film, >= 200 V working"
 			(at 538.48 170.18 0)
 			(hide yes)

Commit message: Resolve the independent PCM review of 033d8d8 (PCM-01..27): verify, classify, fix at the root (D-065..D-072)
Register gen/data/review_pcm.csv: 27 findings, each verified before a change - 21 Confirmed, 2 Firmware
Handled, 3 Improvement Recommended, 1 Not Applicable; 20 closed, 7 open with their closing path.

PV family (D-065, D-072): the 45 A port rating no longer clamps the inductor current in the near-unity
band (inductor rating 47.7 A there; 550/550 V 73.3 kW; rated power from 562 V); control model re-based on
the drawn boards with a published delivered-power envelope per product and direction; leg commutation
re-run on the drawn Jianghai capacitors (1374 V worst vs 1445 V); comparator common-mode term in every
trip band (window 67.9-80.5 A, the 1.10 margin rule missed by 0.58 A and left open; firmware OV derived
from the drawn band, 1034 V); one fan-supply contract; cold-start passive-power restriction modelled;
port A interface declared; aux pull-in and retry rules.

PCS-P125 (D-066, D-067): control study sim/pcs_control.py (PR current loop 1750 Hz, PM >= 48.7 deg to
SCR 5 with the passive damping branch, PLL, DC-link loop, grid forming, state machine); DC-link inventory
409.4 uF with bleeders, precharge rating and the 15 min label re-derived; upper-half limit in firmware;
P-Q-Vdc-Vac envelope (AC-02's 600 V full-load figure not reachable at a +15 % grid: owner's decision);
R_DS(on) acceptance rule for the six paralleled devices; DESAT string 3 -> 2 diodes (band 6.41-9.37 V);
fuse-contactor coordination bands and installation requirements; phase-current sensor frozen to Sinomags
STK-250HO/4 and the control-board ladders re-valued; Al2O3 pad text.

DAB-D60 (D-068): study vs drawn-board identity made explicit; short-circuit chain corrected (energy-
equivalent 0.99 x the assumed withstand; release block t_SC >= 2.22 us / E_SC >= 2.18 J); admitted map
follows the 1200 V deck envelope (900-950 V rows derated until a double-pulse test); zero/light-load policy;
0.41 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
Parts:
- D1602: Manufacturer Bourns -> MDD (Microdiode Semiconductor)
Changed lines of the file:
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@@
 			)
 		)
-		(property "Datasheet" "docs/datasheets/protection/SMBJ_Bourns.pdf"
+		(property "Datasheet" "docs/datasheets/protection/MDD-SMBJ-series.pdf"
 			(at 396.24 170.18 0)
 			(hide yes)
@@
 			)
 		)
-		(property "Manufacturer" "Bourns"
+		(property "Manufacturer" "MDD (Microdiode Semiconductor)"
 			(at 396.24 170.18 0)
 			(hide yes)
