File: hardware/PV-PWR-4/sheets/20_aux75_input.kicad_sch (KiCad schematic)
At the start: 10 parts

Commit message: Megarevo module parity: four-wire inverter, AC-side start-up, Ethernet and recorder on the control board, aux rev A3 (D-073..D-077)
- D-073 parity policy and register (modules only; PMA0125 and PMD-75-G3 sheets, PMA manual notes, catalogue 2026 manifest row)
- D-074 PCS-PWR-4W + PCS-CTL-4W = PCS-P125-4W drawn (fourth leg, L_N, 4-pole AC port, VGN, IL4), AC start-up tap and
  AC precharge on both builds, 30 firmware rows, declarations (kVA tiers, AC short-circuit coordination, airflow, precision)
- D-075 control board: CH9121T Ethernet bridge over CA-IS3842HW (fitted on PCS-CTL), GD25Q32E recorder flash replacing the
  EEPROM, chainable stop / ready / battery-fault inputs and HFD27 ready relay, port roles, altitude 2,000 m with the 15 mm
  isolator option specified, SELV logic allocation 2.2 W
- D-076 AUX-75 rev A3: live 30 W / 48 W for 1 s, one design for every module (turns 50:9:10, sense 3 x 0.866 ohm), four-wire
  DC precharge drawn at 200 ohm; D-077 control study: off-grid secondary restoration, THDu, imbalance, ride-through limiter
  with the stiff-grid derating rule, neutral-leg loop
- sim/compare_megarevo_pcs.py: PCS-P125 / PCS-P125-4W against the PMA0125 (2 better, 38 meets, 4 below, 9 not assessed, 0
  pending of 53); PV comparison 2 / 24 / 3 / 5 / 0 of 34 (standby 12.7 / 22.4 W)
- pin ledger E: control-board parts, shield-pin rule, fuse and connector notes (247 parts, 191 pass, 0 fail); review register
  PCM-14 and PCM-22 closed; magnetics re-run; all 15 boards rebuilt, BOMs, costs, audits and figures regenerated; README,
  guide 01-13 and the decisions mirror updated

Co-Authored-By: Claude Fable 5.1 <noreply@anthropic.com>
Other:
- note added: "2 per tap AHEAD of the fuse (AC10 pulse-rated, 20 R = the smallest E24 value inside AX-01 / 02: hot-plug I2t 18.1 % of the fuse melting I2t (rule 20 %), film surge 1218 V); 4.64 W each at the highest input current (0.48 A, 250 V) Fuse: (30 W case, unchanged) per-port fuse 1000 VDC gPV behind 44R: fault current <= 25 A (breaking 20 kA not needed), hot-plug I2t 0.091 A2s = 16 % of melting"
- note removed: "2 per tap AHEAD of the fuse (AC10 pulse-rated, 20 R = the smallest E24 value inside AX-01 / 02: hot-plug I2t 18.1 % of the fuse melting I2t (rule 20 %), film surge 1218 V); 4.14 W each at 200 V / 75 W Fuse: (30 W case, unchanged) per-port fuse 1000 VDC gPV behind 44R: fault current <= 25 A (breaking 20 kA not needed), hot-plug I2t 0.091 A2s = 16 % of melting"
- moved on the sheet: C2201, C2202, D2202, F2202, R2203, R2204
