File: hardware/PV-PWR-4/sheets/04_ph1_gdb.kicad_sch (KiCad schematic)
At the start: 155 parts, among them Q401 PMV30ENEAR, Q402 PMV30ENEAR, Q403 PMV30ENEAR, Q404 MMBT3906,215, Q405 MMBT3904,215, Q406 MMBT3904,215, Q407 MMBT3906,215, Q408 MMBT3904,215, Q409 PMV30ENEAR, Q410 PMV30ENEAR, Q411 PMV30ENEAR, Q412 MMBT3906,215, Q413 MMBT3904,215, Q414 MMBT3904,215, Q415 MMBT3906,215, Q416 MMBT3904,215, U401 SN74LVC1G17DBVR, U402 NSI6651ASC-Q1SWR, U403 SN74LVC1G17DBVR, U404 NSI6651ASC-Q1SWR

Commit message: Resolve the independent PCM review of 033d8d8 (PCM-01..27): verify, classify, fix at the root (D-065..D-072)
Register gen/data/review_pcm.csv: 27 findings, each verified before a change - 21 Confirmed, 2 Firmware
Handled, 3 Improvement Recommended, 1 Not Applicable; 20 closed, 7 open with their closing path.

PV family (D-065, D-072): the 45 A port rating no longer clamps the inductor current in the near-unity
band (inductor rating 47.7 A there; 550/550 V 73.3 kW; rated power from 562 V); control model re-based on
the drawn boards with a published delivered-power envelope per product and direction; leg commutation
re-run on the drawn Jianghai capacitors (1374 V worst vs 1445 V); comparator common-mode term in every
trip band (window 67.9-80.5 A, the 1.10 margin rule missed by 0.58 A and left open; firmware OV derived
from the drawn band, 1034 V); one fan-supply contract; cold-start passive-power restriction modelled;
port A interface declared; aux pull-in and retry rules.

PCS-P125 (D-066, D-067): control study sim/pcs_control.py (PR current loop 1750 Hz, PM >= 48.7 deg to
SCR 5 with the passive damping branch, PLL, DC-link loop, grid forming, state machine); DC-link inventory
409.4 uF with bleeders, precharge rating and the 15 min label re-derived; upper-half limit in firmware;
P-Q-Vdc-Vac envelope (AC-02's 600 V full-load figure not reachable at a +15 % grid: owner's decision);
R_DS(on) acceptance rule for the six paralleled devices; DESAT string 3 -> 2 diodes (band 6.41-9.37 V);
fuse-contactor coordination bands and installation requirements; phase-current sensor frozen to Sinomags
STK-250HO/4 and the control-board ladders re-valued; Al2O3 pad text.

DAB-D60 (D-068): study vs drawn-board identity made explicit; short-circuit chain corrected (energy-
equivalent 0.99 x the assumed withstand; release block t_SC >= 2.22 us / E_SC >= 2.18 J); admitted map
follows the 1200 V deck envelope (900-950 V rows derated until a double-pulse test); zero/light-load policy;
0.41 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
Other:
- note added: "DESAT > 10.3-10.9 V (above the 10.0 V maximum trip of the -Q1 grade) -> MMBT3904 -> MMBT3906 charges BG to VEE + 10 V; per device AO3400A + 22R pull the gate to VEE; BG holds ~3 us (1k + FET gates)."
- note added: "DESAT pin (internal 500 uA blanking source, trip 8.5-10.0 V) - Rs - 3 x US1M - drain. BAT54S keeps DX between COM and VDD against dv/dt through the string; Cblk footprint DNP."
- note removed: "DESAT > 10.3-10.9 V (above the 9.8 V maximum trip) -> MMBT3904 -> MMBT3906 charges BG to VEE + 10 V; per device AO3400A + 22R pull the gate to VEE; BG holds ~3 us (1k + FET gates)."
- note removed: "DESAT pin (internal 500 uA blanking source, trip 8.5-9.8 V) - Rs - 3 x US1M - drain. BAT54S keeps DX between COM and VDD against dv/dt through the string; Cblk footprint DNP."
- moved on the sheet: C416, C417, C418, C419, C420, C421, C422, C423, C424, C425, C426, C427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

Commit message: Respond to the independent economical re-check R4 of 845131d (D-081): DESAT string re-rated to 1300 V diodes, cable-aware DC-bus window enforced, off-grid envelope stated as declared capability, inverter cold rating -10 C, grade-B rating stated, magnetics RFQ index
- Register gen/data/review_r4.csv: 12 decision areas closed (3 Confirmed, 4 Already Fixed, 3 Improvement Recommended, 2 Not Applicable)
- E01: the DESAT sense string sees the whole DC link (static envelope 1130 V) on an off switch; 2 x Vishay BYG23T-M3/TR (1300 V)
  per channel on both presets, each diode blocking the envelope alone; PCS window unchanged, PV preset 3 -> 2 diodes; grade
  tables identical; +0.96 to +2.12 USD per module at 5k; datasheet, prices, ledger rows, insulation table
- E04: inter-module cable in the coupled PCS/PV bus model (+28 V); product rule default set point 750 V (755 V four-wire mode A),
  782 V firmware clamp in the PV module, PCS refuses an island start above 791 V, 909 V recorded as model validity; harness contract
- E06: AC-04 reworded as the module's declared output capability with the release sequence (grid-following first)
- E11: PCS cold-start passive table modelled; rating full operation from -10 C inlet (AC-02 amended by delegation), cold fan RFQ open
- E05: grade-B rating 124.57 kW at PF 1 stated; E12: docs/requirements/RFQ-MAGNETICS.md (ten RFQs); the port CM ring's catalog
  entry set to the flat-permeability grade and the aux transformer's thermal test to the 94.2 W rating
- All 15 boards, BOMs, costs, comparisons (PV 2/24/3/5/0, PCS 2/38/4/9/0), audits (pin 192/0/55, insulation 98 known) and figures
  regenerated; README, guide 01-13, INSTALLATION.md (77 rows), decisions mirror and the registers updated

Co-Authored-By: Claude Fable 5.1 <noreply@anthropic.com>
Parts:
- removed D435, D436: US1MH, symbol dcdc:US1M
- D416, D417, D434: value US1MH -> BYG23T-M3/TR; symbol dcdc:US1M -> dcdc:BYG23T; MPN US1MH -> BYG23T-M3/TR; Manufacturer Taiwan Semiconductor -> Vishay
- D418: value US1MH -> BAT54; symbol dcdc:US1M -> dcdc:BAT54; Domain CROSSING -> LIVE; MPN US1MH -> BAT54; Manufacturer Taiwan Semiconductor -> Nexperia; Package SMA (DO-214AC) -> SOT-23
- D419: value BAT54 -> BZX84-B20,215; symbol dcdc:BAT54 -> dcdc:BZX84-B20,215; Domain LIVE -> GD_P1S4; MPN BAT54 -> BZX84-B20,215
- D420, D423: value BZX84-B20,215 -> BZX84-B4V7; symbol dcdc:BZX84-B20,215 -> dcdc:BZX84-B4V7; MPN BZX84-B20,215 -> BZX84-B4V7
- D421, D424: value BZX84-B4V7 -> PMEG4010CEJ; symbol dcdc:BZX84-B4V7 -> dcdc:PMEG4010CEJ; MPN BZX84-B4V7 -> PMEG4010CEJ; Package SOT-23 -> SOD-323F
- D422: value PMEG4010CEJ -> BZX84-B20,215; symbol dcdc:PMEG4010CEJ -> dcdc:BZX84-B20,215; MPN PMEG4010CEJ -> BZX84-B20,215; Package SOD-323F -> SOT-23
- D425: value PMEG4010CEJ -> BZX84-B3V3; symbol dcdc:PMEG4010CEJ -> dcdc:BZX84-B3V3,215; MPN PMEG4010CEJ -> BZX84-B3V3; Package SOD-323F -> SOT-23
- D427: value BZX84-B3V3 -> BAT54; symbol dcdc:BZX84-B3V3,215 -> dcdc:BAT54; MPN BZX84-B3V3 -> BAT54
- D428: value BAT54 -> BZX84-B5V6; symbol dcdc:BAT54 -> dcdc:BZX84-B5V6; MPN BAT54 -> BZX84-B5V6
- D429: value BZX84-B5V6 -> BZX84-B10; symbol dcdc:BZX84-B5V6 -> dcdc:BZX84-B10; MPN BZX84-B5V6 -> BZX84-B10
- D431: value BZX84-B10 -> BAT54S; symbol dcdc:BZX84-B10 -> dcdc:BAT54S; MPN BZX84-B10 -> BAT54S
- D432: value BAT54S -> BAT54; symbol dcdc:BAT54S -> dcdc:BAT54; MPN BAT54S -> BAT54
- D433: value BAT54 -> BYG23T-M3/TR; symbol dcdc:BAT54 -> dcdc:BYG23T; Domain GD_P1S4 -> CROSSING; MPN BAT54 -> BYG23T-M3/TR; Manufacturer Nexperia -> Vishay; Package SOT-23 -> SMA (DO-214AC)
Connections:
- net BG_P1S4: now also D430.3 (K); no longer D431.3 (K)
- net BTZ_P1S4: now also D429.1 (A); no longer D430.1 (A)
- net B_BUS+: now also D417.1 (K); no longer D418.1 (K)
- net CLMP_P1S4: now also D421.2 (A), D424.2 (A), D427.3 (K); no longer D422.2 (A), D425.2 (A), D428.3 (K)
- net COM_P1S4: now also D425.1 (A), D431.1 (A); no longer D426.1 (A), D432.1 (A)
- net DS1_P1S4: now also D433.1 (K), D434.2 (A); no longer D434.1 (K)
- net DTS_P1S4: now also D418.3 (K); no longer D419.3 (K)
- net DX_P1S4: now also D429.3 (K), D431.3 (COM); no longer D430.3 (K), D433.3 (K)
- net DY_P1S4: now also D433.2 (A); no longer D434.2 (A)
- net G_P1S4a: now also D419.3 (K), D421.1 (K); no longer D420.3 (K), D422.1 (K)
- net G_P1S4b: now also D422.3 (K), D424.1 (K); no longer D423.3 (K), D425.1 (K)
- net KS_P1S4a: now also D420.3 (K); no longer D421.3 (K)
- net KS_P1S4b: now also D423.3 (K); no longer D424.3 (K)
- net NDX_P1S4: now also D432.1 (A); no longer D433.1 (A)
- net OUTH_P1S4: now also D428.3 (K); no longer D429.3 (K)
- net PWM3_5V: now also D418.1 (A); no longer D419.1 (A)
- net QID_P1S4: now also D426.3 (K); no longer D427.3 (K)
- net QIZ_P1S4: now also D426.1 (A); no longer D428.1 (A)
- net QRZ_P1S4: now also D428.1 (A); no longer D429.1 (A)
- net SW_B1: now also D434.1 (K)
- net VCG_P1S4: now also D425.3 (K); no longer D426.3 (K)
- net VDD_P1S4: now also D431.2 (K); no longer D432.2 (K)
- net VEE_P1S4: now also D430.1 (A); no longer D431.1 (A)
- net ZM1_P1S4: now also D419.1 (A); no longer D421.1 (A)
- net ZM2_P1S4: now also D422.1 (A); no longer D424.1 (A)
- net DS2_P1S3: no longer names the net of D418.2 (NC)
- net DS2_P1S3: no longer D417.1 (K)
Other:
- note added: "DESAT pin (internal 500 uA blanking source, trip 8.5-10.0 V) - Rs - 2 x BYG23T-M3/TR (1300 V each) - drain. BAT54S keeps DX between COM and VDD against dv/dt through the string; Cblk footprint DNP."
- note removed: "DESAT pin (internal 500 uA blanking source, trip 8.5-10.0 V) - Rs - 3 x US1M - drain. BAT54S keeps DX between COM and VDD against dv/dt through the string; Cblk footprint DNP."
- moved on the sheet: C416, C417, C418, C419, C420, C421, C422, C423, C424, C425, C426, C427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
