File: hardware/PV-PWR-4/sheets/09_ph3_gda.kicad_sch (KiCad schematic)
At the start: 155 parts, among them Q901 PMV30ENEAR, Q902 PMV30ENEAR, Q903 PMV30ENEAR, Q904 MMBT3906,215, Q905 MMBT3904,215, Q906 MMBT3904,215, Q907 MMBT3906,215, Q908 MMBT3904,215, Q909 PMV30ENEAR, Q910 PMV30ENEAR, Q911 PMV30ENEAR, Q912 MMBT3906,215, Q913 MMBT3904,215, Q914 MMBT3904,215, Q915 MMBT3906,215, Q916 MMBT3904,215, U901 SN74LVC1G17DBVR, U902 NSI6651ASC-Q1SWR, U903 SN74LVC1G17DBVR, U904 NSI6651ASC-Q1SWR

Commit message: Resolve the independent PCM review of 033d8d8 (PCM-01..27): verify, classify, fix at the root (D-065..D-072)
Register gen/data/review_pcm.csv: 27 findings, each verified before a change - 21 Confirmed, 2 Firmware
Handled, 3 Improvement Recommended, 1 Not Applicable; 20 closed, 7 open with their closing path.

PV family (D-065, D-072): the 45 A port rating no longer clamps the inductor current in the near-unity
band (inductor rating 47.7 A there; 550/550 V 73.3 kW; rated power from 562 V); control model re-based on
the drawn boards with a published delivered-power envelope per product and direction; leg commutation
re-run on the drawn Jianghai capacitors (1374 V worst vs 1445 V); comparator common-mode term in every
trip band (window 67.9-80.5 A, the 1.10 margin rule missed by 0.58 A and left open; firmware OV derived
from the drawn band, 1034 V); one fan-supply contract; cold-start passive-power restriction modelled;
port A interface declared; aux pull-in and retry rules.

PCS-P125 (D-066, D-067): control study sim/pcs_control.py (PR current loop 1750 Hz, PM >= 48.7 deg to
SCR 5 with the passive damping branch, PLL, DC-link loop, grid forming, state machine); DC-link inventory
409.4 uF with bleeders, precharge rating and the 15 min label re-derived; upper-half limit in firmware;
P-Q-Vdc-Vac envelope (AC-02's 600 V full-load figure not reachable at a +15 % grid: owner's decision);
R_DS(on) acceptance rule for the six paralleled devices; DESAT string 3 -> 2 diodes (band 6.41-9.37 V);
fuse-contactor coordination bands and installation requirements; phase-current sensor frozen to Sinomags
STK-250HO/4 and the control-board ladders re-valued; Al2O3 pad text.

DAB-D60 (D-068): study vs drawn-board identity made explicit; short-circuit chain corrected (energy-
equivalent 0.99 x the assumed withstand; release block t_SC >= 2.22 us / E_SC >= 2.18 J); admitted map
follows the 1200 V deck envelope (900-950 V rows derated until a double-pulse test); zero/light-load policy;
0.41 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
Other:
- note added: "DESAT > 10.3-10.9 V (above the 10.0 V maximum trip of the -Q1 grade) -> MMBT3904 -> MMBT3906 charges BG to VEE + 10 V; per device AO3400A + 22R pull the gate to VEE; BG holds ~3 us (1k + FET gates)."
- note added: "DESAT pin (internal 500 uA blanking source, trip 8.5-10.0 V) - Rs - 3 x US1M - drain. BAT54S keeps DX between COM and VDD against dv/dt through the string; Cblk footprint DNP."
- note removed: "DESAT > 10.3-10.9 V (above the 9.8 V maximum trip) -> MMBT3904 -> MMBT3906 charges BG to VEE + 10 V; per device AO3400A + 22R pull the gate to VEE; BG holds ~3 us (1k + FET gates)."
- note removed: "DESAT pin (internal 500 uA blanking source, trip 8.5-9.8 V) - Rs - 3 x US1M - drain. BAT54S keeps DX between COM and VDD against dv/dt through the string; Cblk footprint DNP."
- moved on the sheet: C916, C917, C918, C919, C920, C921, C922, C923, C924, C925, C926, C927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

Commit message: Respond to the independent economical re-check R4 of 845131d (D-081): DESAT string re-rated to 1300 V diodes, cable-aware DC-bus window enforced, off-grid envelope stated as declared capability, inverter cold rating -10 C, grade-B rating stated, magnetics RFQ index
- Register gen/data/review_r4.csv: 12 decision areas closed (3 Confirmed, 4 Already Fixed, 3 Improvement Recommended, 2 Not Applicable)
- E01: the DESAT sense string sees the whole DC link (static envelope 1130 V) on an off switch; 2 x Vishay BYG23T-M3/TR (1300 V)
  per channel on both presets, each diode blocking the envelope alone; PCS window unchanged, PV preset 3 -> 2 diodes; grade
  tables identical; +0.96 to +2.12 USD per module at 5k; datasheet, prices, ledger rows, insulation table
- E04: inter-module cable in the coupled PCS/PV bus model (+28 V); product rule default set point 750 V (755 V four-wire mode A),
  782 V firmware clamp in the PV module, PCS refuses an island start above 791 V, 909 V recorded as model validity; harness contract
- E06: AC-04 reworded as the module's declared output capability with the release sequence (grid-following first)
- E11: PCS cold-start passive table modelled; rating full operation from -10 C inlet (AC-02 amended by delegation), cold fan RFQ open
- E05: grade-B rating 124.57 kW at PF 1 stated; E12: docs/requirements/RFQ-MAGNETICS.md (ten RFQs); the port CM ring's catalog
  entry set to the flat-permeability grade and the aux transformer's thermal test to the 94.2 W rating
- All 15 boards, BOMs, costs, comparisons (PV 2/24/3/5/0, PCS 2/38/4/9/0), audits (pin 192/0/55, insulation 98 known) and figures
  regenerated; README, guide 01-13, INSTALLATION.md (77 rows), decisions mirror and the registers updated

Co-Authored-By: Claude Fable 5.1 <noreply@anthropic.com>
Parts:
- removed D935, D936: US1MH, symbol dcdc:US1M
- D916, D917, D934: value US1MH -> BYG23T-M3/TR; symbol dcdc:US1M -> dcdc:BYG23T; MPN US1MH -> BYG23T-M3/TR; Manufacturer Taiwan Semiconductor -> Vishay
- D918: value US1MH -> BAT54; symbol dcdc:US1M -> dcdc:BAT54; Domain CROSSING -> LIVE; MPN US1MH -> BAT54; Manufacturer Taiwan Semiconductor -> Nexperia; Package SMA (DO-214AC) -> SOT-23
- D919: value BAT54 -> BZX84-B20,215; symbol dcdc:BAT54 -> dcdc:BZX84-B20,215; Domain LIVE -> GD_P3S2; MPN BAT54 -> BZX84-B20,215
- D920, D923: value BZX84-B20,215 -> BZX84-B4V7; symbol dcdc:BZX84-B20,215 -> dcdc:BZX84-B4V7; MPN BZX84-B20,215 -> BZX84-B4V7
- D921, D924: value BZX84-B4V7 -> PMEG4010CEJ; symbol dcdc:BZX84-B4V7 -> dcdc:PMEG4010CEJ; MPN BZX84-B4V7 -> PMEG4010CEJ; Package SOT-23 -> SOD-323F
- D922: value PMEG4010CEJ -> BZX84-B20,215; symbol dcdc:PMEG4010CEJ -> dcdc:BZX84-B20,215; MPN PMEG4010CEJ -> BZX84-B20,215; Package SOD-323F -> SOT-23
- D925: value PMEG4010CEJ -> BZX84-B3V3; symbol dcdc:PMEG4010CEJ -> dcdc:BZX84-B3V3,215; MPN PMEG4010CEJ -> BZX84-B3V3; Package SOD-323F -> SOT-23
- D927: value BZX84-B3V3 -> BAT54; symbol dcdc:BZX84-B3V3,215 -> dcdc:BAT54; MPN BZX84-B3V3 -> BAT54
- D928: value BAT54 -> BZX84-B5V6; symbol dcdc:BAT54 -> dcdc:BZX84-B5V6; MPN BAT54 -> BZX84-B5V6
- D929: value BZX84-B5V6 -> BZX84-B10; symbol dcdc:BZX84-B5V6 -> dcdc:BZX84-B10; MPN BZX84-B5V6 -> BZX84-B10
- D931: value BZX84-B10 -> BAT54S; symbol dcdc:BZX84-B10 -> dcdc:BAT54S; MPN BZX84-B10 -> BAT54S
- D932: value BAT54S -> BAT54; symbol dcdc:BAT54S -> dcdc:BAT54; MPN BAT54S -> BAT54
- D933: value BAT54 -> BYG23T-M3/TR; symbol dcdc:BAT54 -> dcdc:BYG23T; Domain GD_P3S2 -> CROSSING; MPN BAT54 -> BYG23T-M3/TR; Manufacturer Nexperia -> Vishay; Package SOT-23 -> SMA (DO-214AC)
Connections:
- net A_BUS+: now also D917.1 (K); no longer D918.1 (K)
- net BG_P3S2: now also D930.3 (K); no longer D931.3 (K)
- net BTZ_P3S2: now also D929.1 (A); no longer D930.1 (A)
- net CLMP_P3S2: now also D921.2 (A), D924.2 (A), D927.3 (K); no longer D922.2 (A), D925.2 (A), D928.3 (K)
- net COM_P3S2: now also D925.1 (A), D931.1 (A); no longer D926.1 (A), D932.1 (A)
- net DS1_P3S2: now also D933.1 (K), D934.2 (A); no longer D934.1 (K)
- net DTS_P3S2: now also D918.3 (K); no longer D919.3 (K)
- net DX_P3S2: now also D929.3 (K), D931.3 (COM); no longer D930.3 (K), D933.3 (K)
- net DY_P3S2: now also D933.2 (A); no longer D934.2 (A)
- net G_P3S2a: now also D919.3 (K), D921.1 (K); no longer D920.3 (K), D922.1 (K)
- net G_P3S2b: now also D922.3 (K), D924.1 (K); no longer D923.3 (K), D925.1 (K)
- net KS_P3S2a: now also D920.3 (K); no longer D921.3 (K)
- net KS_P3S2b: now also D923.3 (K); no longer D924.3 (K)
- net NDX_P3S2: now also D932.1 (A); no longer D933.1 (A)
- net OUTH_P3S2: now also D928.3 (K); no longer D929.3 (K)
- net PWM9_5V: now also D918.1 (A); no longer D919.1 (A)
- net QID_P3S2: now also D926.3 (K); no longer D927.3 (K)
- net QIZ_P3S2: now also D926.1 (A); no longer D928.1 (A)
- net QRZ_P3S2: now also D928.1 (A); no longer D929.1 (A)
- net SW_A3: now also D934.1 (K)
- net VCG_P3S2: now also D925.3 (K); no longer D926.3 (K)
- net VDD_P3S2: now also D931.2 (K); no longer D932.2 (K)
- net VEE_P3S2: now also D930.1 (A); no longer D931.1 (A)
- net ZM1_P3S2: now also D919.1 (A); no longer D921.1 (A)
- net ZM2_P3S2: now also D922.1 (A); no longer D924.1 (A)
- net DS2_P3S1: no longer names the net of D918.2 (NC)
- net DS2_P3S1: no longer D917.1 (K)
Other:
- note added: "DESAT pin (internal 500 uA blanking source, trip 8.5-10.0 V) - Rs - 2 x BYG23T-M3/TR (1300 V each) - drain. BAT54S keeps DX between COM and VDD against dv/dt through the string; Cblk footprint DNP."
- note removed: "DESAT pin (internal 500 uA blanking source, trip 8.5-10.0 V) - Rs - 3 x US1M - drain. BAT54S keeps DX between COM and VDD against dv/dt through the string; Cblk footprint DNP."
- moved on the sheet: C916, C917, C918, C919, C920, C921, C922, C923, C924, C925, C926, C927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
