File: hardware/PCS-CTL/sheets/01_supply.kicad_sch (KiCad schematic)
At the start: 6 parts, among them J101 X6521FV-2x32-C85D32, U101 TPS3828-33DBVR

Commit message: Complete the inverter control board PCS-CTL rev A0 for the three-wire build (D-064)
Grid-voltage, residual-current and temperature signals into the ADC, the second AC contactor through the
trip latch, the residual-current test output and the inverter pin plan. 8 sheets, 305 parts, 209 nets; every
build check passes; the PV control board's outputs are unchanged. The controller has 23 analog pins, not 25:
the eight temperature inputs share one pin through a multiplexer that is in no trip path. Module PCS-P125:
1,521 USD at catalogue prices, 1,292 USD at 5,000 units. Everything is calculated or estimated.

Co-Authored-By: Claude Fable 5.1 <noreply@anthropic.com>
Connections:
- net IA: no longer names the net of J101.46 (Pin_46)
- net IA_H: no longer names the net of J101.47 (Pin_47)
- net VAX: no longer names the net of J101.52 (Pin_52)
- no-connect marks 1 -> 4
Other:
- title: PV-CTL control board - PC connector, supply, reset -> PCS-CTL control board - PC connector, supply, reset
Changed lines of the file:
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@@
 	(paper "A3")
 	(title_block
-		(title "PV-CTL control board - PC connector, supply, reset")
+		(title "PCS-CTL control board - PC connector, supply, reset")
 		(date "2026-10-05")
 		(rev "A0")
@@
 		(at 139.7 33.02)
 	)
+	(no_connect
+		(at 40.64 91.44)
+	)
+	(no_connect
+		(at 40.64 83.82)
+	)
+	(no_connect
+		(at 27.94 86.36)
+	)
 	(wire
 		(pts
@@
 	(wire
 		(pts
-			(xy 40.64 83.82) (xy 43.18 83.82)
-		)
-		(stroke
-			(width 0)
-			(type default)
-		)
-	)
-	(wire
-		(pts
 			(xy 27.94 76.2) (xy 25.4 76.2)
 		)
@@
 	(wire
 		(pts
-			(xy 40.64 91.44) (xy 43.18 91.44)
-		)
-		(stroke
-			(width 0)
-			(type default)
-		)
-	)
-	(wire
-		(pts
 			(xy 40.64 33.02) (xy 43.18 33.02)
 		)
@@
 	(wire
 		(pts
-			(xy 27.94 86.36) (xy 25.4 86.36)
-		)
-		(stroke
-			(width 0)
-			(type default)
-		)
-	)
-	(wire
-		(pts
 			(xy 208.28 39.37) (xy 208.28 41.91)
 		)
@@
 		)
 	)
-	(global_label "VAX"
-		(shape bidirectional)
-		(at 43.18 91.44 0)
-		(fields_autoplaced yes)
-		(effects
-			(font
-				(size 1 1)
-			)
-			(justify left)
-		)
-		(property "Intersheetrefs" "${INTERSHEET_REFS}"
-			(at 43.18 91.44 0)
-			(hide yes)
-			(show_name no)
-			(do_not_autoplace no)
-			(effects
-				(font
-					(size 1 1)
-				)
-			)
-		)
-	)
 	(global_label "PWM15"
 		(shape bidirectional)
@@
 		)
 	)
-	(global_label "IA_H"
-		(shape bidirectional)
-		(at 25.4 86.36 180)
-		(fields_autoplaced yes)
-		(effects
-			(font
-				(size 1 1)
-			)
-			(justify right)
-		)
-		(property "Intersheetrefs" "${INTERSHEET_REFS}"
-			(at 25.4 86.36 180)
-			(hide yes)
-			(show_name no)
-			(do_not_autoplace no)
-			(effects
-				(font
-					(size 1 1)
-				)
-			)
-		)
-	)
 	(global_label "IL4"
 		(shape bidirectional)
@@
 			(hide yes)
 			(show_name no)
-			(do_not_autoplace no)
-			(effects
-				(font
-					(size 1 1)
-				)
-			)
-		)
-	)
-	(global_label "IA"
-		(shape bidirectional)
-		(at 43.18 83.82 0)
-		(fields_autoplaced yes)
-		(effects
-			(font
-				(size 1 1)
-			)
-			(justify left)
-		)
-		(property "Intersheetrefs" "${INTERSHEET_REFS}"
-			(at 43.18 83.82 0)
-			(hide yes)
-			(show_name no)
