File: hardware/PCS-CTL/sheets/02_mcu.kicad_sch (KiCad schematic)
At the start: 33 parts, among them J201 X1270WVS-2x10B-9TV01, U201 F280039CSPZR, U202 X1G0041710033, U203 BL24C256A-PARC

Commit message: Complete the inverter control board PCS-CTL rev A0 for the three-wire build (D-064)
Grid-voltage, residual-current and temperature signals into the ADC, the second AC contactor through the
trip latch, the residual-current test output and the inverter pin plan. 8 sheets, 305 parts, 209 nets; every
build check passes; the PV control board's outputs are unchanged. The controller has 23 analog pins, not 25:
the eight temperature inputs share one pin through a multiplexer that is in no trip path. Module PCS-P125:
1,521 USD at catalogue prices, 1,292 USD at 5,000 units. Everything is calculated or estimated.

Co-Authored-By: Claude Fable 5.1 <noreply@anthropic.com>
Connections:
- net GND: no longer RN206.4 (R4.1)
- net MUX_A2: now reaches U201.44 (GPIO60)
- net MUX_A0: now reaches U201.67 (GPIO58)
- net K_AC2_M: now reaches U201.91 (GPIO61)
- net K_AC2_M: now also RN206.4 (R4.1)
- net MUX_A1: now reaches U201.92 (GPIO59)
- net RCM_TST: now reaches U201.49 (B11/GPIO21)
- net IA_ADC: no longer names the net of U201.23 (A0/B15/C15/DACA_OUT)
- net IA_H_ADC: no longer names the net of U201.21 (B12/C2)
- net NTC1 renamed VG3_ADC
- net NTC2 renamed VG2_ADC
- net NTC3 renamed VC2_ADC
- net NTC4 renamed VC1_ADC
- net NTC5 renamed NTC_MUX
- net NTC6 renamed RCM_ADC
- net NTC7 renamed NTC9
- net NTC8 renamed VC3_ADC
- net VAX_ADC renamed VG1_ADC
- no-connect marks 8 -> 5
Other:
- note added: "Every MCU output that ends in an AND gate here is low while the MCU is in reset or unprogrammed (GPIOs high impedance): 16 PWM, EN, K_A, K_B, K_PRE, STATUS, FAN_PWM, HEARTBEAT, K_AC2 (24 lines, 0 spare elements). BIAS_EN, IMD_SW1/2 go straight to PC: pulled down on the power board (10k / 100k, PV-PWR)."
- note removed: "Every MCU output that ends in an AND gate here is low while the MCU is in reset or unprogrammed (GPIOs high impedance): 16 PWM, EN, K_A, K_B, K_PRE, STATUS, FAN_PWM, HEARTBEAT (23 lines, 1 spare element). BIAS_EN, IMD_SW1/2 go straight to PC: pulled down on the power board (10k / 100k, PV-PWR)."
- title: PV-CTL control board - F280039C, clock, debug, EEPROM -> PCS-CTL control board - F280039C, clock, debug, EEPROM

Commit message: Megarevo module parity: four-wire inverter, AC-side start-up, Ethernet and recorder on the control board, aux rev A3 (D-073..D-077)
- D-073 parity policy and register (modules only; PMA0125 and PMD-75-G3 sheets, PMA manual notes, catalogue 2026 manifest row)
- D-074 PCS-PWR-4W + PCS-CTL-4W = PCS-P125-4W drawn (fourth leg, L_N, 4-pole AC port, VGN, IL4), AC start-up tap and
  AC precharge on both builds, 30 firmware rows, declarations (kVA tiers, AC short-circuit coordination, airflow, precision)
- D-075 control board: CH9121T Ethernet bridge over CA-IS3842HW (fitted on PCS-CTL), GD25Q32E recorder flash replacing the
  EEPROM, chainable stop / ready / battery-fault inputs and HFD27 ready relay, port roles, altitude 2,000 m with the 15 mm
  isolator option specified, SELV logic allocation 2.2 W
- D-076 AUX-75 rev A3: live 30 W / 48 W for 1 s, one design for every module (turns 50:9:10, sense 3 x 0.866 ohm), four-wire
  DC precharge drawn at 200 ohm; D-077 control study: off-grid secondary restoration, THDu, imbalance, ride-through limiter
  with the stiff-grid derating rule, neutral-leg loop
- sim/compare_megarevo_pcs.py: PCS-P125 / PCS-P125-4W against the PMA0125 (2 better, 38 meets, 4 below, 9 not assessed, 0
  pending of 53); PV comparison 2 / 24 / 3 / 5 / 0 of 34 (standby 12.7 / 22.4 W)
- pin ledger E: control-board parts, shield-pin rule, fuse and connector notes (247 parts, 191 pass, 0 fail); review register
  PCM-14 and PCM-22 closed; magnetics re-run; all 15 boards rebuilt, BOMs, costs, audits and figures regenerated; README,
  guide 01-13 and the decisions mirror updated

Co-Authored-By: Claude Fable 5.1 <noreply@anthropic.com>
Parts:
- added JP201: Solder jumper, open by default, symbol dcdc:JP_OPEN
- added R210: 680R, symbol dcdc:R
- R205, R206: value 4.7k -> 10k
- R209: value 680R -> 10k
- U203: value BL24C256A-PARC -> GD25Q32ESIGR; symbol dcdc:BL24C256A -> dcdc:GD25Q32E; MPN BL24C256A-PARC -> GD25Q32ESIGR; Manufacturer Shanghai Belling -> GigaDevice; Package SOP-8 -> SOP-8 208 mil
Connections:
- net CAN_TX: now also R209.2; no longer R208.2
- net GND: now also D201.1 (K), JP201.2 (B); no longer U203.1 (A0), U203.2 (A1), U203.3 (A2), U203.7 (WP)
- net LATCH_CLR: now also R208.2; no longer R207.2
- net LED_RUN_A: now also R210.2; no longer R209.2
- net TACH1: now also U201.63 (GPIO35/TDI); no longer U201.13 (GPIO54)
- net TACH2: now also U201.94 (GPIO34); no longer U201.43 (GPIO55)
- net SPI_CLK: now reaches U201.68 (GPIO18/X2)
- net SPI_CLK: now also U203.6 (SCLK)
- net VGN_ADC: now reaches U201.21 (B12/C2)
- removed net I2C_SCL: R206.2, U201.66 (GPIO57), U203.6 (SCL)
- removed net I2C_SDA: R205.2, U201.65 (GPIO56), U203.5 (SDA)
- removed net LED_RUN_N: D201.1 (K), U201.94 (GPIO34)
- net OC_N renamed PRE_N
- net OVT_N renamed DI1
- net TDI: no longer names the net of J201.3 (Pin_3)
- net TDI: no longer U201.63 (GPIO35/TDI)
- net TDO: no longer names the net of J201.7 (Pin_7)
- net TDO: no longer U201.61 (GPIO37/TDO)
- new net ETH_RXD: U201.66 (GPIO57)
- new net ETH_TXD: U201.65 (GPIO56)
- new net FLASH_CS_N: R205.2, U201.61 (GPIO37/TDO), U203.1 (CS#)
- new net FLASH_HOLD_N: R206.2, U203.7 (HOLD#)
- new net FLASH_WP_N: JP201.1 (A), R207.2, U203.3 (WP#)
- new net SPI_SIMO: U201.13 (GPIO54), U203.5 (SI)
- new net SPI_SOMI: U201.43 (GPIO55), U203.2 (SO)
- new net WD_OK: R210.1
Other:
- note added: "GD25Q32E 4 MB on SPIA (SCLK GPIO18, SI GPIO54, SO GPIO55, CS# GPIO37). CS# 10k pull-up: deselected in reset and boot (TDO floats until firmware owns it). HOLD# 10k up. WP# 10k up + write-protect strap JP to GND (closed at end of line with SRP0 = 1: status register and the golden-image blocks locked). Replaces the I2C EEPROM."
- note added: "Green, lit while the heartbeat monoflop holds WD_OK high (control ISR running, no MCU reset): the hardware's own view of 'firmware alive'. 680 R, ~2 mA from the 74LVC1G123 output (IOH 24 mA at 3.0 V)."
- note added: "JTAG CTI-20 IN CJTAG MODE - HAZARDOUS LIVE (ISOLATED PROBE ONLY)"
- note added: "Label: 'HAZARDOUS VOLTAGE - up to 1000 V DC to earth - isolated debug probe only'. cJTAG (IEEE 1149.7, TMS + TCK; SPRSP61C 6.12.6): TDI (3) / TDO (7) open, GPIO35 / 37 are TACH1 / flash CS#. TMS 2.2k pull-up; TRST (2) open; EMU0/1 4.7k; RESET (15) on XRSn. Field update over Ethernet / RS-485 / CAN: no live access."
- note added: "RECORDER FLASH: FAULT RECORDS, TWO FIRMWARE IMAGES, CALIBRATION, SERIAL NUMBER, EVENT LOG"
- note added: "RUN LED ON WD_OK (REV A2: GPIO34 FREED; WD_OK FROM SHEET 05)"
- note removed: "BL24C256A at 0x50 (A2-A0 low), WP low (writable; firmware guards the calibration pages), I2C 4.7k pull-ups."
- note removed: "EEPROM (CALIBRATION, SERIAL NUMBER, EVENT LOG)"
- note removed: "Green, GPIO34 low = on (firmware heartbeat), 680 R: ~2 mA."
- note removed: "JTAG CTI-20 - HAZARDOUS LIVE (ISOLATED PROBE ONLY)"
- note removed: "Label: 'HAZARDOUS VOLTAGE - up to 1000 V DC to earth - isolated debug probe only'. TMS 2.2k pull-up (no TRSTn on F28003x, table 5-1); TRST (2) open; EMU0/1 4.7k pull-ups; RESET (15) on XRSn; 17-19 GND. Field firmware update over CAN (DCAN boot option 1 or application loader): no live access needed."
- note removed: "RUN LED"
- title: PCS-CTL control board - F280039C, clock, debug, EEPROM -> PCS-CTL control board - F280039C, clock, debug, recorder flash
- moved on the sheet: C212, D201, R205, R206, R207, R208, R209, RN201, RN202, RN203, RN204, RN205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
