File: hardware/PCS-CTL/sheets/08_pcsx.kicad_sch (KiCad schematic)
At the start: 23 parts, among them J801 X6521FV-2x08-C85D32, U801 TMUX1208PWR

Commit message: Megarevo module parity: four-wire inverter, AC-side start-up, Ethernet and recorder on the control board, aux rev A3 (D-073..D-077)
- D-073 parity policy and register (modules only; PMA0125 and PMD-75-G3 sheets, PMA manual notes, catalogue 2026 manifest row)
- D-074 PCS-PWR-4W + PCS-CTL-4W = PCS-P125-4W drawn (fourth leg, L_N, 4-pole AC port, VGN, IL4), AC start-up tap and
  AC precharge on both builds, 30 firmware rows, declarations (kVA tiers, AC short-circuit coordination, airflow, precision)
- D-075 control board: CH9121T Ethernet bridge over CA-IS3842HW (fitted on PCS-CTL), GD25Q32E recorder flash replacing the
  EEPROM, chainable stop / ready / battery-fault inputs and HFD27 ready relay, port roles, altitude 2,000 m with the 15 mm
  isolator option specified, SELV logic allocation 2.2 W
- D-076 AUX-75 rev A3: live 30 W / 48 W for 1 s, one design for every module (turns 50:9:10, sense 3 x 0.866 ohm), four-wire
  DC precharge drawn at 200 ohm; D-077 control study: off-grid secondary restoration, THDu, imbalance, ride-through limiter
  with the stiff-grid derating rule, neutral-leg loop
- sim/compare_megarevo_pcs.py: PCS-P125 / PCS-P125-4W against the PMA0125 (2 better, 38 meets, 4 below, 9 not assessed, 0
  pending of 53); PV comparison 2 / 24 / 3 / 5 / 0 of 34 (standby 12.7 / 22.4 W)
- pin ledger E: control-board parts, shield-pin rule, fuse and connector notes (247 parts, 191 pass, 0 fail); review register
  PCM-14 and PCM-22 closed; magnetics re-run; all 15 boards rebuilt, BOMs, costs, audits and figures regenerated; README,
  guide 01-13 and the decisions mirror updated

Co-Authored-By: Claude Fable 5.1 <noreply@anthropic.com>
Parts:
- added C810: 100n 50V, symbol dcdc:C
- added R813, R814: 100k, symbol dcdc:R
- C808: value 100n 50V -> 1n 50V
- R807: value 10.0k -> 100R
- R808: value 13.0k -> 1M
- R810: value 100k -> 13.0k
- R811: value 100k -> 10.0k
Connections:
- net +3V3A: now also C810.1; no longer C809.1
- net GND: now also C810.2, R813.2, R814.2; no longer R811.2
- net MUX_A0: now also R812.1; no longer R810.1
- net MUX_A1: now also R813.1; no longer R811.1
- net MUX_A2: now also R814.1; no longer R812.1
- net NTC9: now also C809.1, R811.2; no longer C808.1, R809.2
- net RCM: now also R809.1; no longer R807.1
- net RCM_ADC: now also C808.1, R809.2, R810.1; no longer C807.1, R807.2, R808.1
- net VREF: now also R811.1; no longer R809.1
- net VGN: now reaches J801.14 (Pin_14)
- net VGN: now also R807.1
- new net VGN_ADC: C807.1, R807.2, R808.1
- no-connect marks 2 -> 1
Other:
- note added: "100 R / 1 nF C0G charge buckets as VA / VB. VG1-3 on ADC-A/B/C and VC1-3 on ADC-A/B/C: each set sampled together (synchronisation, relay test VG against VC with one contactor closed). VGN (four-wire N terminal) on ADC-B/C, 1 M to GND: 0 V marks a three-wire power board."
- note added: "VGN = the N terminal of PCS-PWR-4W (left open by the three-wire PCS-PWR). K_AC2 = K_AC2_M AND HEALTHY: a trip opens AC contactor 2 as AC contactor 1. RCM_TST straight from GPIO21 (100k pull-down on PCS-PWR: open = no test current)."
- note removed: "100 R / 1 nF C0G charge buckets as VA / VB. VG1-3 on ADC-A/B/C and VC1-3 on ADC-A/B/C: each set sampled together (synchronisation, relay test VG against VC with one contactor closed)."
- note removed: "VGN (four-wire build) not connected (OPEN 4). K_AC2 = K_AC2_M AND HEALTHY: a trip opens AC contactor 2 as AC contactor 1. RCM_TST straight from GPIO21 (100k pull-down on PCS-PWR: open = no test current)."
- moved on the sheet: C801, C802, C803, C804, C805, C806, C807, C808, C809, R801, R802, R803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

Commit message: Respond to the independent re-check R2 of a427981 (D-078, D-079): gates-off commutation closed, backup band lowered, SiC acceptance, bounded grid-forming transients, ride-through without derating, AC-start repairs, installation requirements
- Register gen/data/review_r2.csv: 14 findings verified and dispositioned (9 Confirmed, 1 Firmware Handled,
  1 Improvement Recommended, 2 Already Fixed, 1 Not Applicable), every row closed with its evidence
- D-078 power stage: the discrete window turns the gates off at 520.8 A, not at the 485.5 A window top; the leg deck
  at that current peaked at 1457 V against 1445 V, closed at zero cost by R_G,off 7.5 -> 8.75 ohm (1437 V, admissible
  533.6 A); L1 inductance trajectory to 700 A (knee 566 A), CMPSS backup band lowered to 423.9-497.5 A on PCS-CTL,
  firmware OV backup 1035 V; R_DS(on) <= 40 mOhm acceptance with per-lot derating; one coil contract (20 W / 4 W);
  residual-current monitor contract; docs/requirements/INSTALLATION.md (74 enforceable requirements with sources)
- D-079 control study: tolerance regression at the assembly tolerances (1,944 + 1,000 cases, worst PM 48.1 deg);
  bounded grid-forming transients 0.43 / 1.77 pu with feed-forward and OV deadbeat (2.17 pu superseded), trip-aware
  DC-load rejection, CV-mode soft-OV hold, weak-grid CV power limits, PV DC-bus coordination row (0.51 ms);
  ride-through 270 A clamp with C_f prediction removes the stiff-grid derating (fallback kept, SCR estimator,
  8.07 MVA declaration); coupled four-wire cases; AC start in the executable state machine (17 states, 35 fault
  cases) with the five sequence holes H1-H5 repaired and an own AC_STOP state
- pcs_spec protection_chain published and read by the control study and the control board; all 15 boards, BOMs,
  costs, comparisons (PV 2/24/3/5/0, PCS 2/38/4/9/0), audits and figures regenerated; README, guide 03-13,
  decisions mirror and architecture reconciliation notes updated; .graphifyignore and graphify-out/ ignored

Co-Auth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
Other:
- note added: "OUT 2.50 V + 1.00 V/A (+/-2.0 A in 0.50-4.50 V; sensor fault <= 0.25 V or >= 4.75 V) through PCS-PWR's 100R into 10.0k / 13.0k: 0.563 V/A at the pin, 1.3 mA per LSB; the 5.25 V supply maximum reads <= 3.0 V; 1 nF C0G charge bucket. Firmware sensor-fault window and the TEST step: design check and firmware table."
- note added: "RESIDUAL CURRENT (TYPE-B SENSOR ON PCS-PWR, RFQ CONTRACT: PCS_SPEC RESIDUAL_CURRENT_CONTRACT)"
- note removed: "10.0k / 13.0k: a sensor output up to its 5.25 V supply reads <= 3.0 V; 1 nF C0G charge bucket."
- note removed: "RESIDUAL CURRENT (TYPE-B SENSOR, RFQ ON PCS-PWR; OUTPUT LEVEL ASSUMED, OPEN 5)"
- moved on the sheet: C808, C809, C810, R809, R810, R811, R812, R813, R814, U801
