File: hardware/CTRL-C2000/CTRL-C2000.kicad_sch (KiCad schematic)
At the start: 0 parts

Commit message: Resolve the independent PCM review of 033d8d8 (PCM-01..27): verify, classify, fix at the root (D-065..D-072)
Register gen/data/review_pcm.csv: 27 findings, each verified before a change - 21 Confirmed, 2 Firmware
Handled, 3 Improvement Recommended, 1 Not Applicable; 20 closed, 7 open with their closing path.

PV family (D-065, D-072): the 45 A port rating no longer clamps the inductor current in the near-unity
band (inductor rating 47.7 A there; 550/550 V 73.3 kW; rated power from 562 V); control model re-based on
the drawn boards with a published delivered-power envelope per product and direction; leg commutation
re-run on the drawn Jianghai capacitors (1374 V worst vs 1445 V); comparator common-mode term in every
trip band (window 67.9-80.5 A, the 1.10 margin rule missed by 0.58 A and left open; firmware OV derived
from the drawn band, 1034 V); one fan-supply contract; cold-start passive-power restriction modelled;
port A interface declared; aux pull-in and retry rules.

PCS-P125 (D-066, D-067): control study sim/pcs_control.py (PR current loop 1750 Hz, PM >= 48.7 deg to
SCR 5 with the passive damping branch, PLL, DC-link loop, grid forming, state machine); DC-link inventory
409.4 uF with bleeders, precharge rating and the 15 min label re-derived; upper-half limit in firmware;
P-Q-Vdc-Vac envelope (AC-02's 600 V full-load figure not reachable at a +15 % grid: owner's decision);
R_DS(on) acceptance rule for the six paralleled devices; DESAT string 3 -> 2 diodes (band 6.41-9.37 V);
fuse-contactor coordination bands and installation requirements; phase-current sensor frozen to Sinomags
STK-250HO/4 and the control-board ladders re-valued; Al2O3 pad text.

DAB-D60 (D-068): study vs drawn-board identity made explicit; short-circuit chain corrected (energy-
equivalent 0.99 x the assumed withstand; release block t_SC >= 2.22 us / E_SC >= 2.18 J); admitted map
follows the 1200 V deck envelope (900-950 V rows derated until a double-pulse test); zero/light-load policy;
0.41 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
Other:
- note added: "INPUTXBAR6 -> TRIP6. CMPSS reference = VDAC = REF5025E; firmware nulls each channel at zero input at start-up; trip bands in the pin plan, asserted against the frozen earlier-platform snapshot gen/data/control_spec_platform1.json (D-044). EN pair = GATE_EN AND CHB_OK AND MCU"
- note added: "enable (74LVC11A); line drivers on only with CHB_OK, MCU enable and RDY; EN readback on GPIO100-103. +24V_GD feeds only the cell eFuses."
- note removed: "CHB_OK, MCU enable and RDY; EN readback on GPIO100-103. +24V_GD feeds only the cell eFuses."
- note removed: "INPUTXBAR6 -> TRIP6. CMPSS reference = VDAC = REF5025E; firmware nulls each channel at zero input at start-up; trip bands in the pin plan, asserted against sim/out/pv_control/control_spec.json. EN pair = GATE_EN AND CHB_OK AND MCU enable (74LVC11A); line drivers on only with"
Changed lines of the file:
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@@
 		)
 	)
-	(text "CHB_OK, MCU enable and RDY; EN readback on GPIO100-103. +24V_GD feeds only the cell eFuses."
+	(text "enable (74LVC11A); line drivers on only with CHB_OK, MCU enable and RDY; EN readback on GPIO100-103. +24V_GD feeds only the cell eFuses."
 		(exclude_from_sim no)
 		(at 20 240 0)
@@
 		)
 	)
-	(text "INPUTXBAR6 -> TRIP6. CMPSS reference = VDAC = REF5025E; firmware nulls each channel at zero input at start-up; trip bands in the pin plan, asserted against sim/out/pv_control/control_spec.json. EN pair = GATE_EN AND CHB_OK AND MCU enable (74LVC11A); line drivers on only with"
+	(text "INPUTXBAR6 -> TRIP6. CMPSS reference = VDAC = REF5025E; firmware nulls each channel at zero input at start-up; trip bands in the pin plan, asserted against the frozen earlier-platform snapshot gen/data/control_spec_platform1.json (D-044). EN pair = GATE_EN AND CHB_OK AND MCU"
 		(exclude_from_sim no)
 		(at 20 236 0)
