File: hardware/PV-PORT-180/sheets/04_portB_power.kicad_sch (KiCad schematic)
At the start: 122 parts, among them J401 DC terminal + (CUSTOM), J402 DC terminal - (CUSTOM), J403 KF2EDGR-3.5-2P, J404 7461057, J405 7461057, J406 7461057, K401 B88269X7340C011, K402 B88269X7340C011, K403 G7L-2A-X DC24, Q401 IRFL214TRPbF, Q402 IRFL214TRPbF, Q403 BSS138BK, Q404 IRFR9214TRPbF, Q405 IRFL214TRPbF, Q406 IRFL214TRPbF, Q407 BSS138BK, Q408 BSS138BK, Q409 IRFL214TRPbF, Q410 C2M1000170D, Q411 BSS138BK, Q412 MMBT3906-7-F, Q413 MMBT3906-7-F, Q414 MMBT3904,215, U401 CNY65B, U402 TPSI3050QDWZRQ1, X401 006710340, X402 006710340, X403 006710340, X404 006710340

Commit message: Resolve the independent PCM review of 033d8d8 (PCM-01..27): verify, classify, fix at the root (D-065..D-072)
Register gen/data/review_pcm.csv: 27 findings, each verified before a change - 21 Confirmed, 2 Firmware
Handled, 3 Improvement Recommended, 1 Not Applicable; 20 closed, 7 open with their closing path.

PV family (D-065, D-072): the 45 A port rating no longer clamps the inductor current in the near-unity
band (inductor rating 47.7 A there; 550/550 V 73.3 kW; rated power from 562 V); control model re-based on
the drawn boards with a published delivered-power envelope per product and direction; leg commutation
re-run on the drawn Jianghai capacitors (1374 V worst vs 1445 V); comparator common-mode term in every
trip band (window 67.9-80.5 A, the 1.10 margin rule missed by 0.58 A and left open; firmware OV derived
from the drawn band, 1034 V); one fan-supply contract; cold-start passive-power restriction modelled;
port A interface declared; aux pull-in and retry rules.

PCS-P125 (D-066, D-067): control study sim/pcs_control.py (PR current loop 1750 Hz, PM >= 48.7 deg to
SCR 5 with the passive damping branch, PLL, DC-link loop, grid forming, state machine); DC-link inventory
409.4 uF with bleeders, precharge rating and the 15 min label re-derived; upper-half limit in firmware;
P-Q-Vdc-Vac envelope (AC-02's 600 V full-load figure not reachable at a +15 % grid: owner's decision);
R_DS(on) acceptance rule for the six paralleled devices; DESAT string 3 -> 2 diodes (band 6.41-9.37 V);
fuse-contactor coordination bands and installation requirements; phase-current sensor frozen to Sinomags
STK-250HO/4 and the control-board ladders re-valued; Al2O3 pad text.

DAB-D60 (D-068): study vs drawn-board identity made explicit; short-circuit chain corrected (energy-
equivalent 0.99 x the assumed withstand; release block t_SC >= 2.22 us / E_SC >= 2.18 J); admitted map
follows the 1200 V deck envelope (900-950 V rows derated until a double-pulse test); zero/light-load policy;
0.41 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
Parts:
- D408: Manufacturer Bourns -> MDD (Microdiode Semiconductor)
Changed lines of the file:
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@@
 			)
 		)
-		(property "Datasheet" "docs/datasheets/protection/SMBJ_Bourns.pdf"
+		(property "Datasheet" "docs/datasheets/protection/MDD-SMBJ-series.pdf"
 			(at 535.94 175.26 0)
 			(hide yes)
@@
 			)
 		)
-		(property "Manufacturer" "Bourns"
+		(property "Manufacturer" "MDD (Microdiode Semiconductor)"
 			(at 535.94 175.26 0)
 			(hide yes)
