File: hardware/PCS-PWR/sheets/01_pc.kicad_sch (KiCad schematic)
At the start: 45 parts, among them J101 X9555WV-2x32-6TV01, J102 X9555WV-2x08-6TV01, U101 SN74AHCT1G08DBVR, U102 SN74AHCT1G08DBVR, U103 SN74AHCT1G08DBVR, U104 SN74AHCT1G08DBVR, U105 SN74AHCT1G08DBVR, U106 SN74AHCT1G08DBVR, U107 SN74AHCT1G08DBVR, U108 SN74AHCT1G08DBVR, U109 SN74AHCT1G08DBVR

Commit message: Megarevo module parity: four-wire inverter, AC-side start-up, Ethernet and recorder on the control board, aux rev A3 (D-073..D-077)
- D-073 parity policy and register (modules only; PMA0125 and PMD-75-G3 sheets, PMA manual notes, catalogue 2026 manifest row)
- D-074 PCS-PWR-4W + PCS-CTL-4W = PCS-P125-4W drawn (fourth leg, L_N, 4-pole AC port, VGN, IL4), AC start-up tap and
  AC precharge on both builds, 30 firmware rows, declarations (kVA tiers, AC short-circuit coordination, airflow, precision)
- D-075 control board: CH9121T Ethernet bridge over CA-IS3842HW (fitted on PCS-CTL), GD25Q32E recorder flash replacing the
  EEPROM, chainable stop / ready / battery-fault inputs and HFD27 ready relay, port roles, altitude 2,000 m with the 15 mm
  isolator option specified, SELV logic allocation 2.2 W
- D-076 AUX-75 rev A3: live 30 W / 48 W for 1 s, one design for every module (turns 50:9:10, sense 3 x 0.866 ohm), four-wire
  DC precharge drawn at 200 ohm; D-077 control study: off-grid secondary restoration, THDu, imbalance, ride-through limiter
  with the stiff-grid derating rule, neutral-leg loop
- sim/compare_megarevo_pcs.py: PCS-P125 / PCS-P125-4W against the PMA0125 (2 better, 38 meets, 4 below, 9 not assessed, 0
  pending of 53); PV comparison 2 / 24 / 3 / 5 / 0 of 34 (standby 12.7 / 22.4 W)
- pin ledger E: control-board parts, shield-pin rule, fuse and connector notes (247 parts, 191 pass, 0 fail); review register
  PCM-14 and PCM-22 closed; magnetics re-run; all 15 boards rebuilt, BOMs, costs, audits and figures regenerated; README,
  guide 01-13 and the decisions mirror updated

Co-Authored-By: Claude Fable 5.1 <noreply@anthropic.com>
Connections:
- net K_ACPRE: now reaches J101.27 (Pin_27)
- no-connect marks 13 -> 12
Other:
- note added: "Pin for pin the PV board's PC: PWM1-6 = legs a, b, c (high, low); K_A = K_AC1, K_B = K_DC, K_PRE. IA, IA_H, VAX held at VMID; PWM7-15, NTC4, NTC8 not connected (three-wire); PWM16 = K_ACPRE; IL4 / IL4R = 0 V."
- note removed: "Pin for pin the PV board's PC: PWM1-6 = legs a, b, c (high, low); K_A = K_AC1, K_B = K_DC, K_PRE. IA, IA_H, VAX held at VMID; PWM7-16, NTC4, NTC8 not connected (three-wire); IL4 / IL4R = 0 V."
- moved on the sheet: C101, C102, J102, R101, R102, R103, R104, R105, R106, R107, R108, R109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
