File: hardware/PCS-PWR/sheets/12_filta.kicad_sch (KiCad schematic)
At the start: 25 parts, among them J1201 7461057, J1202 7461057, J1203 7461057, J1204 7461057, J1205 7461057, J1206 7461057, J1207 7461057, J1208 7461057, J1209 7461057, J1210 7461057, J1211 7461057, J1212 7461057, J1213 7461057

Commit message: Resolve the independent PCM review of 033d8d8 (PCM-01..27): verify, classify, fix at the root (D-065..D-072)
Register gen/data/review_pcm.csv: 27 findings, each verified before a change - 21 Confirmed, 2 Firmware
Handled, 3 Improvement Recommended, 1 Not Applicable; 20 closed, 7 open with their closing path.

PV family (D-065, D-072): the 45 A port rating no longer clamps the inductor current in the near-unity
band (inductor rating 47.7 A there; 550/550 V 73.3 kW; rated power from 562 V); control model re-based on
the drawn boards with a published delivered-power envelope per product and direction; leg commutation
re-run on the drawn Jianghai capacitors (1374 V worst vs 1445 V); comparator common-mode term in every
trip band (window 67.9-80.5 A, the 1.10 margin rule missed by 0.58 A and left open; firmware OV derived
from the drawn band, 1034 V); one fan-supply contract; cold-start passive-power restriction modelled;
port A interface declared; aux pull-in and retry rules.

PCS-P125 (D-066, D-067): control study sim/pcs_control.py (PR current loop 1750 Hz, PM >= 48.7 deg to
SCR 5 with the passive damping branch, PLL, DC-link loop, grid forming, state machine); DC-link inventory
409.4 uF with bleeders, precharge rating and the 15 min label re-derived; upper-half limit in firmware;
P-Q-Vdc-Vac envelope (AC-02's 600 V full-load figure not reachable at a +15 % grid: owner's decision);
R_DS(on) acceptance rule for the six paralleled devices; DESAT string 3 -> 2 diodes (band 6.41-9.37 V);
fuse-contactor coordination bands and installation requirements; phase-current sensor frozen to Sinomags
STK-250HO/4 and the control-board ladders re-valued; Al2O3 pad text.

DAB-D60 (D-068): study vs drawn-board identity made explicit; short-circuit chain corrected (energy-
equivalent 0.99 x the assumed withstand; release block t_SC >= 2.22 us / E_SC >= 2.18 J); admitted map
follows the 1200 V deck envelope (900-950 V rows derated until a double-pulse test); zero/light-load policy;
0.41 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
Parts:
- CS1201: value CS +/-500A RFQ -> STK-250HO/4; MPN (none) -> STK-250HO/4; Manufacturer (none) -> Sinomags Technology; Package PCB mount, integrated primary bar 250 A rms -> screw mount 40.8 x 32.1 mm, aperture 15 x 8 mm busbar, 5-pi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; Sourcing RFQ -> ORDERABLE
Connections:
- net F_A: now also CS1201.P, J1204.1 (Pin_1), J1205.1 (Pin_1), J1206.1 (Pin_1), L1201.2 (B); no longer CS1201.6 (IP-)
- removed net L1O_A: CS1201.5 (IP+), J1204.1 (Pin_1), J1205.1 (Pin_1), J1206.1 (Pin_1), L1201.2 (B)
- no-connect marks 0 -> 1
Other:
- note added: "Board studs (REDCUBE press-fit, 100 A each): 3 x switch node to L1, 3 x L1 out (C_f node, its busbar through the sensor), 3 x C_f node to L2, 3 x L2 out (to AC contactor K1 on the port sheet). Cores bonded to PE."
- note added: "IL1 = Uref + 3.2 mV/A x I (I + = L1 -> C_f: body arrow, verify at incoming inspection), IL1R = its Uref pin; 100R + 1 nF each at the source (as PV-PWR). Primary = L1's output busbar through the aperture (a 50 Hz-smooth node, not the switch node). OCD (open drain, 2.93 x I_PN = 732 A +/-10 %) not used: above both IL windows and the L1 limit."
- note added: "PHASE A CURRENT SENSOR STK-250HO/4 (C_F SIDE OF L1)"
- note removed: "Board studs (REDCUBE press-fit, 100 A each): 3 x switch node to L1, 3 x L1 out, 3 x C_f node to L2, 3 x L2 out (to AC contactor K1 on the port sheet). Cores bonded to PE."
- note removed: "IL1 = Vref + G x I (I + = L1 -> C_f), IL1R = its Vref: 100R + 1 nF each at the source (as PV-PWR). The primary sits between L1 and the C_f node (a 50 Hz-smooth node, not the switch node)."
- note removed: "PHASE A CURRENT SENSOR (C_F SIDE OF L1)"
- moved on the sheet: C1201, C1202, C1203, C1204, C1205, C1206, CS1201, J1204, J1213, R1202, R1203
