File: hardware/PCS-PWR/sheets/22_supplies.kicad_sch (KiCad schematic)
At the start: 48 parts, among them J2201 KF2EDGR-3.5-2P, Q2201 PMV30ENEAR, Q2202 2N7002BK, U2201 LMR38020FDDAR, U2202 LMR38020FDDAR, U2203 TPS3710DDCR, U2204 TPS62130RGTR

Commit message: Megarevo module parity: four-wire inverter, AC-side start-up, Ethernet and recorder on the control board, aux rev A3 (D-073..D-077)
- D-073 parity policy and register (modules only; PMA0125 and PMD-75-G3 sheets, PMA manual notes, catalogue 2026 manifest row)
- D-074 PCS-PWR-4W + PCS-CTL-4W = PCS-P125-4W drawn (fourth leg, L_N, 4-pole AC port, VGN, IL4), AC start-up tap and
  AC precharge on both builds, 30 firmware rows, declarations (kVA tiers, AC short-circuit coordination, airflow, precision)
- D-075 control board: CH9121T Ethernet bridge over CA-IS3842HW (fitted on PCS-CTL), GD25Q32E recorder flash replacing the
  EEPROM, chainable stop / ready / battery-fault inputs and HFD27 ready relay, port roles, altitude 2,000 m with the 15 mm
  isolator option specified, SELV logic allocation 2.2 W
- D-076 AUX-75 rev A3: live 30 W / 48 W for 1 s, one design for every module (turns 50:9:10, sense 3 x 0.866 ohm), four-wire
  DC precharge drawn at 200 ohm; D-077 control study: off-grid secondary restoration, THDu, imbalance, ride-through limiter
  with the stiff-grid derating rule, neutral-leg loop
- sim/compare_megarevo_pcs.py: PCS-P125 / PCS-P125-4W against the PMA0125 (2 better, 38 meets, 4 below, 9 not assessed, 0
  pending of 53); PV comparison 2 / 24 / 3 / 5 / 0 of 34 (standby 12.7 / 22.4 W)
- pin ledger E: control-board parts, shield-pin rule, fuse and connector notes (247 parts, 191 pass, 0 fail); review register
  PCM-14 and PCM-22 closed; magnetics re-run; all 15 boards rebuilt, BOMs, costs, audits and figures regenerated; README,
  guide 01-13 and the decisions mirror updated

Co-Authored-By: Claude Fable 5.1 <noreply@anthropic.com>
Other:
- note added: "AUX-T1 reinforced winding SELV_24V / SELV_0V, cross-regulated 21.4-30.1 V (aux75_spec); full fan speed needs 24.5 V. Full fan speed is only guaranteed while the converter is switching. Fan buck (12-36 V in) + SELV logic on the control board; >= 10 mm from live copper; nothing else of the SELV domain is on this board."
- note removed: "AUX-T1 reinforced winding SELV_24V / SELV_0V, cross-regulated 20.3-29.8 V (aux75_spec); full fan speed needs 24.5 V. Full fan speed is only guaranteed while the converter is switching. Fan buck (12-36 V in) + SELV logic on the control board; >= 10 mm from live copper; nothing else of the SELV domain is on this board."
Changed lines of the file:
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@@
 	(title_block
 		(title "PCS-P125 power - Live 5 V / 3.3 V, SELV connector")
-		(date "2026-10-05")
+		(date "2026-10-06")
 		(rev "A0")
 		(comment 1 "Live board referenced to DC-; gate islands functional; HV-PE basic")
@@
 		)
 	)
-	(text "AUX-T1 reinforced winding SELV_24V / SELV_0V, cross-regulated 20.3-29.8 V (aux75_spec); full fan speed needs\n24.5 V. Full fan speed is only guaranteed while the converter is switching. Fan buck (12-36 V in) + SELV logic on the control board;\n>= 10 mm from live copper; nothing else of the SELV domain is on this board."
+	(text "AUX-T1 reinforced winding SELV_24V / SELV_0V, cross-regulated 21.4-30.1 V (aux75_spec); full fan speed needs\n24.5 V. Full fan speed is only guaranteed while the converter is switching. Fan buck (12-36 V in) + SELV logic on the control board;\n>= 10 mm from live copper; nothing else of the SELV domain is on this board."
 		(exclude_from_sim no)
 		(at 14 260.22 0)
