File: hardware/PCS-PWR/sheets/24_aux75_startup.kicad_sch (KiCad schematic)
At the start: 39 parts, among them Q2401 BSS126H6327XTSA2, Q2402 BSS126H6327XTSA2, Q2403 BSS126H6327XTSA2, Q2404 2N7002BK,215, Q2405 2N7002BK,215, U2401 TPS3710DDCR, U2402 ATL431BIDBZR, U2403 TLV3202AIDGKR

Commit message: Megarevo module parity: four-wire inverter, AC-side start-up, Ethernet and recorder on the control board, aux rev A3 (D-073..D-077)
- D-073 parity policy and register (modules only; PMA0125 and PMD-75-G3 sheets, PMA manual notes, catalogue 2026 manifest row)
- D-074 PCS-PWR-4W + PCS-CTL-4W = PCS-P125-4W drawn (fourth leg, L_N, 4-pole AC port, VGN, IL4), AC start-up tap and
  AC precharge on both builds, 30 firmware rows, declarations (kVA tiers, AC short-circuit coordination, airflow, precision)
- D-075 control board: CH9121T Ethernet bridge over CA-IS3842HW (fitted on PCS-CTL), GD25Q32E recorder flash replacing the
  EEPROM, chainable stop / ready / battery-fault inputs and HFD27 ready relay, port roles, altitude 2,000 m with the 15 mm
  isolator option specified, SELV logic allocation 2.2 W
- D-076 AUX-75 rev A3: live 30 W / 48 W for 1 s, one design for every module (turns 50:9:10, sense 3 x 0.866 ohm), four-wire
  DC precharge drawn at 200 ohm; D-077 control study: off-grid secondary restoration, THDu, imbalance, ride-through limiter
  with the stiff-grid derating rule, neutral-leg loop
- sim/compare_megarevo_pcs.py: PCS-P125 / PCS-P125-4W against the PMA0125 (2 better, 38 meets, 4 below, 9 not assessed, 0
  pending of 53); PV comparison 2 / 24 / 3 / 5 / 0 of 34 (standby 12.7 / 22.4 W)
- pin ledger E: control-board parts, shield-pin rule, fuse and connector notes (247 parts, 191 pass, 0 fail); review register
  PCM-14 and PCM-22 closed; magnetics re-run; all 15 boards rebuilt, BOMs, costs, audits and figures regenerated; README,
  guide 01-13 and the decisions mirror updated

Co-Authored-By: Claude Fable 5.1 <noreply@anthropic.com>
Parts:
- R2416: value 68.1k -> 73.2k
Other:
- note added: "Ch 1: OV lockout -> COMP low. Ch 2: timer divider: trips above 113 / 175 / 278 W (no trip at the 112.2 W 1 s peak); timer 39-100 ms -> latch -> SS crowbar -> hiccup."
- note removed: "Ch 1: OV lockout -> COMP low. Ch 2: timer divider: trips above 103 / 160 / 256 W (no trip at 75 W + 6 W pull-in); timer 35-80 ms -> latch -> SS crowbar -> hiccup."
Changed lines of the file:
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@@
 	(title_block
 		(title "PCS-P125 power - AUX75 start-up, brown-in, OV, timer")
-		(date "2026-10-05")
+		(date "2026-10-06")
 		(rev "A0")
 		(comment 1 "Live board referenced to DC-; gate islands functional; HV-PE basic")
@@
 		)
 	)
-	(text "Ch 1: OV lockout -> COMP low. Ch 2: timer divider: trips above 103 / 160 / 256 W (no trip at 75 W + 6 W pull-in); timer 35-80 ms -> latch -> SS crowbar -> hiccup."
+	(text "Ch 1: OV lockout -> COMP low. Ch 2: timer divider: trips above 113 / 175 / 278 W (no trip at the 112.2 W 1 s peak); timer 39-100 ms -> latch -> SS crowbar -> hiccup."
 		(exclude_from_sim no)
 		(at 163.528 172.548 0)
@@
 			)
 		)
-		(property "Value" "68.1k"
+		(property "Value" "73.2k"
 			(at 215.9 162.436 90)
 			(show_name no)
@@
 			)
 		)
-		(property "Description" "Resistor 68.1k 1% 0603"
+		(property "Description" "Resistor 73.2k 1% 0603"
 			(at 215.9 160.02 0)
 			(hide yes)
