File: hardware/PCS-PWR/sheets/25_aux75_power.kicad_sch (KiCad schematic)
At the start: 56 parts, among them Q2501 BC817-25,215, Q2502 2N7002BK,215, Q2503 2N7002BK,215, Q2504 IV2Q171R0D7Z, T2501 AUX-T1 75 W (CUSTOM), U2501 UCC28C59QDRQ1

Commit message: Megarevo module parity: four-wire inverter, AC-side start-up, Ethernet and recorder on the control board, aux rev A3 (D-073..D-077)
- D-073 parity policy and register (modules only; PMA0125 and PMD-75-G3 sheets, PMA manual notes, catalogue 2026 manifest row)
- D-074 PCS-PWR-4W + PCS-CTL-4W = PCS-P125-4W drawn (fourth leg, L_N, 4-pole AC port, VGN, IL4), AC start-up tap and
  AC precharge on both builds, 30 firmware rows, declarations (kVA tiers, AC short-circuit coordination, airflow, precision)
- D-075 control board: CH9121T Ethernet bridge over CA-IS3842HW (fitted on PCS-CTL), GD25Q32E recorder flash replacing the
  EEPROM, chainable stop / ready / battery-fault inputs and HFD27 ready relay, port roles, altitude 2,000 m with the 15 mm
  isolator option specified, SELV logic allocation 2.2 W
- D-076 AUX-75 rev A3: live 30 W / 48 W for 1 s, one design for every module (turns 50:9:10, sense 3 x 0.866 ohm), four-wire
  DC precharge drawn at 200 ohm; D-077 control study: off-grid secondary restoration, THDu, imbalance, ride-through limiter
  with the stiff-grid derating rule, neutral-leg loop
- sim/compare_megarevo_pcs.py: PCS-P125 / PCS-P125-4W against the PMA0125 (2 better, 38 meets, 4 below, 9 not assessed, 0
  pending of 53); PV comparison 2 / 24 / 3 / 5 / 0 of 34 (standby 12.7 / 22.4 W)
- pin ledger E: control-board parts, shield-pin rule, fuse and connector notes (247 parts, 191 pass, 0 fail); review register
  PCM-14 and PCM-22 closed; magnetics re-run; all 15 boards rebuilt, BOMs, costs, audits and figures regenerated; README,
  guide 01-13 and the decisions mirror updated

Co-Authored-By: Claude Fable 5.1 <noreply@anthropic.com>
Parts:
- R2514, R2515, R2516: value 0.91R -> 0.866R
Other:
- note added: "3 in parallel = 0.288667R (E96): lowest limit 3.04 A delivers 112.8 W (>= the 112.2 W 1 s peak) at every input; highest 4.07 A with the line feed-forward (4.46 A without) line feed-forward HV_BULK -> CS (CRHV2512): CS offset 101 mV at 1000 V cancels most of the 155-250 ns CS-delay overshoot, so the highest current limit no longer rises with the input Clamp: BYG10Y + 6 x SMCJ33A; V_DS 1318 / 1422 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"
- note added: "live 24 V into FB: 23.62 / 24.15 / 24.68 V (VFB 2.45-2.55 V, 0.1 %) type II: mid-band gain 4.0; crossover 259-727 Hz, phase margin >= 60 deg type II zero 139 Hz type II pole 3811 Hz"
- note removed: "3 in parallel = 0.303333R: lowest limit 2.90 A delivers 103 W (>= 110 % of 75 W) at every input; highest 3.91 A with the line feed-forward (4.27 A without) line feed-forward HV_BULK -> CS (CRHV2512): CS offset 101 mV at 1000 V cancels most of the 155-250 ns CS-delay overshoot, so the highest current limit no longer rises with the input Clamp: BYG10Y + 6 x SMCJ33A; V_DS 1316 / 1420 V at 1000 / 110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"
- note removed: "live 24 V into FB: 23.62 / 24.15 / 24.68 V (VFB 2.45-2.55 V, 0.1 %) type II: mid-band gain 4.0; crossover 241-667 Hz, phase margin >= 58 deg type II zero 139 Hz type II pole 3811 Hz"
Changed lines of the file:
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@@
 	(title_block
 		(title "PCS-P125 power - AUX75 PWM, SiC, clamp, AUX-T1")
-		(date "2026-10-05")
+		(date "2026-10-06")
 		(rev "A0")
 		(comment 1 "Live board referenced to DC-; gate islands functional; HV-PE basic")
@@
 		)
 	)
-	(text "3 in parallel = 0.303333R: lowest limit 2.90 A delivers 103 W (>= 110 % of 75 W) at every input; highest 3.91 A with the line feed-forward (4.27 A without)\nline feed-forward HV_BULK -> CS (CRHV2512): CS offset 101 mV at 1000 V cancels most of the 155-250 ns CS-delay overshoot, so the highest current limit no longer rises with the input\nClamp: BYG10Y + 6 x SMCJ33A; V_DS 1316 / 1420 V at 1000 / 1100 V."
+	(text "3 in parallel = 0.288667R (E96): lowest limit 3.04 A delivers 112.8 W (>= the 112.2 W 1 s peak) at every input; highest 4.07 A with the line feed-forward (4.46 A without)\nline feed-forward HV_BULK -> CS (CRHV2512): CS offset 101 mV at 1000 V cancels most of the 155-250 ns CS-delay overshoot, so the highest current limit no longer rises with the input\nClamp: BYG10Y + 6 x SMCJ33A; V_DS 1318 / 1422 V at 1000 / 1100 V."
 		(exclude_from_sim no)
 		(at 14 231.69 0)
@@
 		)
 	)
-	(text "live 24 V into FB: 23.62 / 24.15 / 24.68 V (VFB 2.45-2.55 V, 0.1 %)\ntype II: mid-band gain 4.0; crossover 241-667 Hz, phase margin >= 58 deg type II zero 139 Hz type II pole 3811 Hz"
+	(text "live 24 V into FB: 23.62 / 24.15 / 24.68 V (VFB 2.45-2.55 V, 0.1 %)\ntype II: mid-band gain 4.0; crossover 259-727 Hz, phase margin >= 60 deg type II zero 139 Hz type II pole 3811 Hz"
 		(exclude_from_sim no)
 		(at 14 139.902 0)
@@
 			)
 		)
-		(property "Value" "0.91R"
+		(property "Value" "0.866R"
 			(at 27.94 190.376 90)
 			(show_name no)
@@
 			)
 		)
-		(property "Description" "Resistor 0.91R 1% 1206"
+		(property "Description" "Resistor 0.866R 1% 1206"
 			(at 27.94 187.96 0)
 			(hide yes)
@@
 			)
 		)
-		(property "Description" "CUSTOM AUX-T1 75 W rev M1: DMEGC EC39A DMR95 (ETD39 class), centre-leg gap 1.05 mm, 48:8 live:9 SELV in the order P1 | SH | SELV (TIW-litz) | LIVE | P2, copper set back 2.0 mm from the gapped leg, vacuum-potted case; electrical requirement in sim/out/aux_hv_design/aux75_spec.json"
+		(property "Description" "CUSTOM AUX-T1 75 W rev M1: DMEGC EC39A DMR95 (ETD39 class), centre-leg gap 1.17 mm, 50:9 live:10 SELV in the order P1 | SH | SELV (TIW-litz) | LIVE | P2, copper set back 2.0 mm from the gapped leg, vacuum-potted case; electrical requirement in sim/out/aux_hv_design/aux75_spec.json"
 			(at 223.52 170.18 0)
 			(hide yes)
@@
 			)
 		)
-		(property "Value" "0.91R"
+		(property "Value" "0.866R"
 			(at 172.72 162.436 90)
 			(show_name no)
@@
 			)
 		)
-		(property "Description" "Resistor 0.91R 1% 1206"
+		(property "Description" "Resistor 0.866R 1% 1206"
 			(at 172.72 160.02 0)
 			(hide yes)
@@
 			)
 		)
-		(property "Value" "0.91R"
+		(property "Value" "0.866R"
 			(at 142.24 162.436 90)
 			(show_name no)
@@
 			)
 		)
-		(property "Description" "Resistor 0.91R 1% 1206"
+		(property "Description" "Resistor 0.866R 1% 1206"
 			(at 142.24 160.02 0)
 			(hide yes)
