File: hardware/PCS-PWR/sheets/03_lega.kicad_sch (KiCad schematic)
At the start: 57 parts, among them P301 PAD Al2O3 0.635 mm (CUSTOM), P302 PAD Al2O3 0.635 mm (CUSTOM), P303 PAD Al2O3 0.635 mm (CUSTOM), P304 PAD Al2O3 0.635 mm (CUSTOM), P305 PAD Al2O3 0.635 mm (CUSTOM), P306 PAD Al2O3 0.635 mm (CUSTOM), P307 PAD Al2O3 0.635 mm (CUSTOM), P308 PAD Al2O3 0.635 mm (CUSTOM), P309 PAD Al2O3 0.635 mm (CUSTOM), P310 PAD Al2O3 0.635 mm (CUSTOM), P311 PAD Al2O3 0.635 mm (CUSTOM), P312 PAD Al2O3 0.635 mm (CUSTOM), Q301 SG2M040170HJ, Q302 SG2M040170HJ, Q303 SG2M040170HJ, Q304 SG2M040170HJ, Q305 SG2M040170HJ, Q306 SG2M040170HJ, Q307 SG2M040170HJ, Q308 SG2M040170HJ, Q309 SG2M040170HJ, Q310 SG2M040170HJ, Q311 SG2M040170HJ, Q312 SG2M040170HJ

Commit message: Resolve the independent PCM review of 033d8d8 (PCM-01..27): verify, classify, fix at the root (D-065..D-072)
Register gen/data/review_pcm.csv: 27 findings, each verified before a change - 21 Confirmed, 2 Firmware
Handled, 3 Improvement Recommended, 1 Not Applicable; 20 closed, 7 open with their closing path.

PV family (D-065, D-072): the 45 A port rating no longer clamps the inductor current in the near-unity
band (inductor rating 47.7 A there; 550/550 V 73.3 kW; rated power from 562 V); control model re-based on
the drawn boards with a published delivered-power envelope per product and direction; leg commutation
re-run on the drawn Jianghai capacitors (1374 V worst vs 1445 V); comparator common-mode term in every
trip band (window 67.9-80.5 A, the 1.10 margin rule missed by 0.58 A and left open; firmware OV derived
from the drawn band, 1034 V); one fan-supply contract; cold-start passive-power restriction modelled;
port A interface declared; aux pull-in and retry rules.

PCS-P125 (D-066, D-067): control study sim/pcs_control.py (PR current loop 1750 Hz, PM >= 48.7 deg to
SCR 5 with the passive damping branch, PLL, DC-link loop, grid forming, state machine); DC-link inventory
409.4 uF with bleeders, precharge rating and the 15 min label re-derived; upper-half limit in firmware;
P-Q-Vdc-Vac envelope (AC-02's 600 V full-load figure not reachable at a +15 % grid: owner's decision);
R_DS(on) acceptance rule for the six paralleled devices; DESAT string 3 -> 2 diodes (band 6.41-9.37 V);
fuse-contactor coordination bands and installation requirements; phase-current sensor frozen to Sinomags
STK-250HO/4 and the control-board ladders re-valued; Al2O3 pad text.

DAB-D60 (D-068): study vs drawn-board identity made explicit; short-circuit chain corrected (energy-
equivalent 0.99 x the assumed withstand; release block t_SC >= 2.22 us / E_SC >= 2.18 J); admitted map
follows the 1200 V deck envelope (900-950 V rows derated until a double-pulse test); zero/light-load policy;
0.41 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
Other:
- note added: "Per device: own gate net G_AH<k> and Kelvin net KS_AH<k> (gate network on the gate-drive sheet). BOM NOTE: R_DS(on) of the six within +/-5 % (V_GS 18 V, 38 A, 25 C), V_GS(th) within +/-0.25 V, one lot per switch (pcs_spec device_acceptance, PCM-06)."
- note added: "Per device: own gate net G_AL<k> and Kelvin net KS_AL<k> (gate network on the gate-drive sheet). BOM NOTE: R_DS(on) of the six within +/-5 % (V_GS 18 V, 38 A, 25 C), V_GS(th) within +/-0.25 V, one lot per switch (pcs_spec device_acceptance, PCM-06)."
- note removed: "Per device: own gate net G_AH<k> and Kelvin net KS_AH<k> (gate network on the gate-drive sheet). BOM NOTE: one lot per switch, V_GS(th) binned to +/-0.25 V or a sharing test at incoming inspection (crosscheck_wolfspeed.md claim 5)."
- note removed: "Per device: own gate net G_AL<k> and Kelvin net KS_AL<k> (gate network on the gate-drive sheet). BOM NOTE: one lot per switch, V_GS(th) binned to +/-0.25 V or a sharing test at incoming inspection (crosscheck_wolfspeed.md claim 5)."
- moved on the sheet: C301, C302, C303, C304, C305, C306, C307, C308, C309, C310, C311, C312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
