File: hardware/PCS-PWR/sheets/11_gdcl.kicad_sch (KiCad schematic)
At the start: 170 parts, among them Q1101 PMV30ENEAR, Q1102 PMV30ENEAR, Q1103 PMV30ENEAR, Q1104 PMV30ENEAR, Q1105 PMV30ENEAR, Q1106 PMV30ENEAR, Q1107 PMV30ENEAR, Q1108 ZXTP25040DFHTA, Q1109 ZXTP25040DFHTA, Q1110 ZXTP25040DFHTA, Q1111 ZXTN25040DFHTA, Q1112 MMBT3904,215, Q1113 MMBT3906,215, Q1114 MMBT3904,215, Q1115 PBSS5540X,135, Q1116 PBSS5540X,135, T1101 Gate-bias transformer per pha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, U1101 SN74LVC1G17DBVR, U1102 NSI6651ASC-Q1SWR, U1103 SN6505BDBVR, U1104 ATL431BIDBZR, U1105 ATL431BIDBZR, U1106 ATL431BIDBZR, U1107 ATL431BIDBZR

Commit message: Resolve the independent PCM review of 033d8d8 (PCM-01..27): verify, classify, fix at the root (D-065..D-072)
Register gen/data/review_pcm.csv: 27 findings, each verified before a change - 21 Confirmed, 2 Firmware
Handled, 3 Improvement Recommended, 1 Not Applicable; 20 closed, 7 open with their closing path.

PV family (D-065, D-072): the 45 A port rating no longer clamps the inductor current in the near-unity
band (inductor rating 47.7 A there; 550/550 V 73.3 kW; rated power from 562 V); control model re-based on
the drawn boards with a published delivered-power envelope per product and direction; leg commutation
re-run on the drawn Jianghai capacitors (1374 V worst vs 1445 V); comparator common-mode term in every
trip band (window 67.9-80.5 A, the 1.10 margin rule missed by 0.58 A and left open; firmware OV derived
from the drawn band, 1034 V); one fan-supply contract; cold-start passive-power restriction modelled;
port A interface declared; aux pull-in and retry rules.

PCS-P125 (D-066, D-067): control study sim/pcs_control.py (PR current loop 1750 Hz, PM >= 48.7 deg to
SCR 5 with the passive damping branch, PLL, DC-link loop, grid forming, state machine); DC-link inventory
409.4 uF with bleeders, precharge rating and the 15 min label re-derived; upper-half limit in firmware;
P-Q-Vdc-Vac envelope (AC-02's 600 V full-load figure not reachable at a +15 % grid: owner's decision);
R_DS(on) acceptance rule for the six paralleled devices; DESAT string 3 -> 2 diodes (band 6.41-9.37 V);
fuse-contactor coordination bands and installation requirements; phase-current sensor frozen to Sinomags
STK-250HO/4 and the control-board ladders re-valued; Al2O3 pad text.

DAB-D60 (D-068): study vs drawn-board identity made explicit; short-circuit chain corrected (energy-
equivalent 0.99 x the assumed withstand; release block t_SC >= 2.22 us / E_SC >= 2.18 J); admitted map
follows the 1200 V deck envelope (900-950 V rows derated until a double-pulse test); zero/light-load policy;
0.41 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
Parts:
- removed D1138: PMEG4010CEJ, symbol dcdc:PMEG4010CEJ
- D1130: value US1MH -> PMEG4010CEJ; symbol dcdc:US1M -> dcdc:PMEG4010CEJ; Domain CROSSING -> GD_CH; MPN US1MH -> PMEG4010CEJ; Manufacturer Taiwan Semiconductor -> Nexperia; Package SMA (DO-214AC) -> SOD-323F
- D1134: Domain GD_CH -> GD_CL
Connections:
- net RAW_PHCCH: now also D1130.1 (K); no longer D1132.1 (K)
- net RAW_PHCCL: now also D1134.1 (K); no longer D1136.1 (K)
- net SA_PHCCH: now also D1130.2 (A), D1132.1 (K); no longer D1131.2 (A), D1133.1 (K)
- net SA_PHCCL: now also D1134.2 (A), D1136.1 (K); no longer D1135.2 (A), D1137.1 (K)
- net SB_PHCCH: now also D1131.2 (A), D1133.1 (K); no longer D1132.2 (A), D1134.1 (K)
- net SB_PHCCL: now also D1135.2 (A), D1137.1 (K); no longer D1136.2 (A)
- net SW_C: now also D1129.1 (K); no longer D1130.1 (K)
- net VEE_CH: now also D1132.2 (A); no longer D1134.2 (A)
- net VEE_CL: now also D1136.2 (A)
- removed net DS2_CL: D1129.1 (K), D1130.2 (A)
Other:
- note added: "DESAT > 10.3-10.9 V (above the 10.0 V maximum trip of the -Q1 grade) -> MMBT3904 -> MMBT3906 charges BG to VEE + 10 V; per device AO3400A + 22R pull the gate to VEE; BG holds ~3 us (1k + FET gates)."
- note added: "DESAT pin (internal 500 uA blanking source, trip 8.5-10.0 V) - Rs - 2 x US1M - drain. BAT54S keeps DX between COM and VDD against dv/dt through the string; Cblk footprint DNP."
- note removed: "DESAT > 10.3-10.9 V (above the 9.8 V maximum trip) -> MMBT3904 -> MMBT3906 charges BG to VEE + 10 V; per device AO3400A + 22R pull the gate to VEE; BG holds ~3 us (1k + FET gates)."
- note removed: "DESAT pin (internal 500 uA blanking source, trip 8.5-9.8 V) - Rs - 3 x US1M - drain. BAT54S keeps DX between COM and VDD against dv/dt through the string; Cblk footprint DNP."
- moved on the sheet: D1124, D1125, D1130, D1131, D1132, D1133, D1134, D1135, D1136, D1137, R1153, R1154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

Commit message: Respond to the independent re-check R2 of a427981 (D-078, D-079): gates-off commutation closed, backup band lowered, SiC acceptance, bounded grid-forming transients, ride-through without derating, AC-start repairs, installation requirements
- Register gen/data/review_r2.csv: 14 findings verified and dispositioned (9 Confirmed, 1 Firmware Handled,
  1 Improvement Recommended, 2 Already Fixed, 1 Not Applicable), every row closed with its evidence
- D-078 power stage: the discrete window turns the gates off at 520.8 A, not at the 485.5 A window top; the leg deck
  at that current peaked at 1457 V against 1445 V, closed at zero cost by R_G,off 7.5 -> 8.75 ohm (1437 V, admissible
  533.6 A); L1 inductance trajectory to 700 A (knee 566 A), CMPSS backup band lowered to 423.9-497.5 A on PCS-CTL,
  firmware OV backup 1035 V; R_DS(on) <= 40 mOhm acceptance with per-lot derating; one coil contract (20 W / 4 W);
  residual-current monitor contract; docs/requirements/INSTALLATION.md (74 enforceable requirements with sources)
- D-079 control study: tolerance regression at the assembly tolerances (1,944 + 1,000 cases, worst PM 48.1 deg);
  bounded grid-forming transients 0.43 / 1.77 pu with feed-forward and OV deadbeat (2.17 pu superseded), trip-aware
  DC-load rejection, CV-mode soft-OV hold, weak-grid CV power limits, PV DC-bus coordination row (0.51 ms);
  ride-through 270 A clamp with C_f prediction removes the stiff-grid derating (fallback kept, SCR estimator,
  8.07 MVA declaration); coupled four-wire cases; AC start in the executable state machine (17 states, 35 fault
  cases) with the five sequence holes H1-H5 repaired and an own AC_STOP state
- pcs_spec protection_chain published and read by the control study and the control board; all 15 boards, BOMs,
  costs, comparisons (PV 2/24/3/5/0, PCS 2/38/4/9/0), audits and figures regenerated; README, guide 03-13,
  decisions mirror and architecture reconciliation notes updated; .graphifyignore and graphify-out/ ignored

Co-Auth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
Parts:
- R1109, R1115, R1121, R1127, R1133, R1139: value 7.5R -> 8.75R
Changed lines of the file:
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@@
 			)
 		)
-		(property "Value" "7.5R"
+		(property "Value" "8.75R"
 			(at 335.28 131.956 90)
 			(show_name no)
@@
 			)
 		)
-		(property "Description" "Resistor 7.5R 1% 2512 Roff, pulse-rated thick film 1 W"
+		(property "Description" "Resistor 8.75R 1% 2512 Roff, pulse-rated thick film 1 W"
 			(at 335.28 129.54 0)
 			(hide yes)
@@
 			)
 		)
-		(property "Value" "7.5R"
+		(property "Value" "8.75R"
 			(at 149.86 93.856 90)
 			(show_name no)
@@
 			)
 		)
-		(property "Description" "Resistor 7.5R 1% 2512 Roff, pulse-rated thick film 1 W"
+		(property "Description" "Resistor 8.75R 1% 2512 Roff, pulse-rated thick film 1 W"
 			(at 149.86 91.44 0)
 			(hide yes)
@@
 			)
 		)
-		(property "Value" "7.5R"
+		(property "Value" "8.75R"
 			(at 381 68.456 90)
 			(show_name no)
@@
 			)
 		)
-		(property "Description" "Resistor 7.5R 1% 2512 Roff, pulse-rated thick film 1 W"
+		(property "Description" "Resistor 8.75R 1% 2512 Roff, pulse-rated thick film 1 W"
 			(at 381 66.04 0)
 			(hide yes)
@@
 			)
 		)
-		(property "Value" "7.5R"
+		(property "Value" "8.75R"
 			(at 208.28 106.556 90)
 			(show_name no)
@@
 			)
 		)
-		(property "Description" "Resistor 7.5R 1% 2512 Roff, pulse-rated thick film 1 W"
+		(property "Description" "Resistor 8.75R 1% 2512 Roff, pulse-rated thick film 1 W"
 			(at 208.28 104.14 0)
 			(hide yes)
@@
 			)
 		)
-		(property "Value" "7.5R"
+		(property "Value" "8.75R"
 			(at 271.78 119.256 90)
 			(show_name no)
@@
 			)
 		)
-		(property "Description" "Resistor 7.5R 1% 2512 Roff, pulse-rated thick film 1 W"
+		(property "Description" "Resistor 8.75R 1% 2512 Roff, pulse-rated thick film 1 W"
 			(at 271.78 116.84 0)
 			(hide yes)
@@
 			)
 		)
-		(property "Value" "7.5R"
+		(property "Value" "8.75R"
 			(at 396.24 144.656 90)
 			(show_name no)
@@
 			)
 		)
-		(property "Description" "Resistor 7.5R 1% 2512 Roff, pulse-rated thick film 1 W"
+		(property "Description" "Resistor 8.75R 1% 2512 Roff, pulse-rated thick film 1 W"
 			(at 396.24 142.24 0)
 			(hide yes)

Commit message: Respond to the independent economical re-check R4 of 845131d (D-081): DESAT string re-rated to 1300 V diodes, cable-aware DC-bus window enforced, off-grid envelope stated as declared capability, inverter cold rating -10 C, grade-B rating stated, magnetics RFQ index
- Register gen/data/review_r4.csv: 12 decision areas closed (3 Confirmed, 4 Already Fixed, 3 Improvement Recommended, 2 Not Applicable)
- E01: the DESAT sense string sees the whole DC link (static envelope 1130 V) on an off switch; 2 x Vishay BYG23T-M3/TR (1300 V)
  per channel on both presets, each diode blocking the envelope alone; PCS window unchanged, PV preset 3 -> 2 diodes; grade
  tables identical; +0.96 to +2.12 USD per module at 5k; datasheet, prices, ledger rows, insulation table
- E04: inter-module cable in the coupled PCS/PV bus model (+28 V); product rule default set point 750 V (755 V four-wire mode A),
  782 V firmware clamp in the PV module, PCS refuses an island start above 791 V, 909 V recorded as model validity; harness contract
- E06: AC-04 reworded as the module's declared output capability with the release sequence (grid-following first)
- E11: PCS cold-start passive table modelled; rating full operation from -10 C inlet (AC-02 amended by delegation), cold fan RFQ open
- E05: grade-B rating 124.57 kW at PF 1 stated; E12: docs/requirements/RFQ-MAGNETICS.md (ten RFQs); the port CM ring's catalog
  entry set to the flat-permeability grade and the aux transformer's thermal test to the 94.2 W rating
- All 15 boards, BOMs, costs, comparisons (PV 2/24/3/5/0, PCS 2/38/4/9/0), audits (pin 192/0/55, insulation 98 known) and figures
  regenerated; README, guide 01-13, INSTALLATION.md (77 rows), decisions mirror and the registers updated

Co-Authored-By: Claude Fable 5.1 <noreply@anthropic.com>
Parts:
- D1128, D1129: value US1MH -> BYG23T-M3/TR; symbol dcdc:US1M -> dcdc:BYG23T; MPN US1MH -> BYG23T-M3/TR; Manufacturer Taiwan Semiconductor -> Vishay
Other:
- note added: "DESAT pin (internal 500 uA blanking source, trip 8.5-10.0 V) - Rs - 2 x BYG23T-M3/TR (1300 V each) - drain. BAT54S keeps DX between COM and VDD against dv/dt through the string; Cblk footprint DNP."
- note removed: "DESAT pin (internal 500 uA blanking source, trip 8.5-10.0 V) - Rs - 2 x US1M - drain. BAT54S keeps DX between COM and VDD against dv/dt through the string; Cblk footprint DNP."
- moved on the sheet: C1125, C1126, C1127, C1128, C1129, C1130, C1131, C1132, D1127, D1128, D1129, D1130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
