File: hardware/PV-CTL/PV-CTL.kicad_sch (KiCad schematic)
At the start: 0 parts

Commit message: Board revisions PV-PWR A2 / PV-CTL A1, inverter filter magnetics, documentation refresh (D-056..D-058)
Boards (every build check passes)
- PV-PWR / PV-PWR-4 rev A2: seventh battery-side film capacitor on the three-phase board (closes the
  load-rejection overshoot), bleeder 8 x 73.2 k so the bank still discharges within its 10-minute label.
- PV-CTL rev A1: hardware over-current window 68.9-79.9 A, thresholds derived from each sensor's own
  reference; the board-to-board contract carries the four references on the former 24 V / 5 V pins.
- Records aligned (contract comments, architecture corrections, port-current bandwidth); the frozen
  platform's module BOMs are kept instead of being re-rolled from the cost-first thermal data.

Magnetics
- Inverter filter designed and verified: L1, L2 and the AC common-mode choke (design_pcs_*.json). The filter
  comes to 745 USD at catalogue prices and 611 USD at 5,000 units, against 207 / 167 in the study: the
  inverter's cost is provisional and its stage and filter are being re-optimised.
- PV inductor loss check made non-circular; hot-spot margin reported per build (PV-P100/110: -5.3 K, MG-17).

Results: PV-P75 952 USD at catalogue prices / 796 USD at 5,000 units; Megarevo comparison 2 better,
24 meet, 3 below, 5 not assessed. Documentation corrected for the revised boards (51 statements).
Everything is calculated or estimated; nothing is bench-validated.

Co-Authored-By: Claude Fable 5.1 <noreply@anthropic.com>
Other:
- note added: "7 x TLV9024 on +3V3 (open drain, no firmware): IL windows from each sensor's Uref; VA / VB over-voltage, NTC over-temperature and open probe from VREF ladders"
- note added: "Rev A1 | 2026-10-05 | Schematics authored by Chinmoy Bhuyan | Cost-first PV-P75/100/110 controller: F280039C on BUS-, one trip latch, one SELV barrier"
- note removed: "7 x TLV9024 on +3V3 (open drain, rail-to-rail inputs, no firmware): IL windows, VA / VB over-voltage, NTC over-temperature and open probe; ladders from VREF"
- note removed: "Rev A0 | 2026-10-04 | Schematics authored by Chinmoy Bhuyan | Cost-first PV-P75/100/110 controller: F280039C on BUS-, one trip latch, one SELV barrier"
Changed lines of the file:
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@@
 	(title_block
 		(title "PV-CTL control board - Cover / Hierarchy")
-		(date "2026-10-04")
-		(rev "A0")
+		(date "2026-10-05")
+		(rev "A1")
 		(comment 1 "LIVE zone = BUS- (hazardous live); SELV zone behind reinforced barrier B1")
 		(comment 2 "Schematics authored by Chinmoy Bhuyan")
@@
 		)
 	)
-	(text "7 x TLV9024 on +3V3 (open drain, rail-to-rail inputs, no firmware): IL windows,\nVA / VB over-voltage, NTC over-temperature and open probe; ladders from VREF"
+	(text "7 x TLV9024 on +3V3 (open drain, no firmware): IL windows from each sensor's Uref;\nVA / VB over-voltage, NTC over-temperature and open probe from VREF ladders"
 		(exclude_from_sim no)
 		(at 310.5 54 0)
@@
 		)
 	)
-	(text "Rev A0  |  2026-10-04  |  Schematics authored by Chinmoy Bhuyan  |  Cost-first PV-P75/100/110 controller: F280039C on BUS-, one trip latch, one SELV barrier"
+	(text "Rev A1  |  2026-10-05  |  Schematics authored by Chinmoy Bhuyan  |  Cost-first PV-P75/100/110 controller: F280039C on BUS-, one trip latch, one SELV barrier"
 		(exclude_from_sim no)
 		(at 20 36 0)

Commit message: Megarevo module parity: four-wire inverter, AC-side start-up, Ethernet and recorder on the control board, aux rev A3 (D-073..D-077)
- D-073 parity policy and register (modules only; PMA0125 and PMD-75-G3 sheets, PMA manual notes, catalogue 2026 manifest row)
- D-074 PCS-PWR-4W + PCS-CTL-4W = PCS-P125-4W drawn (fourth leg, L_N, 4-pole AC port, VGN, IL4), AC start-up tap and
  AC precharge on both builds, 30 firmware rows, declarations (kVA tiers, AC short-circuit coordination, airflow, precision)
- D-075 control board: CH9121T Ethernet bridge over CA-IS3842HW (fitted on PCS-CTL), GD25Q32E recorder flash replacing the
  EEPROM, chainable stop / ready / battery-fault inputs and HFD27 ready relay, port roles, altitude 2,000 m with the 15 mm
  isolator option specified, SELV logic allocation 2.2 W
- D-076 AUX-75 rev A3: live 30 W / 48 W for 1 s, one design for every module (turns 50:9:10, sense 3 x 0.866 ohm), four-wire
  DC precharge drawn at 200 ohm; D-077 control study: off-grid secondary restoration, THDu, imbalance, ride-through limiter
  with the stiff-grid derating rule, neutral-leg loop
- sim/compare_megarevo_pcs.py: PCS-P125 / PCS-P125-4W against the PMA0125 (2 better, 38 meets, 4 below, 9 not assessed, 0
  pending of 53); PV comparison 2 / 24 / 3 / 5 / 0 of 34 (standby 12.7 / 22.4 W)
- pin ledger E: control-board parts, shield-pin rule, fuse and connector notes (247 parts, 191 pass, 0 fail); review register
  PCM-14 and PCM-22 closed; magnetics re-run; all 15 boards rebuilt, BOMs, costs, audits and figures regenerated; README,
  guide 01-13 and the decisions mirror updated

Co-Authored-By: Claude Fable 5.1 <noreply@anthropic.com>
Other:
- sheet 02 F280039C, clock, debug, EEPROM renamed 02 F280039C, clock, debug, recorder flash
- sheet 07 SELV supply, fans, enable / status renamed 07 SELV supply, fans, stop, DI1, relay
- added sheet 08 Ethernet bridge (EMS, Modbus TCP) (sheets/08_eth.kicad_sch)
- note added: "Assembly option: the Ethernet bridge (sheet 08_eth) is NOT FITTED on PV-CTL / PV-CTL-P75 (DNP); fitted on PCS-CTL. Debug header in cJTAG mode only."
- note added: "Reinforced barrier B1: CA-IS3050W CAN, CA-IS3082WNX RS-485, 2 x CA-IS3821LG, CA-IS3820LG, CA-IS3842HW (Ethernet UART, DI1); bus TVS, jumper terminations (SELV)"
- note added: "Rev A2 | 2026-10-06 | Schematics authored by Chinmoy Bhuyan | Cost-first PV-P75/100/110 controller: F280039C on BUS-, one trip latch, one SELV barrier"
- note added: "SELV 24 V input (AUX-T1 reinforced winding, 12-36 V), TPS54360B 5 V and fan supply, 3 fan headers + tach, stop (chainable) / ready / DI1 terminals, relay, SELV 0 V to PE"
- note added: "TMS320F280039C (100-pin PZ), decoupling, 25 MHz SPXO, cTI-20 header in cJTAG mode (LIVE), 4 MB recorder flash, boot straps, command pull-downs"
- note added: "WCH CH9121T UART-to-Ethernet bridge on the SELV side, HR913550AE RJ45 with magnetics, SRV05-4, TPS7A2033 3.3 V. NOT FITTED on PV-CTL / PV-CTL-P75: footprints only (DNP)."
- note removed: "Reinforced barrier B1: CA-IS3050W CAN, CA-IS3082WNX RS-485, 2 x CA-IS3821LG, CA-IS3820LG; bus TVS, jumper terminations, pluggable field terminals (SELV)"
- note removed: "Rev A1 | 2026-10-05 | Schematics authored by Chinmoy Bhuyan | Cost-first PV-P75/100/110 controller: F280039C on BUS-, one trip latch, one SELV barrier"
- note removed: "SELV 24 V input (AUX-T1 reinforced winding, 12-36 V), TPS54360B 5 V and fan supply, 3 fan headers + tach, ENABLE / STATUS terminal, SELV 0 V to PE"
- note removed: "TMS320F280039C (100-pin PZ), decoupling, 25 MHz SPXO, cTI-20 JTAG (LIVE), EEPROM, boot straps, command pull-downs, run LED"
Changed lines of the file:
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@@
 	(title_block
 		(title "PV-CTL control board - Cover / Hierarchy")
-		(date "2026-10-05")
-		(rev "A1")
+		(date "2026-10-06")
+		(rev "A2")
 		(comment 1 "LIVE zone = BUS- (hazardous live); SELV zone behind reinforced barrier B1")
 		(comment 2 "Schematics authored by Chinmoy Bhuyan")
@@
 		)
 	)
+	(text "Assembly option: the Ethernet bridge (sheet 08_eth) is NOT FITTED on PV-CTL / PV-CTL-P75 (DNP); fitted on PCS-CTL. Debug header in cJTAG mode only."
+		(exclude_from_sim no)
+		(at 20 240 0)
+		(effects
+			(font
+				(size 1.5 1.5)
+			)
+			(justify left bottom)
+		)
+	)
+	(text "7 x TLV9024 on +3V3 (open drain, no firmware): IL windows from each sensor's Uref;\nVA / VB over-voltage, NTC over-temperature and open probe from VREF ladders"
+		(exclude_from_sim no)
+		(at 310.5 54 0)
+		(effects
+			(font
+				(size 1.3 1.3)
+			)
+			(justify left top)
+		)
+	)
+	(text "Rev A2  |  2026-10-06  |  Schematics authored by Chinmoy Bhuyan  |  Cost-first PV-P75/100/110 controller: F280039C on BUS-, one trip latch, one SELV barrier"
+		(exclude_from_sim no)
+		(at 20 36 0)
+		(effects
+			(font
+				(size 2 2)
+			)
+			(justify left bottom)
+		)
+	)
+	(text "WCH CH9121T UART-to-Ethernet bridge on the SELV side, HR913550AE RJ45 with magnetics,\nSRV05-4, TPS7A2033 3.3 V. NOT FITTED on PV-CTL / PV-CTL-P75: footprints only (DNP)."
+		(exclude_from_sim no)
+		(at 310.5 98 0)
+		(effects
+			(font
+				(size 1.3 1.3)
+			)
+			(justify left top)
+		)
+	)
 	(text "Pin plan: gen/data/pv_ctrl_pin_plan.csv (from SPRSP61C, checked every build)."
 		(exclude_from_sim no)
-		(at 20 240 0)
+		(at 20 244 0)
 		(effects
 			(font
@@
 		)
 	)
-	(text "7 x TLV9024 on +3V3 (open drain, no firmware): IL windows from each sensor's Uref;\nVA / VB over-voltage, NTC over-temperature and open probe from VREF ladders"
-		(exclude_from_sim no)
-		(at 310.5 54 0)
-		(effects
-			(font
-				(size 1.3 1.3)
-			)
-			(justify left top)
-		)
-	)
-	(text "Rev A1  |  2026-10-05  |  Schematics authored by Chinmoy Bhuyan  |  Cost-first PV-P75/100/110 controller: F280039C on BUS-, one trip latch, one SELV barrier"
-		(exclude_from_sim no)
-		(at 20 36 0)
-		(effects
-			(font
-				(size 2 2)
-			)
-			(justify left bottom)
-		)
-	)
 	(text "Assembly option: the two TLV9024 marked 'PV-P100/110 only' are not fitted on PV-P75 (bom/PV-CTL-P75_BOM.csv)."
 		(exclude_from_sim no)
@@
 		)
 	)
-	(text "Reinforced barrier B1: CA-IS3050W CAN, CA-IS3082WNX RS-485, 2 x CA-IS3821LG,\nCA-IS3820LG; bus TVS, jumper terminations, pluggable field terminals (SELV)"
+	(text "Reinforced barrier B1: CA-IS3050W CAN, CA-IS3082WNX RS-485, 2 x CA-IS3821LG,\nCA-IS3820LG, CA-IS3842HW (Ethernet UART, DI1); bus TVS, jumper terminations (SELV)"
 		(exclude_from_sim no)
 		(at 118.5 98 0)
@@
 		)
 	)
-	(text "SELV 24 V input (AUX-T1 reinforced winding, 12-36 V), TPS54360B 5 V and fan supply,\n3 fan headers + tach, ENABLE / STATUS terminal, SELV 0 V to PE"
+	(text "SELV 24 V input (AUX-T1 reinforced winding, 12-36 V), TPS54360B 5 V and fan supply,\n3 fan headers + tach, stop (chainable) / ready / DI1 terminals, relay, SELV 0 V to PE"
 		(exclude_from_sim no)
 		(at 214.5 98 0)
@@
 		)
 	)
-	(text "TMS320F280039C (100-pin PZ), decoupling, 25 MHz SPXO, cTI-20 JTAG (LIVE),\nEEPROM, boot straps, command pull-downs, run LED"
+	(text "TMS320F280039C (100-pin PZ), decoupling, 25 MHz SPXO, cTI-20 header in cJTAG mode\n(LIVE), 4 MB recorder flash, boot straps, command pull-downs"
 		(exclude_from_sim no)
 		(at 118.5 54 0)
@@
 			(color 255 255 225 1)
 		)
-		(property "Sheetname" "07 SELV supply, fans, enable / status"
+		(property "Sheetname" "07 SELV supply, fans, stop, DI1, relay"
 			(at 212 93.3 0)
 			(show_name no)
@@
 	)
 	(sheet
+		(at 308 94)
+		(size 86 26)
+		(exclude_from_sim no)
+		(in_bom yes)
+		(on_board yes)
+		(dnp no)
+		(fields_autoplaced yes)
+		(stroke
+			(width 0.254)
+			(type solid)
+		)
+		(fill
+			(color 255 255 225 1)
+		)
+		(property "Sheetname" "08 Ethernet bridge (EMS, Modbus TCP)"
+			(at 308 93.3 0)
+			(show_name no)
+			(do_not_autoplace no)
+			(effects
+				(font
+					(size 1.6 1.6)
+					(bold yes)
+				)
+				(justify left bottom)
+			)
+		)
+		(property "Sheetfile" "sheets/08_eth.kicad_sch"
+			(at 308 120.6 0)
+			(show_name no)
+			(do_not_autoplace no)
+			(effects
+				(font
+					(size 1.1 1.1)
+				)
+				(justify left top)
+			)
+		)
+		(instances
+			(project "PV-CTL"
+				(path "/27bf8643-f27c-55ee-a16b-008dacca3369"
+					(page "9")
+				)
+			)
+		)
+	)
+	(sheet
 		(at 20 50)
 		(size 86 26)
@@
 			(color 255 255 225 1)
 		)
-		(property "Sheetname" "02 F280039C, clock, debug, EEPROM"
+		(property "Sheetname" "02 F280039C, clock, debug, recorder flash"
 			(at 116 49.3 0)
 			(show_name no)
