File: hardware/PV-CTL/sheets/01_supply.kicad_sch (KiCad schematic)
At the start: 6 parts, among them J101 X6521FV-2x32-C85D32, U101 TPS3828-33DBVR

Commit message: Board revisions PV-PWR A2 / PV-CTL A1, inverter filter magnetics, documentation refresh (D-056..D-058)
Boards (every build check passes)
- PV-PWR / PV-PWR-4 rev A2: seventh battery-side film capacitor on the three-phase board (closes the
  load-rejection overshoot), bleeder 8 x 73.2 k so the bank still discharges within its 10-minute label.
- PV-CTL rev A1: hardware over-current window 68.9-79.9 A, thresholds derived from each sensor's own
  reference; the board-to-board contract carries the four references on the former 24 V / 5 V pins.
- Records aligned (contract comments, architecture corrections, port-current bandwidth); the frozen
  platform's module BOMs are kept instead of being re-rolled from the cost-first thermal data.

Magnetics
- Inverter filter designed and verified: L1, L2 and the AC common-mode choke (design_pcs_*.json). The filter
  comes to 745 USD at catalogue prices and 611 USD at 5,000 units, against 207 / 167 in the study: the
  inverter's cost is provisional and its stage and filter are being re-optimised.
- PV inductor loss check made non-circular; hot-spot margin reported per build (PV-P100/110: -5.3 K, MG-17).

Results: PV-P75 952 USD at catalogue prices / 796 USD at 5,000 units; Megarevo comparison 2 better,
24 meet, 3 below, 5 not assessed. Documentation corrected for the revised boards (51 statements).
Everything is calculated or estimated; nothing is bench-validated.

Co-Authored-By: Claude Fable 5.1 <noreply@anthropic.com>
Connections:
- net IL1R: now reaches J101.1 (Pin_1)
- net IL2R: now reaches J101.2 (Pin_2)
- net IL3R: now reaches J101.5 (Pin_5)
- net IL4R: now reaches J101.6 (Pin_6)
- no-connect marks 5 -> 1
Other:
- note added: "LIVE: GND = AGND = BUS-; nothing on this connector leaves the enclosure. Only +3V3 comes across (the former +24V / +5V pins carry the sensor references IL1R-IL4R since PV-PWR rev A2). +3V3 feeds the MCU, so the power board's 3.3 V signals and VDDIO share one rail and one power-up order (no back-powering)."
- note removed: "LIVE: GND = AGND = BUS-; nothing on this connector leaves the enclosure. +24V and +5V are NOT used (PV-PWR allocation 0 / 50 mA; the live 24 V is already over its rating): pins left open. +3V3 feeds the MCU, so the power board's 3.3 V signals and VDDIO share one rail and one power-up order (no back-powering)."
Changed lines of the file:
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@@
 	(title_block
 		(title "PV-CTL control board - PC connector, supply, reset")
-		(date "2026-10-04")
-		(rev "A0")
+		(date "2026-10-05")
+		(rev "A1")
 		(comment 1 "LIVE zone = BUS- (hazardous live); SELV zone behind reinforced barrier B1")
 		(comment 2 "Schematics authored by Chinmoy Bhuyan")
@@
 		)
 	)
-	(text "LIVE: GND = AGND = BUS-; nothing on this connector leaves the enclosure. +24V and +5V are NOT used (PV-PWR\nallocation 0 / 50 mA; the live 24 V is already over its rating): pins left open. +3V3 feeds the MCU, so the\npower board's 3.3 V signals and VDDIO share one rail and one power-up order (no back-powering)."
+	(text "LIVE: GND = AGND = BUS-; nothing on this connector leaves the enclosure. Only +3V3 comes across (the former\n+24V / +5V pins carry the sensor references IL1R-IL4R since PV-PWR rev A2). +3V3 feeds the MCU, so the\npower board's 3.3 V signals and VDDIO share one rail and one power-up order (no back-powering)."
 		(exclude_from_sim no)
 		(at 14 122.78 0)
@@
 	)
 	(no_connect
-		(at 27.94 27.94)
-	)
-	(no_connect
 		(at 139.7 33.02)
 	)
-	(no_connect
-		(at 40.64 33.02)
-	)
-	(no_connect
-		(at 40.64 27.94)
-	)
-	(no_connect
-		(at 27.94 33.02)
+	(wire
+		(pts
+			(xy 27.94 27.94) (xy 25.4 27.94)
+		)
+		(stroke
+			(width 0)
+			(type default)
+		)
 	)
 	(wire
@@
 	(wire
 		(pts
+			(xy 40.64 33.02) (xy 43.18 33.02)
+		)
+		(stroke
+			(width 0)
+			(type default)
+		)
+	)
+	(wire
+		(pts
 			(xy 40.64 78.74) (xy 43.18 78.74)
 		)
@@
 	(wire
 		(pts
+			(xy 27.94 33.02) (xy 25.4 33.02)
+		)
+		(stroke
+			(width 0)
+			(type default)
+		)
+	)
+	(wire
+		(pts
 			(xy 27.94 91.44) (xy 25.4 91.44)
 		)
@@
 	(wire
 		(pts
+			(xy 40.64 27.94) (xy 43.18 27.94)
+		)
+		(stroke
+			(width 0)
+			(type default)
+		)
+	)
+	(wire
+		(pts
 			(xy 27.94 60.96) (xy 25.4 60.96)
 		)
@@
 		)
 	)
+	(global_label "IL2R"
+		(shape bidirectional)
+		(at 43.18 27.94 0)
+		(fields_autoplaced yes)
+		(effects
+			(font
+				(size 1 1)
+			)
+			(justify left)
+		)
+		(property "Intersheetrefs" "${INTERSHEET_REFS}"
+			(at 43.18 27.94 0)
+			(hide yes)
+			(show_name no)
+			(do_not_autoplace no)
+			(effects
+				(font
+					(size 1 1)
+				)
+			)
+		)
+	)
 	(global_label "VAX"
 		(shape bidirectional)
@@
 		)
 	)
+	(global_label "IL1R"
+		(shape bidirectional)
+		(at 25.4 27.94 180)
+		(fields_autoplaced yes)
+		(effects
+			(font
+				(size 1 1)
+			)
+			(justify right)
+		)
+		(property "Intersheetrefs" "${INTERSHEET_REFS}"
+			(at 25.4 27.94 180)
+			(hide yes)
+			(show_name no)
+			(do_not_autoplace no)
+			(effects
+				(font
+					(size 1 1)
+				)
+			)
+		)
+	)
 	(global_label "IA_H"
 		(shape bidirectional)
@@
 		)
 	)
+	(global_label "IL3R"
+		(shape bidirectional)
+		(at 25.4 33.02 180)
+		(fields_autoplaced yes)
+		(effects
+			(font
+				(size 1 1)
+			)
+			(justify right)
+		)
+		(property "Intersheetrefs" "${INTERSHEET_REFS}"
+			(at 25.4 33.02 180)
+			(hide yes)
+			(show_name no)
+			(do_not_autoplace no)
+			(effects
+				(font
+					(size 1 1)
+				)
+			)
+		)
+	)
 	(global_label "IL2"
 		(shape bidirectional)
@@
 			(hide yes)
 			(show_name no)
+			(do_not_autoplace no)
+			(effects
+				(font
+					(size 1 1)
+				)
+			)
+		)
+	)
+	(global_label "IL4R"
+		(shape bidirectional)
+		(at 43.18 33.02 0)
+		(fields_autoplaced yes)
+		(effects
+			(font
+				(size 1 1)
+			)
+			(justify left)
+		)
+		(property "Intersheetrefs" "${INTERSHEET_REFS}"
+			(at 43.18 33.02 0)
+			(hide yes)
+			(show_name no)
