File: hardware/PV-CTL/sheets/04_trip.kicad_sch (KiCad schematic)
At the start: 33 parts, among them U401 TLV9024PWR, U402 TLV9024PWR, U403 TLV9024PWR, U404 TLV9024PWR, U405 TLV9024PWR, U406 TLV9024PWR (PV-P100/110 only), U407 TLV9024PWR (PV-P100/110 only)

Commit message: Board revisions PV-PWR A2 / PV-CTL A1, inverter filter magnetics, documentation refresh (D-056..D-058)
Boards (every build check passes)
- PV-PWR / PV-PWR-4 rev A2: seventh battery-side film capacitor on the three-phase board (closes the
  load-rejection overshoot), bleeder 8 x 73.2 k so the bank still discharges within its 10-minute label.
- PV-CTL rev A1: hardware over-current window 68.9-79.9 A, thresholds derived from each sensor's own
  reference; the board-to-board contract carries the four references on the former 24 V / 5 V pins.
- Records aligned (contract comments, architecture corrections, port-current bandwidth); the frozen
  platform's module BOMs are kept instead of being re-rolled from the cost-first thermal data.

Magnetics
- Inverter filter designed and verified: L1, L2 and the AC common-mode choke (design_pcs_*.json). The filter
  comes to 745 USD at catalogue prices and 611 USD at 5,000 units, against 207 / 167 in the study: the
  inverter's cost is provisional and its stage and filter are being re-optimised.
- PV inductor loss check made non-circular; hot-spot margin reported per build (PV-P100/110: -5.3 K, MG-17).

Results: PV-P75 952 USD at catalogue prices / 796 USD at 5,000 units; Megarevo comparison 2 better,
24 meet, 3 below, 5 not assessed. Documentation corrected for the revised boards (51 statements).
Everything is calculated or estimated; nothing is bench-validated.

Co-Authored-By: Claude Fable 5.1 <noreply@anthropic.com>
Parts:
- added C414, C415, C416, C417, C418, C419: 100n 50V, symbol dcdc:C
- added R414: 19.1k, symbol dcdc:R
- added R415: 20.0k, symbol dcdc:R
- added R416: 1M, symbol dcdc:R
- added R417: 2.10k, symbol dcdc:R
- added R418: 11.8k, symbol dcdc:R
- added R419: 102k, symbol dcdc:R
- added R420: 10.0k, symbol dcdc:R
- added R421: 30.9k, symbol dcdc:R
- added R422: 1.15k, symbol dcdc:R
- added R423: 115R, symbol dcdc:R
- added R424: 13.7k, symbol dcdc:R
- added R425, R426: 10k, symbol dcdc:R
- C407, C408, C409, C410, C411, C412: value 100n 50V -> 10n 50V
- R401: value 8.25k -> 715R
- R402: value 17.4k -> 19.1k
- R403: value 19.1k -> 20.0k
- R404: value 2.10k -> 1M
- R405: value 11.8k -> 715R
- R406: value 102k -> 19.1k
- R407: value 10.0k -> 20.0k
- R408: value 30.9k -> 1M
- R409: value 1.15k -> 715R
- R410: value 115R -> 19.1k
- R411: value 13.7k -> 20.0k
- R412: value 10k -> 1M
- R413: value 10k -> 715R
Connections:
- net +3V3: now also C414.1, C415.1, C416.1, C417.1, C418.1, C419.1, R425.1, R426.1; no longer C407.1, C408.1, C409.1, C410.1, C411.1, C412.1, R412.1, R413.1
- net GND: now also C414.2, C415.2, C416.2, C417.2, C418.2, C419.2, R415.2, R418.2, R420.2, R422.2, R424.2; no longer R405.2, R409.2
- net OC_N: now also R425.2; no longer R412.2
- net OVT_N: now also R426.2; no longer R413.2
- net TH_OPEN: now also C412.1, R423.2, R424.1; no longer C406.1, R410.2, R411.1
- net TH_OTH: now also C410.1, R419.2, R420.1; no longer C404.1, R406.2, R407.1
- net TH_OTL: now also C411.1, R421.2, R422.1; no longer C405.1, R408.2, R409.1
- net TH_OV: now also C409.1, R417.2, R418.1; no longer C403.1, R404.2, R405.1
- net VREF: now also R412.1, R416.1, R417.1, R419.1, R421.1, R423.1; no longer R401.1, R406.1, R410.1
- net TH_IL_HI renamed TH_IL1_HI
- net TH_IL1_HI: no longer U401.9 (IN3+), U402.5 (IN1+), U406.5 (IN1+)
- net TH_IL_LO renamed TH_IL1_LO
- net TH_IL1_LO: now also R404.2; no longer U401.10 (IN4-), U402.6 (IN2-), U406.6 (IN2-)
- new net IL1R: R401.1
- new net IL2R: R405.1
- new net IL3R: R409.1
- new net IL4R: R413.1
- new net TH_IL2_HI: C403.1, R405.2, R406.1, U401.9 (IN3+)
- new net TH_IL2_LO: C404.1, R406.2, R407.1, R408.2, U401.10 (IN4-)
- new net TH_IL3_HI: C405.1, R409.2, R410.1, U402.5 (IN1+)
- new net TH_IL3_LO: C406.1, R410.2, R411.1, R412.2, U402.6 (IN2-)
- new net TH_IL4_HI: C407.1, R413.2, R414.1, U406.5 (IN1+)
- new net TH_IL4_LO: C408.1, R414.2, R415.1, R416.2, U406.6 (IN2-)
Other:
- note added: "IL THRESHOLD LADDERS (0.1 %, 25 PPM/K), ONE PER PHASE FROM THAT SENSOR'S UREF (ILNR ON PC)"
- note added: "ILnR - 715R - TH_ILn_HI - 19.1k - TH_ILn_LO - 20.0k - GND: the window follows the sensor's own zero (Vref 2.48-2.52 V is no longer an error term; Voe +/-10 mV is). 1 M from VREF to TH_ILn_LO: with the sensor dead (IL = ILR = 0 V) TH_ILn_LO stays ~30 mV above ILn_P and the phase trips. Phase 4: fitted on every build."
- note added: "OC_N (wired-OR, 10k to +3V3): ILn_P above TH_ILn_HI or below TH_ILn_LO, n = 1-3. OVT_N (10k): VA, VB above TH_OV; NTC1-3 (heatsink) below TH_OTH, NTC5-7 (inductor) below TH_OTL; any of them above TH_OPEN. Port over-current (387-413 A) arrives on FLT_N from the power board's own comparators (PV-PWR)."
- note added: "TH_OV: VA/VB 1084 V; TH_OTH: heatsink 87.9 C (PV-PWR: <= 89.9 C); TH_OTL: inductor 150 C; TH_OPEN 2.975 V: an NTC node above it is an open probe (cold limit -30 C)."
- note removed: "OC_N (wired-OR, 10k to +3V3): ILn_P above TH_IL_HI or below TH_IL_LO, n = 1-3. OVT_N (10k): VA, VB above TH_OV; NTC1-3 (heatsink) below TH_OTH, NTC5-7 (inductor) below TH_OTL; any of them above TH_OPEN. Port over-current (387-413 A) arrives on FLT_N from the power board's own comparators (PV-PWR)."
- note removed: "TH_IL_HI/LO: IL window (+/-73 A); TH_OV: VA/VB 1084 V; TH_OTH: heatsink 87.9 C (PV-PWR: <= 89.9 C); TH_OTL: inductor 150 C; TH_OPEN 2.975 V: an NTC node above it is an open probe (cold limit -30 C)."
- moved on the sheet: C402, C403, C404, C405, C406, C407, C408, C409, C410, C411, C412, C413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

Commit message: Resolve the independent PCM review of 033d8d8 (PCM-01..27): verify, classify, fix at the root (D-065..D-072)
Register gen/data/review_pcm.csv: 27 findings, each verified before a change - 21 Confirmed, 2 Firmware
Handled, 3 Improvement Recommended, 1 Not Applicable; 20 closed, 7 open with their closing path.

PV family (D-065, D-072): the 45 A port rating no longer clamps the inductor current in the near-unity
band (inductor rating 47.7 A there; 550/550 V 73.3 kW; rated power from 562 V); control model re-based on
the drawn boards with a published delivered-power envelope per product and direction; leg commutation
re-run on the drawn Jianghai capacitors (1374 V worst vs 1445 V); comparator common-mode term in every
trip band (window 67.9-80.5 A, the 1.10 margin rule missed by 0.58 A and left open; firmware OV derived
from the drawn band, 1034 V); one fan-supply contract; cold-start passive-power restriction modelled;
port A interface declared; aux pull-in and retry rules.

PCS-P125 (D-066, D-067): control study sim/pcs_control.py (PR current loop 1750 Hz, PM >= 48.7 deg to
SCR 5 with the passive damping branch, PLL, DC-link loop, grid forming, state machine); DC-link inventory
409.4 uF with bleeders, precharge rating and the 15 min label re-derived; upper-half limit in firmware;
P-Q-Vdc-Vac envelope (AC-02's 600 V full-load figure not reachable at a +15 % grid: owner's decision);
R_DS(on) acceptance rule for the six paralleled devices; DESAT string 3 -> 2 diodes (band 6.41-9.37 V);
fuse-contactor coordination bands and installation requirements; phase-current sensor frozen to Sinomags
STK-250HO/4 and the control-board ladders re-valued; Al2O3 pad text.

DAB-D60 (D-068): study vs drawn-board identity made explicit; short-circuit chain corrected (energy-
equivalent 0.99 x the assumed withstand; release block t_SC >= 2.22 us / E_SC >= 2.18 J); admitted map
follows the 1200 V deck envelope (900-950 V rows derated until a double-pulse test); zero/light-load policy;
0.41 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
Parts:
- R417: value 2.10k -> 2.05k
- R418: value 11.8k -> 11.3k
Other:
- note added: "TH_OV: VA/VB 1075 V; TH_OTH: heatsink 87.9 C (PV-PWR: <= 89.9 C); TH_OTL: inductor 150 C; TH_OPEN 2.975 V: an NTC node above it is an open probe (cold limit -30 C)."
- note removed: "TH_OV: VA/VB 1084 V; TH_OTH: heatsink 87.9 C (PV-PWR: <= 89.9 C); TH_OTL: inductor 150 C; TH_OPEN 2.975 V: an NTC node above it is an open probe (cold limit -30 C)."
Changed lines of the file:
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@@
 		)
 	)
-	(text "TH_OV: VA/VB 1084 V; TH_OTH: heatsink 87.9 C (PV-PWR: <= 89.9 C); TH_OTL: inductor 150 C;\nTH_OPEN 2.975 V: an NTC node above it is an open probe (cold limit -30 C)."
+	(text "TH_OV: VA/VB 1075 V; TH_OTH: heatsink 87.9 C (PV-PWR: <= 89.9 C); TH_OTL: inductor 150 C;\nTH_OPEN 2.975 V: an NTC node above it is an open probe (cold limit -30 C)."
 		(exclude_from_sim no)
 		(at 257.608 86.86 0)
@@
 			)
 		)
-		(property "Value" "11.8k"
+		(property "Value" "11.3k"
 			(at 279.146 36.46 0)
 			(show_name no)
@@
 			)
 		)
-		(property "Description" "Resistor 11.8k 0.1% 0603 25 ppm/K"
+		(property "Description" "Resistor 11.3k 0.1% 0603 25 ppm/K"
 			(at 274.32 35.56 0)
 			(hide yes)
@@
 			)
 		)
-		(property "Value" "2.10k"
+		(property "Value" "2.05k"
 			(at 266.446 36.46 0)
 			(show_name no)
@@
 			)
 		)
-		(property "Description" "Resistor 2.10k 0.1% 0603 25 ppm/K"
+		(property "Description" "Resistor 2.05k 0.1% 0603 25 ppm/K"
 			(at 261.62 35.56 0)
 			(hide yes)
