File: hardware/PV-CTL/sheets/05_latch.kicad_sch (KiCad schematic)
At the start: 35 parts, among them U501 SN74LVC07APWR, U502 SN74LVC1G74DCUR, U503 SN74LVC1G123DCUR, U504 SN74LVC1G32DBVR, U505 SN74LVC08APWR, U506 SN74LVC08APWR, U507 SN74LVC08APWR, U508 SN74LVC08APWR, U509 SN74LVC08APWR, U510 SN74LVC08APWR

Commit message: Megarevo module parity: four-wire inverter, AC-side start-up, Ethernet and recorder on the control board, aux rev A3 (D-073..D-077)
- D-073 parity policy and register (modules only; PMA0125 and PMD-75-G3 sheets, PMA manual notes, catalogue 2026 manifest row)
- D-074 PCS-PWR-4W + PCS-CTL-4W = PCS-P125-4W drawn (fourth leg, L_N, 4-pole AC port, VGN, IL4), AC start-up tap and
  AC precharge on both builds, 30 firmware rows, declarations (kVA tiers, AC short-circuit coordination, airflow, precision)
- D-075 control board: CH9121T Ethernet bridge over CA-IS3842HW (fitted on PCS-CTL), GD25Q32E recorder flash replacing the
  EEPROM, chainable stop / ready / battery-fault inputs and HFD27 ready relay, port roles, altitude 2,000 m with the 15 mm
  isolator option specified, SELV logic allocation 2.2 W
- D-076 AUX-75 rev A3: live 30 W / 48 W for 1 s, one design for every module (turns 50:9:10, sense 3 x 0.866 ohm), four-wire
  DC precharge drawn at 200 ohm; D-077 control study: off-grid secondary restoration, THDu, imbalance, ride-through limiter
  with the stiff-grid derating rule, neutral-leg loop
- sim/compare_megarevo_pcs.py: PCS-P125 / PCS-P125-4W against the PMA0125 (2 better, 38 meets, 4 below, 9 not assessed, 0
  pending of 53); PV comparison 2 / 24 / 3 / 5 / 0 of 34 (standby 12.7 / 22.4 W)
- pin ledger E: control-board parts, shield-pin rule, fuse and connector notes (247 parts, 191 pass, 0 fail); review register
  PCM-14 and PCM-22 closed; magnetics re-run; all 15 boards rebuilt, BOMs, costs, audits and figures regenerated; README,
  guide 01-13 and the decisions mirror updated

Co-Authored-By: Claude Fable 5.1 <noreply@anthropic.com>
Other:
- note added: "74LVC07 (Ioff, 5 V tolerant): OC_N, OVT_N, FLT_N (driver DESAT/UVLO + port OC of PV-PWR), RDY (gate supplies, +5V, live 24 V on PV-PWR), STOP_OK (ENABLE), WD_OK (heartbeat and MCU reset). Any low -> PRE_N low -> latch set asynchronously (Q = TRIP = 1). The MCU reads PRE_N on GPIO17 (rev A2, diagnosis only)."
- note removed: "74LVC07 (Ioff, 5 V tolerant): OC_N, OVT_N, FLT_N (driver DESAT/UVLO + port OC of PV-PWR), RDY (gate supplies, +5V, live 24 V on PV-PWR), STOP_OK (ENABLE), WD_OK (heartbeat and MCU reset). Any low -> PRE_N low -> latch set asynchronously (Q = TRIP = 1)."
- moved on the sheet: C501, C502, C503, C504, C505, D501, R501, R502, R503, R504, U502, U503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
