File: hardware/PV-CTL/sheets/07_selv.kicad_sch (KiCad schematic)
At the start: 59 parts, among them J701 KF2EDGR-3.81-2P, J702 X6511WV-03H-C60D30, J703 X6511WV-03H-C60D30, J704 X6511WV-03H-C60D30, J705 KF2EDGR-3.81-4P, Q701 2N7002BK,215, U701 TPS54360BDDAR, U702 TPS54360BDDAR

Commit message: Resolve the independent PCM review of 033d8d8 (PCM-01..27): verify, classify, fix at the root (D-065..D-072)
Register gen/data/review_pcm.csv: 27 findings, each verified before a change - 21 Confirmed, 2 Firmware
Handled, 3 Improvement Recommended, 1 Not Applicable; 20 closed, 7 open with their closing path.

PV family (D-065, D-072): the 45 A port rating no longer clamps the inductor current in the near-unity
band (inductor rating 47.7 A there; 550/550 V 73.3 kW; rated power from 562 V); control model re-based on
the drawn boards with a published delivered-power envelope per product and direction; leg commutation
re-run on the drawn Jianghai capacitors (1374 V worst vs 1445 V); comparator common-mode term in every
trip band (window 67.9-80.5 A, the 1.10 margin rule missed by 0.58 A and left open; firmware OV derived
from the drawn band, 1034 V); one fan-supply contract; cold-start passive-power restriction modelled;
port A interface declared; aux pull-in and retry rules.

PCS-P125 (D-066, D-067): control study sim/pcs_control.py (PR current loop 1750 Hz, PM >= 48.7 deg to
SCR 5 with the passive damping branch, PLL, DC-link loop, grid forming, state machine); DC-link inventory
409.4 uF with bleeders, precharge rating and the 15 min label re-derived; upper-half limit in firmware;
P-Q-Vdc-Vac envelope (AC-02's 600 V full-load figure not reachable at a +15 % grid: owner's decision);
R_DS(on) acceptance rule for the six paralleled devices; DESAT string 3 -> 2 diodes (band 6.41-9.37 V);
fuse-contactor coordination bands and installation requirements; phase-current sensor frozen to Sinomags
STK-250HO/4 and the control-board ladders re-valued; Al2O3 pad text.

DAB-D60 (D-068): study vs drawn-board identity made explicit; short-circuit chain corrected (energy-
equivalent 0.99 x the assumed withstand; release block t_SC >= 2.22 us / E_SC >= 2.18 J); admitted map
follows the 1200 V deck envelope (900-950 V rows derated until a double-pulse test); zero/light-load policy;
0.41 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
Parts:
- D701, D705: Manufacturer Bourns -> MDD (Microdiode Semiconductor)
Changed lines of the file:
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@@
 			)
 		)
-		(property "Datasheet" "docs/datasheets/protection/SMBJ_Bourns.pdf"
+		(property "Datasheet" "docs/datasheets/protection/MDD-SMBJ-series.pdf"
 			(at 93.98 195.58 0)
 			(hide yes)
@@
 			)
 		)
-		(property "Manufacturer" "Bourns"
+		(property "Manufacturer" "MDD (Microdiode Semiconductor)"
 			(at 93.98 195.58 0)
 			(hide yes)
@@
 			)
 		)
-		(property "Datasheet" "docs/datasheets/protection/SMBJ_Bourns.pdf"
+		(property "Datasheet" "docs/datasheets/protection/MDD-SMBJ-series.pdf"
 			(at 17.78 35.56 0)
 			(hide yes)
@@
 			)
 		)
-		(property "Manufacturer" "Bourns"
+		(property "Manufacturer" "MDD (Microdiode Semiconductor)"
 			(at 17.78 35.56 0)
 			(hide yes)

Commit message: Megarevo module parity: four-wire inverter, AC-side start-up, Ethernet and recorder on the control board, aux rev A3 (D-073..D-077)
- D-073 parity policy and register (modules only; PMA0125 and PMD-75-G3 sheets, PMA manual notes, catalogue 2026 manifest row)
- D-074 PCS-PWR-4W + PCS-CTL-4W = PCS-P125-4W drawn (fourth leg, L_N, 4-pole AC port, VGN, IL4), AC start-up tap and
  AC precharge on both builds, 30 firmware rows, declarations (kVA tiers, AC short-circuit coordination, airflow, precision)
- D-075 control board: CH9121T Ethernet bridge over CA-IS3842HW (fitted on PCS-CTL), GD25Q32E recorder flash replacing the
  EEPROM, chainable stop / ready / battery-fault inputs and HFD27 ready relay, port roles, altitude 2,000 m with the 15 mm
  isolator option specified, SELV logic allocation 2.2 W
- D-076 AUX-75 rev A3: live 30 W / 48 W for 1 s, one design for every module (turns 50:9:10, sense 3 x 0.866 ohm), four-wire
  DC precharge drawn at 200 ohm; D-077 control study: off-grid secondary restoration, THDu, imbalance, ride-through limiter
  with the stiff-grid derating rule, neutral-leg loop
- sim/compare_megarevo_pcs.py: PCS-P125 / PCS-P125-4W against the PMA0125 (2 better, 38 meets, 4 below, 9 not assessed, 0
  pending of 53); PV comparison 2 / 24 / 3 / 5 / 0 of 34 (standby 12.7 / 22.4 W)
- pin ledger E: control-board parts, shield-pin rule, fuse and connector notes (247 parts, 191 pass, 0 fail); review register
  PCM-14 and PCM-22 closed; magnetics re-run; all 15 boards rebuilt, BOMs, costs, audits and figures regenerated; README,
  guide 01-13 and the decisions mirror updated

Co-Authored-By: Claude Fable 5.1 <noreply@anthropic.com>
Parts:
- added C722: 4.7n 1kV, symbol dcdc:C
- added D706: BZX84-C5V1,215, symbol dcdc:BZX84C5V1
- added D707: SMBJ58CA, symbol dcdc:SMBJ58CA
- added J706: KF2EDGR-3.81-8P, symbol dcdc:J_KF8
- added K701: HFD27/005-S, symbol dcdc:HFD27
- added R723, R724: 10k, symbol dcdc:R
- added R725: 1M, symbol dcdc:R
- C721: value 4.7n 1kV -> 100n 50V; Domain CROSSING -> SELV; Package 1206 -> 0603
- D705: value SMBJ58CA -> BAS16; symbol dcdc:SMBJ58CA -> dcdc:BAS16; Domain CROSSING -> SELV; MPN SMBJ58CA -> BAS16; Manufacturer MDD (Microdiode Semiconductor) -> Nexperia; Package SMB -> SOT-23
- J705: value KF2EDGR-3.81-4P -> KF2EDGR-3.81-6P; symbol dcdc:J_KF4 -> dcdc:J_KF6; Domain SELV -> CROSSING; MPN KF2EDGR-3.81-4P -> KF2EDGR-3.81-6P; Package pluggable 4-pos 3.81 mm R/A -> pluggable 6-pos 3.81 mm R/A
- R722: value 1M -> 1.0k; Domain CROSSING -> SELV; Package 1206 -> 0603
Connections:
- net PE: now also J705.6 (Pin_6), C722.2, D707.2 (A2), R725.2; no longer C721.2, D705.2 (A2), R722.2
- net S_5V: now also D705.3 (K), R722.1, K701.1 (COIL1)
- net S_EN_IN: now also J706.7 (Pin_7); no longer J705.2 (Pin_2)
- net S_GND: now also C721.2, J705.5 (Pin_5), C722.1, D706.1 (A), D707.1 (A1), J706.8 (Pin_8), R723.2, R725.1; no longer C721.1, D705.1 (A1), R722.1
- net S_STATUS renamed S_EN_BUS
- net S_EN_BUS: now also J705.2 (Pin_2), J706.6 (Pin_6); no longer Q701.3 (D)
- new net S_DI1: C721.1, D706.3 (K), R724.2
- new net S_DI1_IN: J706.5 (Pin_5), R723.1, R724.1
- new net S_DI1_SRC: J706.4 (Pin_4), R722.2
- new net S_RLY_COM: J706.2 (Pin_2), K701.13 (COM2), K701.4 (COM1)
- new net S_RLY_K: D705.1 (A), K701.16 (COIL2), Q701.3 (D)
- new net S_RLY_NC: J706.3 (Pin_3), K701.11 (NC2), K701.6 (NC1)
- new net S_RLY_NO: J706.1 (Pin_1), K701.8 (NO1), K701.9 (NO2)
- no-connect marks 2 -> 4
Other:
- note added: "J_STOP 1 S_EN_SRC (S_24V via 10k: dry-contact supply for ONE module), 2 / 3 stop line in / out (loop-through: chain a cabinet 24 V stop line module to module), 4 / 5 0 V in / out, 6 screen to PE. J_IO 6-7: ready permissive in series (wire link if unused) -> S_EN_IN -> 33k / 10k, 5.1 V clamp, 100 nF -> isolator -> STOP_OK -> latch (no firmware): open stop contact, open permissive, broken wire or l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"
- note added: "RELAY OUTPUT (READY / FAULT) AND DI1 (BATTERY FAULT / BMS CONTACT)"
- note added: "STATUS channel -> 2N7002BK -> HFD27/005-S coil from S_5V, BAS16 across it: energised = healthy (NO closed); a trip, stop, lost SELV or live side = NC closed. Both poles in parallel; SELV circuits only (<= 30 V AC / 60 V DC). J_IO 4 = 5 V wetting (1.0k from S_5V), 5 = DI1 (10k down, 10k + 100 nF = 1 ms, 5.1 V clamp) -> CA-IS3842HW VI3."
- note added: "STOP INPUT (HARDWARE, CHAINABLE) AND READY PERMISSIVE"
- note removed: "1 S_EN_SRC (S_24V via 10k: dry-contact supply), 2 S_EN_IN (contact return or a PLC output), 3 STATUS (open drain 2N7002BK, conducting = healthy), 4 0 V. S_EN_IN -> 33k / 10k (5.1 V clamp, 100 nF: 0.77 ms) -> isolator: open contact, broken wire or lost SELV = STOP_OK low = latch set (no firmware)."
- note removed: "ENABLE (EXTERNAL STOP) AND STATUS TERMINAL"
- title: PV-CTL control board - SELV supply, fans, enable / status -> PV-CTL control board - SELV supply, fans, stop, DI1, relay
- moved on the sheet: C721, H701, Q701, R719, R721, R722
