File: hardware/PCS-PWR-4W/PCS-PWR-4W.kicad_sch (KiCad schematic)
At the start: 0 parts

Commit message: Respond to the independent re-check R2 of a427981 (D-078, D-079): gates-off commutation closed, backup band lowered, SiC acceptance, bounded grid-forming transients, ride-through without derating, AC-start repairs, installation requirements
- Register gen/data/review_r2.csv: 14 findings verified and dispositioned (9 Confirmed, 1 Firmware Handled,
  1 Improvement Recommended, 2 Already Fixed, 1 Not Applicable), every row closed with its evidence
- D-078 power stage: the discrete window turns the gates off at 520.8 A, not at the 485.5 A window top; the leg deck
  at that current peaked at 1457 V against 1445 V, closed at zero cost by R_G,off 7.5 -> 8.75 ohm (1437 V, admissible
  533.6 A); L1 inductance trajectory to 700 A (knee 566 A), CMPSS backup band lowered to 423.9-497.5 A on PCS-CTL,
  firmware OV backup 1035 V; R_DS(on) <= 40 mOhm acceptance with per-lot derating; one coil contract (20 W / 4 W);
  residual-current monitor contract; docs/requirements/INSTALLATION.md (74 enforceable requirements with sources)
- D-079 control study: tolerance regression at the assembly tolerances (1,944 + 1,000 cases, worst PM 48.1 deg);
  bounded grid-forming transients 0.43 / 1.77 pu with feed-forward and OV deadbeat (2.17 pu superseded), trip-aware
  DC-load rejection, CV-mode soft-OV hold, weak-grid CV power limits, PV DC-bus coordination row (0.51 ms);
  ride-through 270 A clamp with C_f prediction removes the stiff-grid derating (fallback kept, SCR estimator,
  8.07 MVA declaration); coupled four-wire cases; AC start in the executable state machine (17 states, 35 fault
  cases) with the five sequence holes H1-H5 repaired and an own AC_STOP state
- pcs_spec protection_chain published and read by the control study and the control board; all 15 boards, BOMs,
  costs, comparisons (PV 2/24/3/5/0, PCS 2/38/4/9/0), audits and figures regenerated; README, guide 03-13,
  decisions mirror and architecture reconciliation notes updated; .graphifyignore and graphify-out/ ignored

Co-Auth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
Other:
- note added: "gdrv.channel() 6 x SG2M040170HJ: NSI6651ASC-Q1 +18/-3.5 V, 8.75/8.75 ohm per device; PNP turn-off buffers, Miller clamps, booster, DESAT"
- note added: "gdrv.channel() 6 x SG2M040170HJ: NSI6651ASC-Q1 +18/-3.5 V, 8.75/8.75 ohm per device; PNP turn-off buffers, Miller clamps, booster, DESAT; bias SN6505B + T_BIAS4"
- note removed: "gdrv.channel() 6 x SG2M040170HJ: NSI6651ASC-Q1 +18/-3.5 V, 8.75/7.5 ohm per device; PNP turn-off buffers, Miller clamps, booster, DESAT"
- note removed: "gdrv.channel() 6 x SG2M040170HJ: NSI6651ASC-Q1 +18/-3.5 V, 8.75/7.5 ohm per device; PNP turn-off buffers, Miller clamps, booster, DESAT; bias SN6505B + T_BIAS4"
Changed lines of the file:
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@@
 		(comment 4 "Not bench-validated. Values read from sim/out/pcs_design/pcs_spec.json; checks: design_check()")
 	)
-	(text "gdrv.channel() 6 x SG2M040170HJ: NSI6651ASC-Q1 +18/-3.5 V, 8.75/7.5 ohm per device;\nPNP turn-off buffers, Miller clamps, booster, DESAT"
+	(text "gdrv.channel() 6 x SG2M040170HJ: NSI6651ASC-Q1 +18/-3.5 V, 8.75/8.75 ohm per device;\nPNP turn-off buffers, Miller clamps, booster, DESAT"
 		(exclude_from_sim no)
 		(at 22.5 142 0)
@@
 		)
 	)
-	(text "gdrv.channel() 6 x SG2M040170HJ: NSI6651ASC-Q1 +18/-3.5 V, 8.75/7.5 ohm per device;\nPNP turn-off buffers, Miller clamps, booster, DESAT; bias SN6505B + T_BIAS4"
+	(text "gdrv.channel() 6 x SG2M040170HJ: NSI6651ASC-Q1 +18/-3.5 V, 8.75/8.75 ohm per device;\nPNP turn-off buffers, Miller clamps, booster, DESAT; bias SN6505B + T_BIAS4"
 		(exclude_from_sim no)
 		(at 118.5 142 0)
@@
 		)
 	)
-	(text "gdrv.channel() 6 x SG2M040170HJ: NSI6651ASC-Q1 +18/-3.5 V, 8.75/7.5 ohm per device;\nPNP turn-off buffers, Miller clamps, booster, DESAT; bias SN6505B + T_BIAS4"
+	(text "gdrv.channel() 6 x SG2M040170HJ: NSI6651ASC-Q1 +18/-3.5 V, 8.75/8.75 ohm per device;\nPNP turn-off buffers, Miller clamps, booster, DESAT; bias SN6505B + T_BIAS4"
 		(exclude_from_sim no)
 		(at 118.5 186 0)
@@
 		)
 	)
-	(text "gdrv.channel() 6 x SG2M040170HJ: NSI6651ASC-Q1 +18/-3.5 V, 8.75/7.5 ohm per device;\nPNP turn-off buffers, Miller clamps, booster, DESAT"
+	(text "gdrv.channel() 6 x SG2M040170HJ: NSI6651ASC-Q1 +18/-3.5 V, 8.75/8.75 ohm per device;\nPNP turn-off buffers, Miller clamps, booster, DESAT"
 		(exclude_from_sim no)
 		(at 214.5 98 0)
@@
 		)
 	)
-	(text "gdrv.channel() 6 x SG2M040170HJ: NSI6651ASC-Q1 +18/-3.5 V, 8.75/7.5 ohm per device;\nPNP turn-off buffers, Miller clamps, booster, DESAT"
+	(text "gdrv.channel() 6 x SG2M040170HJ: NSI6651ASC-Q1 +18/-3.5 V, 8.75/8.75 ohm per device;\nPNP turn-off buffers, Miller clamps, booster, DESAT"
 		(exclude_from_sim no)
 		(at 22.5 186 0)
@@
 		)
 	)
-	(text "gdrv.channel() 6 x SG2M040170HJ: NSI6651ASC-Q1 +18/-3.5 V, 8.75/7.5 ohm per device;\nPNP turn-off buffers, Miller clamps, booster, DESAT; bias SN6505B + T_BIAS4"
+	(text "gdrv.channel() 6 x SG2M040170HJ: NSI6651ASC-Q1 +18/-3.5 V, 8.75/8.75 ohm per device;\nPNP turn-off buffers, Miller clamps, booster, DESAT; bias SN6505B + T_BIAS4"
 		(exclude_from_sim no)
 		(at 310.5 142 0)
@@
 		)
 	)
-	(text "gdrv.channel() 6 x SG2M040170HJ: NSI6651ASC-Q1 +18/-3.5 V, 8.75/7.5 ohm per device;\nPNP turn-off buffers, Miller clamps, booster, DESAT; bias SN6505B + T_BIAS4"
+	(text "gdrv.channel() 6 x SG2M040170HJ: NSI6651ASC-Q1 +18/-3.5 V, 8.75/8.75 ohm per device;\nPNP turn-off buffers, Miller clamps, booster, DESAT; bias SN6505B + T_BIAS4"
 		(exclude_from_sim no)
 		(at 310.5 98 0)
@@
 		)
 	)
-	(text "gdrv.channel() 6 x SG2M040170HJ: NSI6651ASC-Q1 +18/-3.5 V, 8.75/7.5 ohm per device;\nPNP turn-off buffers, Miller clamps, booster, DESAT"
+	(text "gdrv.channel() 6 x SG2M040170HJ: NSI6651ASC-Q1 +18/-3.5 V, 8.75/8.75 ohm per device;\nPNP turn-off buffers, Miller clamps, booster, DESAT"
 		(exclude_from_sim no)
 		(at 214.5 142 0)
